File: rover/T_REX/gripper_2024/gripper_2024.kicad_pcb (KiCad board)
At the start: 2 copper layers, 54 parts, among them J1 XT30PW-M, J2 XT30PW-F, J3 XT30PW-F, J4 B3B-XH-A_LF__SN_, J5 RJ45, J6 RJ45, SW1 TS09-63-25-WT-160-SMT-TR, SW2 TS09-63-25-WT-160-SMT-TR, SW3 TS09-63-25-WT-160-SMT-TR, SW4 TS09-63-25-WT-160-SMT-TR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

Commit message: Started routing
Parts:
- removed H4: MountingHole_Pad, MountingHole:MountingHole_3.2mm_M3_DIN965_Pad_TopBottom
- added C10: 10uF, Capacitor_SMD:C_0805_2012Metric_Pad1.18x1.45mm_HandSolder, B.Cu at (22.7, 69.8)
- added C11: 10uF, Capacitor_SMD:C_0805_2012Metric_Pad1.18x1.45mm_HandSolder, F.Cu at (32.7, 65.0)
- added C12: 100nF, Capacitor_SMD:C_0805_2012Metric_Pad1.18x1.45mm_HandSolder, F.Cu at (42.2, 27.3)
- added C13: 10uF, Capacitor_SMD:C_0805_2012Metric_Pad1.18x1.45mm_HandSolder, F.Cu at (42.2, 23.0)
- added C14: 10uF, Capacitor_SMD:C_0805_2012Metric_Pad1.18x1.45mm_HandSolder, F.Cu at (50.1, 65.9)
- added C15: 10uF, Capacitor_SMD:C_0805_2012Metric_Pad1.18x1.45mm_HandSolder, F.Cu at (54.6, 65.9)
- added C16: 10uF, Capacitor_SMD:C_0805_2012Metric_Pad1.18x1.45mm_HandSolder, F.Cu at (64.1, 54.6)
- added C17: 10uF, Capacitor_SMD:C_0805_2012Metric_Pad1.18x1.45mm_HandSolder, F.Cu at (69.9, 70.1)
- added C18: 10uF, Capacitor_SMD:C_0805_2012Metric_Pad1.18x1.45mm_HandSolder, B.Cu at (40.6, 49.4)
- added C19: 10uF, Capacitor_SMD:C_0805_2012Metric_Pad1.18x1.45mm_HandSolder, B.Cu at (39.5, 37.1)
- added C20: 10uF, Capacitor_SMD:C_0805_2012Metric_Pad1.18x1.45mm_HandSolder, B.Cu at (37.2, 37.5)
- added C21: 10uF, Capacitor_SMD:C_0805_2012Metric_Pad1.18x1.45mm_HandSolder, B.Cu at (42.0, 43.0)
- added C7: 10uF, Capacitor_SMD:C_0805_2012Metric_Pad1.18x1.45mm_HandSolder, B.Cu at (39.9, 47.7)
- added C9: 100nf, Capacitor_SMD:C_0805_2012Metric_Pad1.18x1.45mm_HandSolder, B.Cu at (22.9, 72.6)
- C3, C4, C5: footprint Capacitor_Tantalum_SMD:CP_EIA-7343-15_Kemet-W_Pad2.25x2.55mm_HandSolder -> Capacitor_SMD:C_0805_2012Metric_Pad1.18x1.45mm_HandSolder; moved to B.Cu
- R11, R12, R13, R14, U4, U5, U6: moved to B.Cu
- moved R1 152.3 mm to (25.3, 36.2)
- moved U6 150.5 mm to (39.9, 40.5), turned to 90 degrees
- moved R14 150.1 mm to (37.1, 45.0)
- moved H3 150.1 mm to (20.5, 18.5)
- moved R13 149.8 mm to (37.1, 42.8), turned to 180 degrees
- moved R11 148.2 mm to (37.2, 39.9), turned to 180 degrees
- moved R16 146.3 mm to (41.0, 40.0), turned to 180 degrees
- moved R12 146.2 mm to (37.1, 47.4)
- moved R17 143.3 mm to (41.0, 50.1), turned to 180 degrees
- moved R15 143.0 mm to (41.0, 44.9), turned to 180 degrees
- moved R18 142.5 mm to (41.0, 55.0), turned to 180 degrees
- moved R2 140.6 mm to (42.2, 32.1), turned to -90 degrees
- moved F3 138.4 mm to (23.6, 63.8), turned to -90 degrees
- moved U4 135.7 mm to (24.6, 41.7), turned to -90 degrees
- moved J6 132.2 mm to (25.3, 87.1)
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Connections:
- net MA_DIAG_A renamed Net-(U1-ENB/DIAGB)
- net MA_DIAG_B renamed Net-(U1-ENA/DIAGB)
- net MB_DIAG_A renamed Net-(U2-ENB/DIAGB)
- net MB_DIAG_B renamed Net-(U2-ENA/DIAGB)
- C6 pad 1: Net-(U7-V_{OUT}) -> 7.4V
- C6 pad 2: Net-(C6-Pad2) -> GND
- C8 pad 1: Net-(C6-Pad2) -> 7.4V
- C8 pad 2: 7.4V -> GND
Routing:
- net 24V: track 0.00 -> 84.2 mm
- net GND: track 0.00 -> 75.7 mm, vias 0 -> 9
- net 7.4V: track 0.00 -> 69.0 mm
- net MA-: track 0.00 -> 34.9 mm
- net MA+_F: track 0.00 -> 20.8 mm
- net 5V: track 0.00 -> 20.1 mm
- net Net-(F4-Pad1): track 0.00 -> 10.5 mm
- net MA+: track 0.00 -> 8.46 mm
- net Net-(U7-V_{IN}): track 0.00 -> 6.48 mm
- net Net-(U1-INA): track 0.00 -> 6.26 mm
- net Net-(U1-INB): track 0.00 -> 3.90 mm
- net Net-(U1-ENB/DIAGB): track 0.00 -> 3.58 mm
- net Net-(U1-ENA/DIAGB): track 0.00 -> 2.68 mm
- added copper zone on In1.Cu, net GND
Other:
- board outline added: 60 x 80.5 mm
- copper layers 2 -> 4

Commit message: Final V1 version, ready to order
Parts:
- removed C14, C15, C16, C17, C18, C19, C20, C21: 10uF, Capacitor_SMD:C_0805_2012Metric_Pad1.18x1.45mm_HandSolder
- removed C4, C5: 47nF, Capacitor_SMD:C_0805_2012Metric_Pad1.18x1.45mm_HandSolder
- removed F4: 4A, Custom:3425L200_60MR
- removed R11, R12, R13, R14: 60, Resistor_SMD:R_0805_2012Metric_Pad1.20x1.40mm_HandSolder
- added D2: R, LED_SMD:LED_0805_2012Metric_Pad1.15x1.40mm_HandSolder, F.Cu at (47.8, 75.0)
- added D3: R, LED_SMD:LED_0805_2012Metric_Pad1.15x1.40mm_HandSolder, F.Cu at (41.4, 75.0)
- added D4: R, LED_SMD:LED_0805_2012Metric_Pad1.15x1.40mm_HandSolder, F.Cu at (58.7, 75.0)
- added D5: R, LED_SMD:LED_0805_2012Metric_Pad1.15x1.40mm_HandSolder, F.Cu at (52.4, 75.0)
- added R21: 0, Resistor_SMD:R_0805_2012Metric_Pad1.20x1.40mm_HandSolder, B.Cu at (41.7, 38.2)
- added R23: 1K, Resistor_SMD:R_0805_2012Metric_Pad1.20x1.40mm_HandSolder, F.Cu at (52.4, 68.3)
- added R24: 3.3K, Resistor_SMD:R_0805_2012Metric_Pad1.20x1.40mm_HandSolder, F.Cu at (58.8, 71.7)
- added U8: INA219AxD, Package_SO:SOIC-8_3.9x4.9mm_P1.27mm, B.Cu at (32.7, 88.0)
- C10, C9, U4, U5: moved to F.Cu
- C11: value 10uF -> 100nF; moved to B.Cu
- J4: footprint digikey-footprints:PinHeader_1x3_P2.5mm_Drill1.1mm -> Connector_JST:JST_XH_B3B-XH-AM_1x03_P2.50mm_Vertical
- R10: value 3.3K -> 0; moved to B.Cu
- R6: value 1K -> 3.3K
- R7: value 3.3K -> 0.010; footprint Resistor_SMD:R_0805_2012Metric_Pad1.20x1.40mm_HandSolder -> Resistor_SMD:R_1206_3216Metric_Pad1.30x1.75mm_HandSolder; moved to B.Cu
- moved H1 99.3 mm to (20.5, 102.5)
- moved H2 89.4 mm to (20.5, 19.5)
- moved U4 69.4 mm to (72.5, 91.9), turned to 90 degrees
- moved U5 60.0 mm to (64.5, 91.9), turned to 90 degrees
- moved R10 59.1 mm to (23.2, 35.7)
- moved C8 54.4 mm to (36.4, 83.1), turned to 90 degrees
- moved H3 52.5 mm to (73.0, 19.5)
- moved C6 52.1 mm to (30.7, 83.1), turned to 90 degrees
- moved R7 51.0 mm to (27.1, 87.7)
- moved R5 46.3 mm to (41.4, 68.4), turned to 180 degrees
- moved SW1 45.6 mm to (71.0, 72.6)
- moved R4 45.6 mm to (27.1, 47.4)
- moved J4 44.6 mm to (21.5, 94.5)
- moved R3 41.1 mm to (23.9, 47.4), turned to 90 degrees
- moved R16 37.5 mm to (63.7, 69.9)
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Connections:
- net 5V renamed +5V
- C1 pad 1: 24V -> +24V
- C11 pad 2: 7.4V -> +7.4V
- C2 pad 1: 24V -> +24V
- C6 pad 1: 7.4V -> +7.4V
- C8 pad 1: 7.4V -> +7.4V
- F1 pad 1: MA+_F -> +24V
- F1 pad 2: MA+ -> MA_24V
- F2 pad 1: MB+_F -> +24V
- F2 pad 2: MB+ -> MB_24V
- F3 pad 1: 24V -> +24V
- J1 pad P: 24V -> +24V
- J4 pad 2: Net-(F4-Pad1) -> SERVO_POW
- J5 pad 3: Net-(J5-Pad3) -> unconnected-(J5-Pad3)
- J5 pad 4: Net-(J5-Pad4) -> unconnected-(J5-Pad4)
- J5 pad 5: Net-(J5-Pad5) -> unconnected-(J5-Pad5)
- J5 pad 6: Net-(J5-Pad6) -> unconnected-(J5-Pad6)
- J6 pad 3: Net-(J5-Pad3) -> unconnected-(J6-Pad3)
- J6 pad 4: Net-(J5-Pad4) -> unconnected-(J6-Pad4)
- J6 pad 5: Net-(J5-Pad5) -> unconnected-(J6-Pad5)
- J6 pad 6: Net-(J5-Pad6) -> unconnected-(J6-Pad6)
- R10 pad 1: Net-(U2-ENA/DIAGB) -> SDA
- R10 pad 2: 3.3V -> Net-(U3-D2)
- R15 pad 1: PB_POIGNET_FWD -> +3.3V
- R15 pad 2: 3.3V -> PB_POIGNET_FWD
- R16 pad 2: 3.3V -> +3.3V
- R17 pad 2: 3.3V -> +3.3V
- R18 pad 2: 3.3V -> +3.3V
- R20 pad 1: 7.4V -> +7.4V
- R6 pad 1: Net-(U2-CS) -> Net-(D5-A)
- R6 pad 2: GND -> +3.3V
- R7 pad 1: Net-(U2-ENB/DIAGB) -> SERVO_POW
- R7 pad 2: 3.3V -> +7.4V
- R8 pad 2: 3.3V -> +3.3V
- R9 pad 1: Net-(U1-ENB/DIAGB) -> +3.3V
- R9 pad 2: 3.3V -> Net-(D2-A)
- U1 pad 11: Net-(U1-ENB/DIAGB) -> Net-(D2-A)
- U1 pad 12: 24V -> MA_24V
- U1 pad 15: MA+_F -> MA+
- U1 pad 2: MA+_F -> MA+
- U1 pad 4: 24V -> MA_24V
- U1 pad 5: 24V -> MA_24V
- U2 pad 11: Net-(U2-ENB/DIAGB) -> Net-(D4-A)
- U2 pad 12: 24V -> MB_24V
- U2 pad 14: Net-(U2-ENA/DIAGB) -> Net-(D5-A)
- U2 pad 15: MB+_F -> MB+
- U2 pad 2: MB+_F -> MB+
- U2 pad 4: 24V -> MB_24V
- U2 pad 5: 24V -> MB_24V
- U3 pad 1: 3.3V -> +3.3V
- U3 pad 26: unconnected-(U3-D14-Pad26) -> Net-(U3-D14)
- U3 pad 4: unconnected-(U3-D2-Pad4) -> Net-(U3-D2)
- U7 pad 3: 7.4V -> +7.4V
Routing:
- net +5V: track 20.1 -> 155.5 mm, vias 0 -> 1
- net LED_B: track 0.00 -> 99.3 mm
- net 24V: track 84.2 -> 0.00 mm
- net MOSI: track 0.00 -> 79.4 mm
- net CANH: track 0.00 -> 77.8 mm
- net CS_Poignet: track 0.00 -> 77.0 mm, vias 0 -> 1
- net SCK: track 0.00 -> 76.5 mm, vias 0 -> 1
- net CANL: track 0.00 -> 72.8 mm
- net LED_G: track 0.00 -> 72.0 mm, vias 0 -> 1
- net CS_Rotation: track 0.00 -> 71.3 mm, vias 0 -> 1
- net 7.4V: track 69.0 -> 0.00 mm
- net MISO: track 0.00 -> 66.3 mm
- net SDA: track 0.00 -> 59.2 mm
- net Net-(U2-INA): track 0.00 -> 58.6 mm, vias 0 -> 2
- net Net-(U2-INB): track 0.00 -> 57.1 mm, vias 0 -> 2
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- added copper zone on F.Cu, net +24V
- added copper zone on In2.Cu, net +3.3V
- added copper zone on B.Cu, net +7.4V
- added copper zone on F.Cu, net GND
Other:
- board size 60 x 80.5 mm -> 59.5 x 90 mm
- board text added: "-"
- board text added: "24V / 6S"
- board text added: "5V ONLY"
- board text added: "7.4V"
- board text added: "<-USB"
- board text added: "B_MA"
- board text added: "B_MB"
- board text added: "CCW"
- board text added: "CW"
- board text added: "DWN"
- board text added: "ENC_MA"
- board text added: "ENC_MB"
- board text added: "FMA"
- board text added: "FMB"
- board text added: "FML"
- board text added: "MA"
- board text added: "MB"
- board text added: "Rovus - Gripper Made by Philippe Michaud 2024-03-27 (yinke en 3 jours fait pas chier) - Bonne nuit"
- board text added: "UP"
- board text added: "~"

Commit message: BOM
Parts:
- J4: footprint Connector_JST:JST_XH_B3B-XH-AM_1x03_P2.50mm_Vertical -> Connector_JST:JST_XH_B3B-XH-A_1x03_P2.50mm_Vertical
- U4, U5: footprint Connector_JST:JST_XH_B6B-XH-AM_1x06_P2.50mm_Vertical -> Connector_JST:JST_XH_B6B-XH-A_1x06_P2.50mm_Vertical
- renumbered LED1 to D6
