File: rover/T_REX/terminaison_can/terminaison_can.kicad_sch (KiCad schematic)
At the start: 9 parts

Commit message: fix terminaison
Parts:
- removed C3: 47nF, Capacitor_SMD:C_0805_2012Metric_Pad1.18x1.45mm_HandSolder, symbol Device:C
- removed R3, R4: 60, Resistor_SMD:R_0805_2012Metric_Pad1.20x1.40mm_HandSolder, symbol Device:R
Other:
- moved on the sheet: C2, R1, R2

Commit message: Compass PCB
Other:
- moved on the sheet: C2, D1, R1, R2, R5
Changed lines of the file:
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@@
 	)
 	(junction
-		(at 113.03 64.77)
+		(at 109.22 64.77)
 		(diameter 0)
 		(color 0 0 0 0)
@@
 	(wire
 		(pts
-			(xy 106.68 64.77) (xy 113.03 64.77)
+			(xy 102.87 64.77) (xy 109.22 64.77)
 		)
 		(stroke
@@
 	(wire
 		(pts
-			(xy 113.03 64.77) (xy 120.65 64.77)
+			(xy 109.22 64.77) (xy 116.84 64.77)
 		)
 		(stroke
@@
 	(global_label "CAN_H"
 		(shape input)
-		(at 99.06 64.77 180)
+		(at 95.25 64.77 180)
 		(fields_autoplaced yes)
 		(effects
@@
 		)
 		(property "Intersheetrefs" "${INTERSHEET_REFS}"
-			(at 90.0876 64.77 0)
+			(at 86.2776 64.77 0)
 			(effects
 				(font
@@
 	(global_label "CAN_L"
 		(shape input)
-		(at 128.27 64.77 0)
+		(at 124.46 64.77 0)
 		(fields_autoplaced yes)
 		(effects
@@
 		)
 		(property "Intersheetrefs" "${INTERSHEET_REFS}"
-			(at 136.94 64.77 0)
+			(at 133.13 64.77 0)
 			(effects
 				(font
@@
 	(symbol
 		(lib_id "power:GND")
-		(at 113.03 72.39 0)
+		(at 109.22 72.39 0)
 		(unit 1)
 		(exclude_from_sim no)
@@
 		(fields_autoplaced yes)
 		(property "Reference" "#PWR01"
-			(at 113.03 78.74 0)
+			(at 109.22 78.74 0)
 			(effects
 				(font
@@
 		)
 		(property "Value" "GND"
-			(at 113.03 77.47 0)
+			(at 109.22 77.47 0)
 			(effects
 				(font
@@
 		)
 		(property "Footprint" ""
-			(at 113.03 72.39 0)
+			(at 109.22 72.39 0)
 			(effects
 				(font
@@
 		)
 		(property "Datasheet" ""
-			(at 113.03 72.39 0)
+			(at 109.22 72.39 0)
 			(effects
 				(font
@@
 		)
 		(property "Description" "Power symbol creates a global label with name \"GND\" , ground"
-			(at 113.03 72.39 0)
+			(at 109.22 72.39 0)
 			(effects
 				(font
@@
 	(symbol
 		(lib_id "Device:R")
-		(at 124.46 64.77 90)
+		(at 120.65 64.77 90)
 		(unit 1)
 		(exclude_from_sim no)
@@
 		(fields_autoplaced yes)
 		(property "Reference" "R2"
-			(at 124.46 58.42 90)
+			(at 120.65 58.42 90)
 			(effects
 				(font
@@
 		)
 		(property "Value" "60"
-			(at 124.46 60.96 90)
+			(at 120.65 60.96 90)
 			(effects
 				(font
@@
 		)
 		(property "Footprint" "Resistor_SMD:R_0805_2012Metric_Pad1.20x1.40mm_HandSolder"
-			(at 124.46 66.548 90)
+			(at 120.65 66.548 90)
 			(effects
 				(font
@@
 		)
 		(property "Datasheet" "~"
-			(at 124.46 64.77 0)
+			(at 120.65 64.77 0)
 			(effects
 				(font
@@
 		)
 		(property "Description" "Resistor"
-			(at 124.46 64.77 0)
+			(at 120.65 64.77 0)
 			(effects
 				(font
@@
 	(symbol
 		(lib_id "Device:R")
-		(at 149.86 59.69 180)
+		(at 148.59 63.5 180)
 		(unit 1)
 		(exclude_from_sim no)
@@
 		(fields_autoplaced yes)
 		(property "Reference" "R5"
-			(at 152.4 58.4199 0)
+			(at 151.13 62.2299 0)
 			(effects
 				(font
@@
 		)
 		(property "Value" "2k"
-			(at 152.4 60.9599 0)
+			(at 151.13 64.7699 0)
 			(effects
 				(font
@@
 		)
 		(property "Footprint" "Resistor_SMD:R_0805_2012Metric_Pad1.20x1.40mm_HandSolder"
-			(at 151.638 59.69 90)
+			(at 150.368 63.5 90)
 			(effects
 				(font
@@
 		)
 		(property "Datasheet" "~"
-			(at 149.86 59.69 0)
+			(at 148.59 63.5 0)
 			(effects
 				(font
@@
 		)
 		(property "Description" "Resistor"
-			(at 149.86 59.69 0)
+			(at 148.59 63.5 0)
 			(effects
 				(font
@@
 	(symbol
 		(lib_id "power:GND")
-		(at 149.86 71.12 0)
+		(at 148.59 74.93 0)
 		(unit 1)
 		(exclude_from_sim no)
@@
 		(fields_autoplaced yes)
 		(property "Reference" "#PWR06"
-			(at 149.86 77.47 0)
+			(at 148.59 81.28 0)
 			(effects
 				(font
@@
 		)
 		(property "Value" "GND"
-			(at 149.86 76.2 0)
+			(at 148.59 80.01 0)
 			(effects
 				(font
@@
 		)
 		(property "Footprint" ""
-			(at 149.86 71.12 0)
+			(at 148.59 74.93 0)
 			(effects
 				(font
@@
 		)
 		(property "Datasheet" ""
-			(at 149.86 71.12 0)
+			(at 148.59 74.93 0)
 			(effects
 				(font
@@
 		)
 		(property "Description" "Power symbol creates a global label with name \"GND\" , ground"
-			(at 149.86 71.12 0)
+			(at 148.59 74.93 0)
 			(effects
 				(font
@@
 	(symbol
 		(lib_id "Device:C")
-		(at 113.03 68.58 0)
+		(at 109.22 68.58 0)
 		(unit 1)
 		(exclude_from_sim no)
@@
 		(dnp no)
 		(property "Reference" "C2"
-			(at 115.824 67.31 0)
+			(at 112.014 67.31 0)
 			(effects
 				(font
@@
 		)
 		(property "Value" "47nF"
-			(at 115.824 69.85 0)
+			(at 112.014 69.85 0)
 			(effects
 				(font
@@
 		)
 		(property "Footprint" "Capacitor_SMD:C_0805_2012Metric_Pad1.18x1.45mm_HandSolder"
-			(at 113.9952 72.39 0)
+			(at 110.1852 72.39 0)
 			(effects
 				(font
@@
 		)
 		(property "Datasheet" "~"
-			(at 113.03 68.58 0)
+			(at 109.22 68.58 0)
 			(effects
 				(font
@@
 		)
 		(property "Description" "Unpolarized capacitor"
-			(at 113.03 68.58 0)
+			(at 109.22 68.58 0)
 			(effects
 				(font
@@
 	(symbol
 		(lib_id "Device:LED")
-		(at 149.86 67.31 90)
+		(at 148.59 71.12 90)
 		(unit 1)
 		(exclude_from_sim no)
@@
 		(fields_autoplaced yes)
 		(property "Reference" "D1"
-			(at 153.67 67.6274 90)
+			(at 152.4 71.4374 90)
 			(effects
 				(font
@@
 		)
 		(property "Value" "LED"
-			(at 153.67 70.1674 90)
+			(at 152.4 73.9774 90)
 			(effects
 				(font
@@
 		)
 		(property "Footprint" "LED_SMD:LED_0805_2012Metric_Pad1.15x1.40mm_HandSolder"
-			(at 149.86 67.31 0)
+			(at 148.59 71.12 0)
 			(effects
 				(font
@@
 		)
 		(property "Datasheet" ""
-			(at 149.86 67.31 0)
+			(at 148.59 71.12 0)
 			(effects
 				(font
@@
 		)
 		(property "Description" "150080RS75000 | 732-4984-2-ND "
-			(at 149.86 67.31 0)
+			(at 148.59 71.12 0)
 			(effects
 				(font
@@
 	(symbol
 		(lib_id "Device:R")
-		(at 102.87 64.77 90)
+		(at 99.06 64.77 90)
 		(unit 1)
 		(exclude_from_sim no)
@@
 		(fields_autoplaced yes)
 		(property "Reference" "R1"
-			(at 102.87 58.42 90)
+			(at 99.06 58.42 90)
 			(effects
 				(font
@@
 		)
 		(property "Value" "60"
-			(at 102.87 60.96 90)
+			(at 99.06 60.96 90)
 			(effects
 				(font
@@
 		)
 		(property "Footprint" "Resistor_SMD:R_0805_2012Metric_Pad1.20x1.40mm_HandSolder"
-			(at 102.87 66.548 90)
+			(at 99.06 66.548 90)
 			(effects
 				(font
@@
 		)
 		(property "Datasheet" "~"
-			(at 102.87 64.77 0)
+			(at 99.06 64.77 0)
 			(effects
 				(font
@@
 		)
 		(property "Description" "Resistor"
-			(at 102.87 64.77 0)
+			(at 99.06 64.77 0)
 			(effects
 				(font
@@
 	(symbol
 		(lib_id "power:VCC")
-		(at 149.86 55.88 0)
+		(at 148.59 59.69 0)
 		(unit 1)
 		(exclude_from_sim no)
@@
 		(fields_autoplaced yes)
 		(property "Reference" "#PWR05"
-			(at 149.86 59.69 0)
+			(at 148.59 63.5 0)
 			(effects
 				(font
@@
 		)
 		(property "Value" "VCC"
-			(at 149.86 50.8 0)
+			(at 148.59 54.61 0)
 			(effects
 				(font
@@
 		)
 		(property "Footprint" ""
-			(at 149.86 55.88 0)
+			(at 148.59 59.69 0)
 			(effects
 				(font
@@
 		)
 		(property "Datasheet" ""
-			(at 149.86 55.88 0)
+			(at 148.59 59.69 0)
 			(effects
 				(font
@@
 		)
 		(property "Description" "Power symbol creates a global label with name \"VCC\""
-			(at 149.86 55.88 0)
-			(effects
-				(font
+			(at 148.59 59.69 0)
+			(effects
+				(font
