File: rover/T_REX/pdb/pdb.kicad_sch (KiCad schematic)
At the start: 74 parts, among them J1 Screw_Terminal_01x04, Q1 GSF2302, Q2 GSF2302, U3 TJA1050T_CM_118

Commit message: pdb pcb
Parts:
- removed E_12V_SIYI_A2_IN_1, E_12V_SIYI_A2_OUT_1, E_12V_SIYI_R1M_IN_1, E_12V_SIYI_R1M_IN_2, E_12V_SIYI_R1M_IN_3, E_12V_SIYI_R1M_OUT_1, E_12V_SIYI_R1M_OUT_2, E_12V_SIYI_R1M_OUT_3: RJ45, 54601-908WPLF:AMPHENOL_54601-908WPLF, symbol Connector:RJ45
- added C7, C8, C9: 100uf, Capacitor_SMD:C_0805_2012Metric_Pad1.18x1.45mm_HandSolder, symbol Device:C
- added J2, J3: Screw_Terminal_01x02, 1790335:PHOENIX_1790335_2pin, symbol Connector:Screw_Terminal_01x02
- added JP1, JP2, JP3, JP4, JP5, JP6: Jumper_2_Open, Connector_PinHeader_2.54mm:PinHeader_1x02_P2.54mm_Vertical, symbol Jumper:Jumper_2_Open
- added R29, R32, R36, R40: 100k, Resistor_SMD:R_0805_2012Metric_Pad1.20x1.40mm_HandSolder, symbol Device:R
- added R30: 1.8M, Resistor_SMD:R_0805_2012Metric_Pad1.20x1.40mm_HandSolder, symbol Device:R
- added R31: 200k, Resistor_SMD:R_0805_2012Metric_Pad1.20x1.40mm_HandSolder, symbol Device:R
- added R33: 6.2M, Resistor_SMD:R_0805_2012Metric_Pad1.20x1.40mm_HandSolder, symbol Device:R
- added R34: 240k, Resistor_SMD:R_0805_2012Metric_Pad1.20x1.40mm_HandSolder, symbol Device:R
- added R35: 262k, Resistor_SMD:R_0805_2012Metric_Pad1.20x1.40mm_HandSolder, symbol Device:R
- added R37: 13M, Resistor_SMD:R_0805_2012Metric_Pad1.20x1.40mm_HandSolder, symbol Device:R
- added R38: 270k, Resistor_SMD:R_0805_2012Metric_Pad1.20x1.40mm_HandSolder, symbol Device:R
- added R39: 30k, Resistor_SMD:R_0805_2012Metric_Pad1.20x1.40mm_HandSolder, symbol Device:R
- added U10: ~, CRJ036-5-TH:CUI_CRJ036-5-TH, symbol Custom:CRJ036-5-TH_2x4
- added U4, U6, U8: ~, Package_TO_SOT_SMD:TSOT-23-8_HandSoldering, symbol Custom:LTC4365
- added U5, U7, U9: ~, Custom:SOIC-8-1EP_3.9x4.9mm_P1.27mm_hand_solder, symbol Custom:DMG4822SSD
- D4: footprint CLP6C-FKB-CKNPRGJBB7A363:CLP6C-FKB-CKNPRGJBB7A363_CRE -> footprints:CLP6C-FKB-CKNPRGJBB7A363_CRE-M
- E_12V_1, E_24V_POE_IN_1, E_24V_POE_OUT_1, E_24V_POE_OUT_2: footprint 54601-908WPLF:AMPHENOL_54601-908WPLF -> A-2014-2-4-N-T-R:ASSMANN_A-2014-2-4-N-T-R
- F1, F2: footprint (none) -> 3568-20:FUSE_3568-20
- J1: footprint (none) -> 1790335:PHOENIX_1790335_4pin
- U1: footprint (none) -> Package_SO:SOIC-14_3.9x8.7mm_P1.27mm
- U2: footprint (none) -> ESP32-DEVKIT-V1:MODULE_ESP32_DEVKIT_V1
Connections:
- net +12V: now also C8.1, JP2.2 (B), JP5.2 (B), U6.7 (V_{out}), U7.5 (D2), U7.6 (D2); no longer J1.2 (Pin_2)
- net +24V: now also C9.1, JP3.2 (B), JP6.2 (B), U8.7 (V_{out}), U9.5 (D2), U9.6 (D2); no longer J1.3 (Pin_3)
- net +5V: now also C7.1, JP1.2 (B), JP4.2 (B), U4.7 (V_{out}), U5.5 (D2), U5.6 (D2); no longer J1.1 (Pin_1)
- net ACC1_LOAD_LOW: now also E_12V_1.8
- net ACC2_LOAD_LOW: no longer E_12V_1.8
- net CAM_POW_0: now also U10.1_1T
- net CAM_POW_1: now also U10.2_1T
- net CAM_POW_2: now also U10.3_1T
- net CAM_POW_3: now also U10.4_1T
- net CANH: now also J3.1 (Pin_1)
- net CANL: now also J3.2 (Pin_2)
- net GND: now also C7.2, C8.2, C9.2, J2.2 (Pin_2), R32.1, R35.1, R39.1, U10.1_8T, U10.2_2T, U10.3_2T, U10.4_2T, U10.S1 (GND), U4.4 (GND), U6.4 (GND), U8.4 (GND)
- net LED_B: now also U2.8 (D5); no longer U2.21 (D32)
- net PWM_0: now also U2.21 (D32), U10.1_7T
- net RX+_0: now also U10.1_1B, U10.1_5T
- net RX+_1: now also U10.2_1B, U10.2_5T
- net RX+_2: now also U10.3_1B, U10.3_5T
- net RX+_3: now also U10.4_1B, U10.4_5T
- net RX-_0: now also U10.1_2B, U10.1_6T
- net RX-_1: now also U10.2_2B, U10.2_6T
- net RX-_2: now also U10.3_2B, U10.3_6T
- net RX-_3: now also U10.4_2B, U10.4_6T
- net TX+_0: now also U10.1_3B, U10.1_3T
- net TX+_1: now also U10.2_3B, U10.2_3T
- net TX+_2: now also U10.3_3B, U10.3_3T
- net TX+_3: now also U10.4_3B, U10.4_3T
- net TX-_0: now also U10.1_4T, U10.1_6B
- net TX-_1: now also U10.2_4T, U10.2_6B
- net TX-_2: now also U10.3_4T, U10.3_6B
- net TX-_3: now also U10.4_4T, U10.4_6B
- net PWM_1: now reaches U2.22 (D33)
- net PWM_1: now also U10.1_2T
- new net: R38.1, R39.2, U8.3 (OV)
- new net: U5.1 (S1), U5.3 (S2)
- new net: U4.8 (GATE), U5.2 (G1), U5.4 (G2)
- new net: J2.1 (Pin_1), JP1.1 (A), JP2.1 (A), JP3.1 (A)
- new net: R37.1, R38.2, U8.2 (UV)
- new net: R30.1, R31.2, U4.2 (UV)
- new net: R31.1, R32.2, U4.3 (OV)
- new net: R29.1, U4.5 (SHDN)
- new net: U9.1 (S1), U9.3 (S2)
- new net: U8.8 (GATE), U9.2 (G1), U9.4 (G2)
- new net: R40.1, U8.5 (SHDN)
- new net: R33.1, R34.2, U6.2 (UV)
- new net: R36.1, U6.5 (SHDN)
- new net: U7.1 (S1), U7.3 (S2)
- new net: U6.8 (GATE), U7.2 (G1), U7.4 (G2)
- new net: R34.1, R35.2, U6.3 (OV)
- new net +12V IN: JP5.1 (A), R33.2, R36.2, U6.1 (V_{in}), U7.7 (D1), U7.8 (D1)
- new net +12V_IN: J1.2 (Pin_2)
- new net +24V IN: JP6.1 (A), R37.2, R40.2, U8.1 (V_{in}), U9.7 (D1), U9.8 (D1)
- new net +24V_IN: J1.3 (Pin_3)
- new net +5V IN: J1.1 (Pin_1), JP4.1 (A), R29.2, R30.2, U4.1 (V_{in}), U5.7 (D1), U5.8 (D1)
- no-connect marks 72 -> 80
Other:
- note added: "12V Over/Under Voltage Protection (10.83V - 13.541)"
- note added: "24V Over/Under Voltage Protection (22.16-24.63)"
- note added: "5V Over/Under Voltage Protection (3.5-5.25)"
- note added: "I_{uv} = 10uA V_{os} = 3mV UV_{th} = 11.0V OV_{th} = 13.0V R1 = 62k R2 = 240k R3 = 6.2M"
- note added: "I_{uv} = 10uA V_{os} = 3mV UV_{th} = 22V OV_{th} = 25V R1 = 13.0M R2 = 270k R3 = 30k"
- note added: "I_{uv} = 10uA V_{os} = 3mV UV_{th} = 3.5V OV_{th} = 5.5V R1 = 100k R2 = 200k R3 = 1.8M"
- note added: "Power OUT rj45 Switch"
- note added: "R3 = V_{os}/I_{uv} * (UV_{th} - 0.5)/0.5 R1 = (0.5/OV_{oh}) * (V_{os}/I_{uv}) + R3) R2 = V_{os}/I_{uv} - R1"
- note added: "Resistor for voltage range"
- note added: "Screw terminal faire le bon footprint!! 3x (le bon nb) Package Infinion watcher plate en dessous de la chip"
- note removed: "TODO: (x) ESP32 (x) Board Power in (x) Diag LED (x) Fuse Cam + Modems ( ) Wrong Voltage Protection on input (see LTC4365)"
- moved on the sheet: C3, C4, C5, C6, D1, D10, D11, D2, D3, D5, D6, D7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

Commit message: PDB routing
Parts:
- removed C7, C8, C9: 100uf, Capacitor_SMD:C_0805_2012Metric_Pad1.18x1.45mm_HandSolder, symbol Device:C
- added C7, C8, C9: 100uf, Capacitor_THT:CP_Radial_D5.0mm_P2.00mm, symbol Device:C_Polarized
Connections:
- net +12V_IN is gone; now on net +12V IN: J1.2 (Pin_2)
- net +24V_IN is gone; now on net +24V IN: J1.3 (Pin_3)
- net +12V: now also R3.2, R6.2, C8.1
- net +24V: now also C9.1
- net +5V: now also C7.1
- net ACC1_LOAD_LOW: now also D10.1 (K)
- net ACC2_LOAD_LOW: now also D11.1 (K)
- net CAM_SIGN_2: now also U2.22 (D33); no longer U2.11 (D21)
- net CAM_SIGN_3: now also U2.21 (D32); no longer U2.14 (D22)
- net GND: now also C7.2, C8.2, C9.2; no longer D10.1 (K), D11.1 (K), R3.2, R6.2
- net LED_B: now also U2.24 (D26); no longer U2.8 (D5)
- net LED_R: now also U2.26 (D14); no longer U2.24 (D26)
- net PWM_0: now also U2.11 (D21); no longer U2.21 (D32)
- net PWM_1: now also U2.14 (D22); no longer U2.22 (D33)
- net RXC: now also U2.7 (TX2); no longer U2.5 (D4)
- net TXC: now also U2.6 (RX2); no longer U2.28 (D13)
- net at R15.2: now also U1.15 (VS); no longer U1. (VS)
Other:
- moved on the sheet: D10, D11, Q1, Q2, R1, R2, R3, R4, R5, R6

Commit message: Generated BOM
Parts:
- C1, C4: value 100nf -> 100nF
- C2, C3: value 10uf -> 10uF
- C7, C8, C9: value 100uf -> 100uF
Changed lines of the file:
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@@
 			)
 		)
-		(property "Value" "100uf"
+		(property "Value" "100uF"
 			(at 149.86 362.3309 0)
 			(effects
@@
 			)
 		)
-		(property "Value" "100uf"
+		(property "Value" "100uF"
 			(at 234.95 362.3309 0)
 			(effects
@@
 			)
 		)
-		(property "Datasheet" ""
+		(property "Datasheet" "~"
 			(at 312.42 31.75 0)
 			(effects
@@
 			)
 		)
-		(property "Value" "10uf"
+		(property "Value" "10uF"
 			(at 186.69 64.7699 0)
 			(effects
@@
 			)
 		)
-		(property "Value" "10uf"
+		(property "Value" "10uF"
 			(at 198.12 137.1599 0)
 			(effects
@@
 			)
 		)
-		(property "Datasheet" ""
+		(property "Datasheet" "~"
 			(at 300.99 31.75 0)
 			(effects
@@
 			)
 		)
-		(property "Value" "100nf"
+		(property "Value" "100nF"
 			(at 209.55 137.1599 0)
 			(effects
@@
 			)
 		)
-		(property "Value" "100nf"
+		(property "Value" "100nF"
 			(at 198.12 64.7699 0)
 			(effects
@@
 			)
 		)
-		(property "Value" "100uf"
+		(property "Value" "100uF"
 			(at 64.77 362.3309 0)
 			(effects

Commit message: dik
Parts:
- R35: value 262k -> 62k
Changed lines of the file:
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@@
 			)
 		)
-		(property "Value" "262k"
+		(property "Value" "62k"
 			(at 109.474 384.81 90)
 			(effects
