File: exo/ACE 2025/BNOV2/BNO_BREAKOUT.kicad_sch (KiCad schematic)
At the start: 18 parts, among them J1 Conn_02x04_Counter_Clockwise, J2 RJ45, SW1 SW_SPDT, U1 4754, U2 PCA9615DPZ, U3 AP7361C-33E

Commit message: BNOV2 V0.2
Parts:
- removed C4: 4.7uF, Capacitor_SMD:C_1812_4532Metric_Pad1.57x3.40mm_HandSolder, symbol Device:C
- removed D2: BAV99, Package_TO_SOT_SMD:SOT-23, symbol Diode:BAV99
- removed J1: Conn_02x04_Counter_Clockwise, Molex:Molex_Nano-Fit_105314-xx08_2x04_P2.50mm_Horizontal, symbol Connector_Generic:Conn_02x04_Counter_Clockwise
- C2, C3: value 4.7uF -> 1n
- D4: footprint (none) -> Diode_SMD:D_0805_2012Metric
Connections:
- net 3V3: now also C2.1, C3.1
- net SCL: no longer C3.1
- net SDA: no longer C2.1
Other:
- moved on the sheet: C2, C3, D4

Commit message: Changement BNO et moustache
Parts:
- U2: footprint Other symbols:TSSOP10_SOT552-1_NXP -> Package_SO:TSSOP-10_3x3mm_P0.5mm
Changed lines of the file:
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@@
 			)
 		)
-		(property "Footprint" "Other symbols:TSSOP10_SOT552-1_NXP"
+		(property "Footprint" "Package_SO:TSSOP-10_3x3mm_P0.5mm"
 			(at 158.75 116.84 0)
 			(effects
@@
 		)
 		(instances
-			(project ""
+			(project "BNO_BREAKOUT"
 				(path "/eb12f455-3dfb-4bde-967e-67cb3a10b836"
 					(reference "U2")
@@
 		)
 		(instances
-			(project ""
+			(project "BNO_BREAKOUT"
 				(path "/eb12f455-3dfb-4bde-967e-67cb3a10b836"
 					(reference "J2")
