File: exo/ACE 2025/Motherboard/MOBO_V2/ESP32_SD.kicad_sch (KiCad schematic)
At the start: 0 parts

Commit message: push schema électrique
Parts:
- added J601: Conn_Module_SD, Connector_PinSocket_2.54mm:PinSocket_1x06_P2.54mm_Vertical, symbol Connector_Generic:Conn_01x06
- added U601: ~, MDT320E01001:AMPHENOL_MDT320E01001, symbol connecteur_m2_SoM_esp32_keyE:connecteur_SOM_ESP32_V2
Connections:
- new net CS_1: J601.2 (Pin_2), U601.20 (CS_1)
- new net CS_2: U601.21 (CS_2)
- new net GND: J601.6 (Pin_6)
- new net GPIO15: U601.40 (GPIO15)
- new net GPIO16: U601.41 (GPIO16)
- new net GPIO26: U601.42 (GPIO26)
- new net GPIO33: U601.43 (GPIO33)
- new net GPIO34: U601.44 (GPIO34)
- new net GPIO38_ADDRESSABLE_LED: U601.6 (GPIO38&LED)
- new net GPIO45: U601.52 (GPIO45)
- new net GPIO46: U601.53 (GPIO46)
- new net GPIO47: U601.34 (RST_OTHER)
- new net GPIO48/CAN_INT: U601.36 (GPIO48)
- new net I2S_BCLK: U601.8 (I2S_BCLK)
- new net I2S_DIN/DOUT: U601.12 (I2S_DIN/DOUT)
- new net I2S_WS: U601.10 (I2S_WS)
- new net PWM_1: U601.64 (PWM_1_PCA)
- new net PWM_2: U601.66 (PWM_2_PCA)
- new net PWM_3: U601.68 (PWM_3_PCA)
- new net PWM_4: U601.70 (PWM_4_PCA)
- new net SPI_CLK_ESP32: J601.4 (Pin_4), U601.23 (SPI_CLK)
- new net SPI_MISO_ESP32: J601.5 (Pin_5), U601.37 (SPI_MISO)
- new net SPI_MOSI_ESP32: J601.3 (Pin_3), U601.35 (SPI_MOSI)
- new net Vcc_3V3: J601.1 (Pin_1)
Other:
- note added: "CS"
- note added: "Connecteur pour lecteur de carte µSD."
- note added: "MOSI CLK MISO"
