File: exo/ACE 2025/Motherboard/MOBO_V2/Connecteurs.kicad_sch (KiCad schematic)
At the start: 10 parts, among them J701 RJ45, J702 RJ45, J703 RJ45

Commit message: ajout infromation et d'épaisseur des traces selon le netclass et de joli couleur hehe
Parts:
- added JP703, JP704, JP705, JP706, JP707, JP708, JP709, JP710, JP711, JP712, JP713, JP714: SolderJumper_2_Bridged, Jumper:SolderJumper-2_P1.3mm_Bridged_RoundedPad1.0x1.5mm, symbol Jumper:SolderJumper_2_Bridged
- renumbered H703 to H702, H702 to H703
Connections:
- net D.SCL1: now also JP705.1 (A); no longer J702.3
- net D.SCL2: now also JP709.1 (A); no longer J702.4
- net D.SDA1: now also JP711.1 (A); no longer J702.5
- net D.SDA2: now also JP713.1 (A); no longer J702.6
- net DOS.SCL1: now also JP703.1 (A); no longer J701.3
- net DOS.SCL2: now also JP707.1 (A); no longer J701.4
- net DOS.SDA1: now also JP704.1 (A); no longer J701.5
- net DOS.SDA2: now also JP708.1 (A); no longer J701.6
- net D_SCL+: now also J702.3, JP705.2 (B)
- net D_SCL-: now also J702.4, JP709.2 (B)
- net G.SCL1: now also JP706.1 (A); no longer J703.3
- net G.SCL2: now also JP710.1 (A); no longer J703.4
- net G.SDA1: now also JP712.1 (A); no longer J703.5
- net G.SDA2: now also JP714.1 (A); no longer J703.6
- net G_SCL+: now also J703.3, JP706.2 (B)
- net G_SCL-: now also J703.4, JP710.2 (B)
- new net DOS_SCL+: J701.3, JP703.2 (B)
- new net DOS_SCL-: J701.4, JP707.2 (B)
- new net DOS_SDA+: J701.5, JP704.2 (B)
- new net DOS_SDA-: J701.6, JP708.2 (B)
- new net D_SDA+: J702.5, JP711.2 (B)
- new net D_SDA-: J702.6, JP713.2 (B)
- new net G_SDA+: J703.5, JP712.2 (B)
- new net G_SDA-: J703.6, JP714.2 (B)
