File: exo/ACE 2025/Motherboard/MOBO_V2/USB.kicad_sch (KiCad schematic)
At the start: 0 parts

Commit message: push schema électrique
Parts:
- added J301: USB_C_UART, Connector_USB:USB_C_Receptacle_G-Switch_GT-USB-7010ASV, symbol Connector:USB_C_Receptacle_USB2.0
- added J302: USB_C_DEBUG, Connector_USB:USB_C_Receptacle_G-Switch_GT-USB-7010ASV, symbol Connector:USB_C_Receptacle_USB2.0
- added R301, R302, R303, R304: 5.1k, Resistor_SMD:R_0603_1608Metric_Pad0.98x0.95mm_HandSolder, symbol Device:R_US
- added U203: ~, MDT320E01001:AMPHENOL_MDT320E01001, symbol connecteur_m2_key_E:connecteur_SOM_ESP32_V2
- added U301: SRV05-4, Package_TO_SOT_SMD:SOT-23-6, symbol Power_Protection:SRV05-4
Connections:
- new net: J301.B5 (CC2), R301.1
- new net: J302.A5 (CC1), R304.1
- new net: J302.B5 (CC2), R302.1
- new net: J301.A5 (CC1), R303.1
- new net DEBUG_D+: J302.A6 (D+), J302.B6 (D+), U203.48 (USB_DEBUG_D+), U301.6 (IO4)
- new net DEBUG_D-: J302.A7 (D-), J302.B7 (D-), U203.46 (USB_DEBUG_D-), U301.4 (IO3)
- new net FT231_D+: J301.A6 (D+), J301.B6 (D+), U203.3 (USB_D+_FT231), U301.3 (IO2)
- new net FT231_D-: J301.A7 (D-), J301.B7 (D-), U203.5 (USB_D-_FT231), U301.1 (IO1)
- new net GND: J301.A1 (GND), J301.A12 (GND), J301.B1 (GND), J301.B12 (GND), J301.S1 (SHIELD), J302.A1 (GND), J302.A12 (GND), J302.B1 (GND), J302.B12 (GND), J302.S1 (SHIELD), R301.2, R302.2, R303.2, R304.2, U301.2 (VN)
- new net VBUS: J301.A4 (VBUS), J301.A9 (VBUS), J301.B4 (VBUS), J301.B9 (VBUS), J302.A4 (VBUS), J302.A9 (VBUS), J302.B4 (VBUS), J302.B9 (VBUS), U301.5 (VP)
- no-connect marks 0 -> 4
