File: rover/2025/PDB/PDB.kicad_sch (KiCad schematic)
At the start: 20 parts, among them J1 USB_C_USB4105-GF-A, SW1 TS09-63-25-WT-160-SMT-TR, SW2 TS09-63-25-WT-160-SMT-TR, U1 ESP32-S3-WROVER, U2 TVS, U3 SN65HVD232

Commit message: .
Parts:
- added J2, J3: Eth-Horiz-54601-908WPLF, RoverFootprint:Ethernet_Horizontal, symbol 0_RoverLibrary:Eth-Horiz-54601-908WPLF
- added JP1: SolderJumper_3_Open, symbol Jumper:SolderJumper_3_Open
- added U4: LDO-LM317DCYR, Package_TO_SOT_SMD:SOT-223-3_TabPin2, symbol 0_RoverLibrary:LDO-LM317DCYR
Connections:
- net +5V: now also JP1.3 (B)
- net CANH: now also J2.1 (CANH), J3.1 (CANH)
- net CANL: now also J2.2 (CANL), J3.2 (CANL)
- net GND: now also J2.6, J2.8, J3.6, J3.8, U4.1 (GND)
- new net: JP1.2 (C), U4.3 (INPUT)
- new net +24V_L: J2.5, J2.7, J3.5, J3.7, JP1.1 (A)
- no-connect marks 12 -> 16
Other:
- note added: "Data input"
- moved on the sheet: C5, H5, H6, H7, H8, SW2

Commit message: PDB progress
Parts:
- removed U4: LDO-LM317DCYR, Package_TO_SOT_SMD:SOT-223-3_TabPin2, symbol 0_RoverLibrary:LDO-LM317DCYR
- added C10, C9: 10 uF, Capacitor_SMD:C_0805_2012Metric_Pad1.18x1.45mm_HandSolder, symbol Device:C
- added C8: 100 nF, Capacitor_SMD:C_0805_2012Metric_Pad1.18x1.45mm_HandSolder, symbol Device:C
- added D1: R, symbol Device:LED
- added D2, D4, D5: B, symbol Device:LED
- added D3: G, symbol Device:LED
- added F1: 20A, 0_RoverFootprint:FUSE_3568-20, symbol 0_RoverLibrary:FuseHolder
- added R4, R5, R6, R7, R8, R9: 1k, Resistor_SMD:R_0805_2012Metric_Pad1.20x1.40mm_HandSolder, symbol Device:R
- added U4: LDO-LM7805MPX/NOPB, Package_TO_SOT_SMD:TO-252-2, symbol 0_RoverLibrary:LDO-TLE4284DV33ATMA1
- added U5: XT60PW-M, RoverFootprint:AMASS_XT60PW-M_1x02_P7.20mm_Horizontal, symbol 0_RoverLibrary:XT60PW-M
- added U6: HSS-VN7004SLHTR, 0_RoverFootprint:OCTAPACK_VN7004_STM-M, symbol 0_RoverLibrary:HSS-VN7004SLHTR
- J1: STATUS (none) -> TO BE APPROVED
- J2, J3, SW1, SW2, U3: STATUS (none) -> APPROVED
- U1: STATUS (none) -> TO BE VERIFIED
- U2: STATYS (none) -> APPROVED
Connections:
- net +24V_L: now also R4.1, U6.1 (OUT), U6.2 (OUT), U6.3 (OUT)
- net +3.3V: now also C10.1, R6.1, U4.2 (OUTPUT)
- net GND: now also C10.2, C8.2, C9.2, D1.1 (K), D2.1 (K), D3.1 (K), D4.1 (K), D5.1 (K), R9.2, U4.1 (GND), U5.1 (-), U6.7 (GND)
- net at JP1.2 (C): now also C8.1, C9.1, U4.3 (INPUT)
- new net: D2.2 (A), R5.2
- new net: D1.2 (A), R4.2
- new net: D4.2 (A), R7.2
- new net: D3.2 (A), R6.2
- new net: D5.2 (A), R8.2
- new net: F1.1, U5.2 (+)
- new net: F1.2, U6.8 (Vcc)
- new net: R9.1, U6.5 (CS)
- new net +12V: R5.1
- new net CAN_LED: R7.1
- new net LED_BUILDIN: R8.1
- new net LOW_PW_EN: U6.4 (INPUT), U6.6 (FR_DIAG)
Other:
- note added: "LDO 3.3V"
- note added: "Power Input"
- note added: "Power LED"
- note added: "TODO: (X) LED Build_in (X) LDO + LED (X) CAN INPUT ( ) Connect selector input (X) Power input ( ) 12V Switches ( ) 24v Switches ( ) Low power en signal ( ) Big power relay ( ) Other"
- note removed: "TODO: ( ) LED Build_in ( ) LDO + LED ( ) CAN INPUT ( ) Power input ( ) 12V Switches ( ) 24v Switches ( ) Low power en signal ( ) Big power relay ( ) Other"
- moved on the sheet: C6, C7, JP1, U3

Commit message: .
Parts:
- removed J2, J3: Eth-Horiz-54601-908WPLF, RoverFootprint:Ethernet_Horizontal, symbol 0_RoverLibrary:Eth-Horiz-54601-908WPLF
- D1, D2, D3, D4, D5: footprint (none) -> Diode_SMD:D_0805_2012Metric_Pad1.15x1.40mm_HandSolder
- F1: footprint 0_RoverFootprint:FUSE_3568-20 -> RoverFootprint:FUSE_3568-20
- JP1: footprint (none) -> Connector_PinHeader_2.54mm:PinHeader_1x03_P2.54mm_Vertical
- U4: value LDO-LM7805MPX/NOPB -> LDO-TLE4284DV33ATMA1
- U6: footprint 0_RoverFootprint:OCTAPACK_VN7004_STM-M -> RoverFootprint:OCTAPACK_VN7004_STM-M
Connections:
- no-connect marks 16 -> 12
Other:
- note removed: "Data input"

Commit message: PDB
Parts:
- added D6, D7, D8, D9: R, Diode_SMD:D_0805_2012Metric_Pad1.15x1.40mm_HandSolder, symbol Device:LED
- added F2, F3, F4, F5: 3A, RoverFootprint:FUSE_3568-20, symbol 0_RoverLibrary:FuseHolder
- added J2: ETH-CRJ036-5-TH, RoverFootprint:ETH-CRJ036-5-TH-2x4, symbol 0_RoverLibrary:ETH-CRJ036-5-TH
- added J3: TerminalBlock, RoverFootprint:TerminalBlock-4_P5.00mm-691137710004, symbol 0_RoverLibrary:TerminalBlock-4-691137710004
- added R10, R11, R13, R14, R15, R19, R20, R21, R22: 15k, Resistor_SMD:R_0805_2012Metric_Pad1.20x1.40mm_HandSolder, symbol Device:R
- added R12, R16, R17, R18, R23, R24, R25, R26: 1k, Resistor_SMD:R_0805_2012Metric_Pad1.20x1.40mm_HandSolder, symbol Device:R
- added U10, U7, U8, U9: HSS-VN7140ASTR, Package_SO:SOIC-8_3.9x4.9mm_P1.27mm, symbol 0_RoverLibrary:HSS-VN7140ASTR
Connections:
- net +24V_L: now also F2.1, F3.1, F4.1, F5.1
- net CANH: now also J2.1_1B (CANH), J2.1_1T (CANH), J2.2_1B (CANH), J2.2_1T (CANH), J2.3_1B (CANH), J2.3_1T (CANH), J2.4_1B (CANH), J2.4_1T (CANH), J3.1
- net CANL: now also J2.1_2B (CANL), J2.1_2T (CANL), J2.2_2B (CANL), J2.2_2T (CANL), J2.3_2B (CANL), J2.3_2T (CANL), J2.4_2B (CANL), J2.4_2T (CANL), J3.2
- net GND: now also D6.1 (K), D7.1 (K), D8.1 (K), D9.1 (K), J2.1_6B (GND), J2.1_6T (GND), J2.1_8B (GND), J2.1_8T (GND), J2.2_6B (GND), J2.2_6T (GND), J2.2_8B (GND), J2.2_8T (GND), J2.3_6B (GND), J2.3_6T (GND), J2.3_8B (GND), J2.3_8T (GND), J2.4_6B (GND), J2.4_6T (GND), J2.4_8B (GND), J2.4_8T (GND), J2.S1, J2.S2, J2.S3, J2.S4, J2.S5, J2.S6, J3.3, R10.2, R11.2, R12.2, R13.2, R14.2, R15.2, R16.2, R19.2, R20.2, R21.2, R22.2, R23.2, R24.2, U10.3 (GND), U7.3 (GND), U8.3 (GND), U9.3 (GND)
- net LOW_PW_EN: now also J3.4, R10.1
- new net: D6.2 (A), R17.2
- new net: R16.1, U8.4 (Multisense)
- new net: D8.2 (A), R25.2
- new net: R21.1, U9.2 (SEn)
- new net: D7.2 (A), R18.2
- new net: F4.2, U9.5 (Vcc), U9.8 (Vcc)
- new net: R24.1, U10.4 (Multisense)
- new net: D9.2 (A), R26.2
- new net: R23.1, U9.4 (Multisense)
- new net: R13.1, U7.2 (SEn)
- new net: F3.2, U8.5 (Vcc), U8.8 (Vcc)
- new net: R15.1, U8.2 (SEn)
- new net: R12.1, U7.4 (Multisense)
- new net: F2.2, U7.5 (Vcc), U7.8 (Vcc)
- new net: F5.2, U10.5 (Vcc), U10.8 (Vcc)
- new net: R22.1, U10.2 (SEn)
- new net +24V_OUT_1: J2.1_5T (Vcc), J2.1_7T (Vcc), R17.1, U7.6 (OUT), U7.7 (OUT)
- new net +24V_OUT_2: J2.2_5T (Vcc), J2.2_7T (Vcc), R18.1, U8.6 (OUT), U8.7 (OUT)
- new net +24V_OUT_3: J2.3_5T (Vcc), J2.3_7T (Vcc), R26.1, U9.6 (OUT), U9.7 (OUT)
- new net +24V_OUT_4: J2.4_5T (Vcc), J2.4_7T (Vcc), R25.1, U10.6 (OUT), U10.7 (OUT)
- new net SIGN_OUT_24_1: R11.1, U7.1 (INPUT)
- new net SIGN_OUT_24_2: R14.1, U8.1 (INPUT)
- new net SIGN_OUT_24_3: R19.1, U9.1 (INPUT)
- new net SIGN_OUT_24_4: R20.1, U10.1 (INPUT)
- no-connect marks 12 -> 28
Other:
- note added: "24V Outputs"
- note added: "Data Input"
- note added: "TODO: (X) LED Build_in (X) LDO + LED (X) CAN INPUT (X) Connect selector input (X) Power input ( ) 12V Switches ( ) 5V Switches (X) 24v Switches (X) Low power en signal (X) Big power relay ( ) Other"
- note removed: "TODO: (X) LED Build_in (X) LDO + LED (X) CAN INPUT ( ) Connect selector input (X) Power input ( ) 12V Switches ( ) 24v Switches ( ) Low power en signal ( ) Big power relay ( ) Other"
- moved on the sheet: C10, C8, C9, F1, JP1, R9, U4, U5, U6

Commit message: .
Parts:
- removed R21, R22: 15k, Resistor_SMD:R_0805_2012Metric_Pad1.20x1.40mm_HandSolder, symbol Device:R
- removed R23, R24: 1k, Resistor_SMD:R_0805_2012Metric_Pad1.20x1.40mm_HandSolder, symbol Device:R
- R12, R16: value 1k -> 15k
Connections:
- net SIGN_OUT_24_2: now also R12.1; no longer R14.1
- net SIGN_OUT_24_3: now also R15.1; no longer R19.1
- net SIGN_OUT_24_4: now also R19.1; no longer R20.1
- net at R16.1: now also U9.2 (SEn); no longer U8.4 (Multisense)
- net SIGN_SENSE_24_4: now reaches U10.4 (Multisense)
- net SIGN_SENSE_24_3: now reaches U9.4 (Multisense)
- net at U8.2 (SEn): now also R14.1; no longer R15.1
- net SIGN_SENSE_24_1: now reaches U7.4 (Multisense)
- net SIGN_SENSE_24_1: no longer R12.1
- net at U10.2 (SEn): now also R20.1
- new net SIGN_SENSE_24_2: U8.4 (Multisense)
Other:
- moved on the sheet: R13

Commit message: .
Parts:
- removed D6, D7, D8, D9: R, Diode_SMD:D_0805_2012Metric_Pad1.15x1.40mm_HandSolder, symbol Device:LED
- removed J2: ETH-CRJ036-5-TH, RoverFootprint:ETH-CRJ036-5-TH-2x4, symbol 0_RoverLibrary:ETH-CRJ036-5-TH
- removed R25, R26: 1k, Resistor_SMD:R_0805_2012Metric_Pad1.20x1.40mm_HandSolder, symbol Device:R
- added J2: ETH-RJHSE508104, RoverFootprint:ETH-RJHSE508104, symbol 0_RoverLibrary:ETH-RJHSE508104
- added R21, R22: 5.1k, Resistor_SMD:R_0805_2012Metric_Pad1.20x1.40mm_HandSolder, symbol Device:R
- R17, R18: value 1k -> 5.1k
Connections:
- net +24V_OUT_1: now also J2.1_10 (G_L+), J2.1_5 (Vcc), J2.1_7 (Vcc); no longer R17.1
- net +24V_OUT_2: now also J2.2_10 (G_L+), J2.2_5 (Vcc), J2.2_7 (Vcc); no longer R18.1
- net +24V_OUT_3: now also J2.3_10 (G_L+), J2.3_5 (Vcc), J2.3_7 (Vcc)
- net +24V_OUT_4: now also J2.4_10 (G_L+), J2.4_5 (Vcc), J2.4_7 (Vcc)
- net CANH: now also J2.1_1 (CANH), J2.2_1 (CANH), J2.3_1 (CANH), J2.4_1 (CANH)
- net CANL: now also J2.1_2 (CANL), J2.2_2 (CANL), J2.3_2 (CANL), J2.4_2 (CANL)
- net GND: now also R17.1, R18.1, J2.1_6 (GND), J2.1_8 (GND), J2.2_6 (GND), J2.2_8 (GND), J2.3_6 (GND), J2.3_8 (GND), J2.4_6 (GND), J2.4_8 (GND), R21.1, R22.1
- net at R17.2: now also J2.1_9 (G_L-)
- net at R18.2: now also J2.2_9 (G_L-)
- new net: J2.3_9 (G_L-), R21.2
- new net: J2.4_9 (G_L-), R22.2

Commit message: .
Parts:
- added F6: 8A, RoverFootprint:FUSE_3568-20, symbol 0_RoverLibrary:FuseHolder
- added F7: 7A, RoverFootprint:FUSE_3568-20, symbol 0_RoverLibrary:FuseHolder
- added F8, F9: 3A, RoverFootprint:FUSE_3568-20, symbol 0_RoverLibrary:FuseHolder
- added J4, J8: XT30PW-F, RoverFootprint:AMASS_XT30PW-F_1x02_P2.50mm_Horizontal, symbol 0_RoverLibrary:XT30PW-F
- added J5: XT30PW-M, RoverFootprint:AMASS_XT30PW-M_1x02_P2.50mm_Horizontal, symbol 0_RoverLibrary:XT30PW-M
- added J6, J7: ETH-RJHSE508102, RoverFootprint:ETH-RJHSE508102, symbol 0_RoverLibrary:ETH-RJHSE508102
- added R23, R24, R25, R26: 15k, Resistor_SMD:R_0805_2012Metric_Pad1.20x1.40mm_HandSolder, symbol Device:R
- added R27, R28, R29, R30: 5.1k, Resistor_SMD:R_0805_2012Metric_Pad1.20x1.40mm_HandSolder, symbol Device:R
- added U11, U12: HSS-VN7140ASTR, Package_SO:SOIC-8_3.9x4.9mm_P1.27mm, symbol 0_RoverLibrary:HSS-VN7140ASTR
Connections:
- net +12V: now also F6.1, F8.1, F9.1, J5.2 (+)
- net +24V_L: now also F7.1
- net CANH: now also J6.1_1 (CANH), J6.2_1 (CANH), J7.1_1 (CANH), J7.2_1 (CANH)
- net CANL: now also J6.1_2 (CANL), J6.2_2 (CANL), J7.1_2 (CANL), J7.2_2 (CANL)
- net GND: now also J4.1 (-), J5.1 (-), J6.1_6 (GND), J6.1_8 (GND), J6.2_6 (GND), J6.2_8 (GND), J7.1_6 (GND), J7.1_8 (GND), J7.2_6 (GND), J7.2_8 (GND), J8.1 (-), R23.2, R24.2, R25.2, R26.2, R27.1, R28.1, R29.1, R30.1, U11.3 (GND), U12.3 (GND)
- new net: R25.1, U11.2 (SEn)
- new net: F8.2, U11.5 (Vcc), U11.8 (Vcc)
- new net: F7.2, J4.2 (+)
- new net: R26.1, U12.2 (SEn)
- new net: F9.2, U12.5 (Vcc), U12.8 (Vcc)
- new net: J6.1_9 (G_L-), R27.2
- new net: J6.2_9 (G_L-), R28.2
- new net: F6.2, J8.2 (+)
- new net: J7.1_5 (Vcc), J7.1_7 (Vcc)
- new net: J7.1_9 (G_L-), R29.2
- new net: J7.2_5 (Vcc), J7.2_7 (Vcc)
- new net: J7.2_9 (G_L-), R30.2
- new net +12V_OUT_1: J6.1_10 (G_L+), J6.1_5 (Vcc), J6.1_7 (Vcc), U11.6 (OUT), U11.7 (OUT)
- new net +12V_OUT_2: J6.2_10 (G_L+), J6.2_5 (Vcc), J6.2_7 (Vcc), U12.6 (OUT), U12.7 (OUT)
- new net SIGN_OUT_12_1: R23.1, U11.1 (INPUT)
- new net SIGN_OUT_12_2: R24.1, U12.1 (INPUT)
- new net SIGN_SENSE_12_1: U11.4 (Multisense)
- new net SIGN_SENSE_12_2: U12.4 (Multisense)
- no-connect marks 28 -> 44
Other:
- note added: "12V HSS"
- note added: "12V Outputs"
- note added: "12V PC Power"
- note added: "12V Regulator"
- note added: "24V HSS"
- note added: "24V Output"
- note added: "5V Outputs"
- note added: "TODO: (X) LED Build_in (X) LDO + LED (X) CAN INPUT (X) Connect selector input (X) Power input (X) 12V Switches ( ) 5V Switches (X) 24v Switches (X) Low power en signal (X) Big power relay ( ) Other ( ) ETH Switch PW"
- note removed: "24V Outputs"
- note removed: "TODO: (X) LED Build_in (X) LDO + LED (X) CAN INPUT (X) Connect selector input (X) Power input ( ) 12V Switches ( ) 5V Switches (X) 24v Switches (X) Low power en signal (X) Big power relay ( ) Other"
- moved on the sheet: D1, D2, D3, J2, R17, R18, R21, R22, R4, R5, R6

Commit message: Start of PDB layout
Parts:
- removed H5: MountingHole_Pad, MountingHole:MountingHole_3.2mm_M3_DIN965_Pad_TopBottom, symbol RoverLibrary:MountingHole_Pad
- added F10, F11: 3A, RoverFootprint:FUSE_3568-20, symbol 0_RoverLibrary:FuseHolder
- added R31, R32, R33, R34: 15k, Resistor_SMD:R_0805_2012Metric_Pad1.20x1.40mm_HandSolder, symbol Device:R
- added U13, U14: HSS-VN7140ASTR, Package_SO:SOIC-8_3.9x4.9mm_P1.27mm, symbol 0_RoverLibrary:HSS-VN7140ASTR
- J1: footprint Connector_USB:USB_C_Receptacle_GCT_USB4105-xx-A_16P_TopMnt_Horizontal -> Connector_USB:USB_C_Receptacle_HRO_TYPE-C-31-M-12
Connections:
- net +24V_L: now also F10.1, F11.1
- net GND: now also R31.2, R32.2, R33.2, R34.2, U13.3 (GND), U14.3 (GND)
- net +24V_OUT_5: now reaches J7.1_10 (G_L+)
- net +24V_OUT_5: now also J7.1_5 (Vcc), J7.1_7 (Vcc), U13.6 (OUT), U13.7 (OUT)
- net +24V_OUT_6: now reaches J7.2_10 (G_L+)
- net +24V_OUT_6: now also J7.2_5 (Vcc), J7.2_7 (Vcc), U14.6 (OUT), U14.7 (OUT)
- new net: R34.1, U14.2 (SEn)
- new net: F11.2, U14.5 (Vcc), U14.8 (Vcc)
- new net: F10.2, U13.5 (Vcc), U13.8 (Vcc)
- new net: R33.1, U13.2 (SEn)
- new net SIGN_OUT_24_5: R31.1, U13.1 (INPUT)
- new net SIGN_OUT_24_6: R32.1, U14.1 (INPUT)
- new net SIGN_SENSE_24_5: U13.4 (Multisense)
- new net SIGN_SENSE_24_6: U14.4 (Multisense)
Other:
- note added: "TODO: (X) LED Build_in (X) LDO + LED (X) CAN INPUT (X) Connect selector input (X) Power input (X) 12V Switches (X) 24v Switches (X) Low power en signal (X) Big power relay"
- note removed: "TODO: (X) LED Build_in (X) LDO + LED (X) CAN INPUT (X) Connect selector input (X) Power input (X) 12V Switches ( ) 5V Switches (X) 24v Switches (X) Low power en signal (X) Big power relay ( ) Other ( ) ETH Switch PW"
- moved on the sheet: F8, F9, H6, H7, H8, R23, R24, R25, R26, U11, U12
