File: rover/2025/regulator/latest/regulator.kicad_pcb (KiCad board)
At the start: 4 copper layers, 46.4 x 32.6 mm, 31 parts, among them J1 ETH-RJHSE508102, J2 Conn_01x01_Pin, J3 Conn_01x01_Pin, J4 Conn_01x01_Pin, J5 Conn_01x01_Pin, J6 ETH-RJHSE5081, U1 DC_DC-AP64501

Commit message: .
Parts:
- turned F1 to 180 degrees
- turned F2 to 180 degrees
Connections:
- F1 pad 1: +24V -> Net-(JP1-B)
- F1 pad 2: Net-(JP1-B) -> +24V
- F2 pad 1: Net-(JP2-A) -> +V_{out}
- F2 pad 2: +V_{out} -> Net-(JP2-A)
