File: rover/2025/ARM-JL/latest/motor_driver.kicad_sch (KiCad schematic)
At the start: 14 parts, among them SW3 SW-PTS815SJM250SMTRLFS, SW4 SW-PTS815SJM250SMTRLFS, U7 IFX007TAUMA1, U8 IFX007TAUMA1, U9 XT60PM-F

Commit message: ARM-JL Drawing Done
Parts:
- removed U9: XT60PM-F, RoverFootprint:AMASS_XT60PW-F_1x02_P7.20mm_Horizontal, symbol RoverLibrary:XT60PW-F
- added J5: XT30PW-F, RoverFootprint:AMASS_XT30PW-F_1x02_P2.50mm_Horizontal, symbol RoverLibrary:XT30PW-F
- SW3, SW4: footprint (none) -> RoverFootprint:SW-PTS815 SJM250SMTRLFS
- U7, U8: footprint footprints:PG-TO263-7-1_INF-M -> Package_TO_SOT_SMD:TO-263-7_TabPin8
Connections:
- net M_OUT_A: now also J5.2 (+)
- net M_OUT_B: now also J5.1 (-)
Changed lines of the file:
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@@
 	(wire
 		(pts
-			(xy 158.75 82.55) (xy 168.91 82.55)
+			(xy 158.75 82.55) (xy 171.45 82.55)
 		)
 		(stroke
@@
 	(wire
 		(pts
-			(xy 158.75 80.01) (xy 168.91 80.01)
+			(xy 158.75 80.01) (xy 171.45 80.01)
 		)
 		(stroke
@@
 			)
 		)
-		(property "Footprint" ""
+		(property "Footprint" "RoverFootprint:SW-PTS815 SJM250SMTRLFS"
 			(at 40.64 110.49 0)
 			(effects
@@
 			)
 		)
-		(property "Footprint" "footprints:PG-TO263-7-1_INF-M"
+		(property "Footprint" "Package_TO_SOT_SMD:TO-263-7_TabPin8"
 			(at 71.12 11.43 0)
 			(effects
@@
 			)
 		)
-		(property "Footprint" "footprints:PG-TO263-7-1_INF-M"
+		(property "Footprint" "Package_TO_SOT_SMD:TO-263-7_TabPin8"
 			(at 157.48 11.43 0)
 			(effects
@@
 	)
 	(symbol
-		(lib_id "RoverLibrary:XT60PW-F")
-		(at 175.26 74.93 0)
-		(mirror y)
-		(unit 1)
-		(exclude_from_sim no)
-		(in_bom yes)
-		(on_board yes)
-		(dnp no)
-		(fields_autoplaced yes)
-		(property "Reference" "U9"
-			(at 180.34 80.0099 0)
-			(effects
-				(font
-					(size 1.27 1.27)
-				)
-				(justify right)
-			)
-		)
-		(property "Value" "XT60PM-F"
-			(at 180.34 82.5499 0)
-			(effects
-				(font
-					(size 1.27 1.27)
-				)
-				(justify right)
-			)
-		)
-		(property "Footprint" "RoverFootprint:AMASS_XT60PW-F_1x02_P7.20mm_Horizontal"
-			(at 175.26 86.868 0)
-			(effects
-				(font
-					(size 1.27 1.27)
-				)
-				(hide yes)
-			)
-		)
-		(property "Datasheet" ""
-			(at 175.26 74.93 0)
-			(effects
-				(font
-					(size 1.27 1.27)
-				)
-				(hide yes)
-			)
-		)
-		(property "Description" ""
-			(at 175.26 74.93 0)
-			(effects
-				(font
-					(size 1.27 1.27)
-				)
-				(hide yes)
-			)
-		)
-		(property "STATUS" "APPROVED"
-			(at 175.006 73.152 0)
-			(effects
-				(font
-					(size 1.27 1.27)
-				)
-				(hide yes)
-			)
-		)
-		(pin "2"
-		)
-		(pin "1"
-		)
-		(instances
-			(project ""
-				(path "/ea96555f-a650-48ef-b94f-b65180d69193/f8cb5055-73a1-4708-9add-8b73c04101c0/96acb7c0-97f3-4638-83e2-54e7d2feb040"
-					(reference "U9")
-					(unit 1)
-				)
-			)
-		)
-	)
-	(symbol
 		(lib_id "power:+24V")
 		(at 114.3 30.48 0)
@@
 	)
 	(symbol
+		(lib_id "RoverLibrary:XT30PW-F")
+		(at 173.99 80.01 0)
+		(mirror y)
+		(unit 1)
+		(exclude_from_sim no)
+		(in_bom yes)
+		(on_board yes)
+		(dnp no)
+		(fields_autoplaced yes)
+		(property "Reference" "J5"
+			(at 182.88 78.7399 0)
+			(effects
+				(font
+					(size 1.27 1.27)
+				)
+				(justify right)
+			)
+		)
+		(property "Value" "XT30PW-F"
+			(at 182.88 81.2799 0)
+			(effects
+				(font
+					(size 1.27 1.27)
+				)
+				(justify right)
+			)
+		)
+		(property "Footprint" "RoverFootprint:AMASS_XT30PW-F_1x02_P2.50mm_Horizontal"
+			(at 173.99 74.93 0)
+			(effects
+				(font
+					(size 1.27 1.27)
+				)
+				(justify bottom)
+				(hide yes)
+			)
+		)
+		(property "Datasheet" ""
+			(at 173.99 80.01 0)
+			(effects
+				(font
+					(size 1.27 1.27)
+				)
+				(hide yes)
+			)
+		)
+		(property "Description" ""
+			(at 173.99 80.01 0)
+			(effects
+				(font
+					(size 1.27 1.27)
+				)
+				(hide yes)
+			)
+		)
+		(property "MF" "amass"
+			(at 173.99 73.66 0)
+			(effects
+				(font
+					(size 1.27 1.27)
+				)
+				(justify bottom)
+				(hide yes)
+			)
+		)
+		(property "MAXIMUM_PACKAGE_HEIGHT" "5 mm"
+			(at 173.99 72.39 0)
+			(effects
+				(font
+					(size 1.27 1.27)
+				)
+				(justify bottom)
+				(hide yes)
+			)
+		)
+		(property "Package" "None"
+			(at 173.99 74.93 0)
+			(effects
+				(font
+					(size 1.27 1.27)
+				)
+				(justify bottom)
+				(hide yes)
+			)
+		)
+		(property "Price" "None"
+			(at 173.99 73.66 0)
+			(effects
+				(font
+					(size 1.27 1.27)
+				)
+				(justify bottom)
+				(hide yes)
+			)
+		)
+		(property "Check_prices" "https://www.snapeda.com/parts/XT30PW-F/AMASS/view-part/?ref=eda"
+			(at 173.99 72.39 0)
+			(effects
+				(font
+					(size 1.27 1.27)
+				)
+				(justify bottom)
+				(hide yes)
+			)
+		)
+		(property "STANDARD" "Manufacturer Recommendations"
+			(at 173.99 73.66 0)
+			(effects
+				(font
+					(size 1.27 1.27)
+				)
+				(justify bottom)
+				(hide yes)
+			)
+		)
+		(property "PARTREV" "1.2"
+			(at 173.99 73.66 0)
+			(effects
+				(font
+					(size 1.27 1.27)
+				)
+				(justify bottom)
+				(hide yes)
+			)
+		)
+		(property "SnapEDA_Link" "https://www.snapeda.com/parts/XT30PW-F/AMASS/view-part/?ref=snap"
+			(at 173.99 74.93 0)
+			(effects
+				(font
+					(size 1.27 1.27)
+				)
+				(justify bottom)
+				(hide yes)
+			)
+		)
+		(property "MP" "XT30PW-F"
+			(at 173.99 73.66 0)
+			(effects
+				(font
+					(size 1.27 1.27)
+				)
+				(justify bottom)
+				(hide yes)
+			)
+		)
+		(property "Description_1" "\nSocket; DC supply; XT30; female; PIN: 2; on PCBs; THT; yellow; 15A\n"
+			(at 173.99 72.39 0)
+			(effects
+				(font
+					(size 1.27 1.27)
+				)
+				(justify bottom)
+				(hide yes)
+			)
+		)
+		(property "MANUFACTURER" "Amass"
+			(at 173.99 73.66 0)
+			(effects
+				(font
+					(size 1.27 1.27)
+				)
+				(justify bottom)
+				(hide yes)
+			)
+		)
+		(property "Availability" "Not in stock"
+			(at 173.99 72.39 0)
+			(effects
+				(font
+					(size 1.27 1.27)
+				)
+				(justify bottom)
+				(hide yes)
+			)
+		)
+		(property "SNAPEDA_PN" "XT30PW-F"
+			(at 173.99 73.66 0)
+			(effects
+				(font
+					(size 1.27 1.27)
+				)
+				(justify bottom)
+				(hide yes)
+			)
+		)
+		(property "STATUS" "APPROVED"
+			(at 182.88 83.8199 0)
+			(effects
+				(font
+					(size 1.27 1.27)
+				)
+				(justify right)
+			)
+		)
+		(pin "1"
+		)
+		(pin "2"
+		)
+		(instances
+			(project ""
+				(path "/ea96555f-a650-48ef-b94f-b65180d69193/f8cb5055-73a1-4708-9add-8b73c04101c0/96acb7c0-97f3-4638-83e2-54e7d2feb040"
+					(reference "J5")
+					(unit 1)
+				)
+			)
+		)
+	)
+	(symbol
 		(lib_id "power:+3.3V")
 		(at 48.26 76.2 0)
@@
 			)
 		)
-		(property "Datasheet" "https://www.chemi-con.co.jp/products/relatedfiles/capacitor/catalog/HXJRA-e.PDF"
+		(property "Datasheet" "~"
 			(at 30.48 40.64 0)
 			(effects
@@
 			)
 		)
-		(property "Footprint" ""
+		(property "Footprint" "RoverFootprint:SW-PTS815 SJM250SMTRLFS"
 			(at 40.64 81.28 0)
 			(effects

Commit message: ARM-JL Routing in progress
Parts:
- U7, U8: footprint Package_TO_SOT_SMD:TO-263-7_TabPin8 -> Package_TO_SOT_SMD:TO-263-7_TabPin4
Connections:
- net M_OUT_A: no longer U7.8 (OUT)
- net M_OUT_B: no longer U8.8 (OUT)
Changed lines of the file:
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@@
-	)
-	(junction
-		(at 142.24 40.64)
-		(diameter 0)
-		(color 0 0 0 0)
 	)
 	(junction
@@
 	)
 	(junction
-		(at 86.36 40.64)
-		(diameter 0)
-		(color 0 0 0 0)
-	)
-	(junction
 		(at 128.27 40.64)
 		(diameter 0)
@@
 	(wire
 		(pts
-			(xy 142.24 38.1) (xy 142.24 40.64)
-		)
-		(stroke
-			(width 0)
-			(type default)
-		)
-	)
-	(wire
-		(pts
 			(xy 48.26 113.03) (xy 48.26 115.57)
 		)
@@
 		(pts
 			(xy 86.36 50.8) (xy 88.9 50.8)
-		)
-		(stroke
-			(width 0)
-			(type default)
-		)
-	)
-	(wire
-		(pts
-			(xy 86.36 38.1) (xy 86.36 40.64)
 		)
 		(stroke
@@
 			)
 		)
-		(property "Footprint" "Package_TO_SOT_SMD:TO-263-7_TabPin8"
+		(property "Footprint" "Package_TO_SOT_SMD:TO-263-7_TabPin4"
 			(at 71.12 11.43 0)
 			(effects
@@
 				)
 			)
-		)
-		(pin "8"
 		)
 		(pin "3"
@@
 			)
 		)
-		(property "Footprint" "Package_TO_SOT_SMD:TO-263-7_TabPin8"
+		(property "Footprint" "Package_TO_SOT_SMD:TO-263-7_TabPin4"
 			(at 157.48 11.43 0)
 			(effects
@@
 			)
 		)
-		(pin "8"
-		)
 		(pin "3"
