File: rover/2025/ARM-JL/latest/alims.kicad_sch (KiCad schematic)
At the start: 5 parts, among them U1 LDO-TLV74033PDBVR

Commit message: ARM-JL
Parts:
- added C10: 1uF, Capacitor_SMD:C_0805_2012Metric_Pad1.18x1.45mm_HandSolder, symbol RoverLibrary:C_0805
- added C11: 10nF, Capacitor_SMD:C_0805_2012Metric_Pad1.18x1.45mm_HandSolder, symbol RoverLibrary:C_0805
- added C12, C13: 10uF, Capacitor_SMD:C_0805_2012Metric_Pad1.18x1.45mm_HandSolder, symbol RoverLibrary:C_0805
- added JP1: Selector-Jumper_3_Open, Connector_PinHeader_2.54mm:PinHeader_1x03_P2.54mm_Vertical, symbol RoverLibrary:Selector-Jumper_3_Open
- added U2: LDO-LM7805MPX/NOPB, Package_TO_SOT_SMD:SOT-223-3_TabPin2, symbol RoverLibrary:LDO-LM7805MPX/NOPB
Connections:
- net +5V: now also C12.1, C13.1, U2.3 (OUTPUT)
- net GND: now also C10.2, C11.2, C12.2, C13.2, U2.2 (GND)
- new net +24V: C10.1, C11.1, JP1.2 (C), U2.1 (INPUT)
- new net +24V_H: JP1.1 (A)
- new net +24V_L: JP1.3 (B)
Other:
- note added: "3.3V LDO"
- note added: "<35V to 5V"
- note added: "Power Source Selection"
- moved on the sheet: C1, C2, C3, C4

Commit message: ARM-JL Drawing Done
Parts:
- removed JP1: Selector-Jumper_3_Open, Connector_PinHeader_2.54mm:PinHeader_1x03_P2.54mm_Vertical, symbol RoverLibrary:Selector-Jumper_3_Open
- added D3: 40V, Diode_SMD:D_SMA, symbol Device:D_Schottky
- added J4: Conn_02x03_Odd_Even, Connector_PinHeader_2.54mm:PinHeader_2x03_P2.54mm_Vertical_SMD, symbol Connector_Generic:Conn_02x03_Odd_Even
Connections:
- net +24V: now also J4.2 (Pin_2), J4.4 (Pin_4)
- net +24V_H: now also J4.1 (Pin_1)
- net +24V_L: now also J4.3 (Pin_3)
- net +5V: now also J4.6 (Pin_6)
- net NC: no longer names the net of U1.4 (NC)
- new net: D3.1 (K), J4.5 (Pin_5)
- new net +5V_USB: D3.2 (A)

Commit message: ARM-JL REV0 done
Parts:
- removed C2: 10nF, Capacitor_SMD:C_0805_2012Metric_Pad1.18x1.45mm_HandSolder, symbol RoverLibrary:C_0805
- removed C4: 10uF, Capacitor_SMD:C_0805_2012Metric_Pad1.18x1.45mm_HandSolder, symbol RoverLibrary:C_0805
- added D1: B, LED_SMD:LED_0805_2012Metric_Pad1.15x1.40mm_HandSolder, symbol RoverLibrary:LED
- added R6: 1k, Resistor_SMD:R_0805_2012Metric_Pad1.20x1.40mm_HandSolder, symbol RoverLibrary:R_0805
- C1: value 1uF -> 10uF
Connections:
- net +3.3V: now also D1.2 (A)
- net GND: now also R6.1
- new net: D1.1 (K), R6.2
Other:
- note added: "Power LED"
- moved on the sheet: C1, C3, U1
