File: rover/2025/ARM-JL/latest/board.kicad_sch (KiCad schematic)
At the start: 0 parts

Commit message: ARM-JL
Other:
- added sheet POTENC_connections (potenc_connections.kicad_sch)
- added sheet canbus (canbus.kicad_sch)
- added sheet motor_driver (motor_driver.kicad_sch)
Changed lines of the file:
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@@
 	)
 	(sheet
-		(at 27.94 43.18)
+		(at 25.4 45.72)
 		(size 21.59 3.81)
 		(fields_autoplaced yes)
@@
 		)
 		(property "Sheetname" "alims"
-			(at 27.94 42.4684 0)
+			(at 25.4 45.0084 0)
 			(effects
 				(font
@@
 		)
 		(property "Sheetfile" "alims.kicad_sch"
-			(at 27.94 47.5746 0)
+			(at 25.4 50.1146 0)
 			(effects
 				(font
@@
 	)
 	(sheet
-		(at 27.94 21.59)
+		(at 25.4 25.4)
 		(size 21.59 3.81)
 		(fields_autoplaced yes)
@@
 		)
 		(property "Sheetname" "external_connections"
-			(at 27.94 20.8784 0)
+			(at 25.4 24.6884 0)
 			(effects
 				(font
@@
 		)
 		(property "Sheetfile" "external_connections.kicad_sch"
-			(at 27.94 25.9846 0)
+			(at 25.4 29.7946 0)
+			(effects
+				(font
+					(size 1.27 1.27)
+				)
+				(justify left top)
+			)
+		)
+		(instances
+			(project "ARM-JL"
+				(path "/ea96555f-a650-48ef-b94f-b65180d69193/f8cb5055-73a1-4708-9add-8b73c04101c0"
+					(page "4")
+				)
+			)
+		)
+	)
+	(sheet
+		(at 25.4 76.2)
+		(size 21.59 3.81)
+		(fields_autoplaced yes)
+		(stroke
+			(width 0.1524)
+			(type solid)
+		)
+		(fill
+			(color 0 0 0 0.0000)
+		)
+		(property "Sheetname" "motor_driver"
+			(at 25.4 75.4884 0)
+			(effects
+				(font
+					(size 1.27 1.27)
+				)
+				(justify left bottom)
+			)
+		)
+		(property "Sheetfile" "motor_driver.kicad_sch"
+			(at 25.4 80.5946 0)
+			(effects
+				(font
+					(size 1.27 1.27)
+				)
+				(justify left top)
+			)
+		)
+		(instances
+			(project "ARM-JL"
+				(path "/ea96555f-a650-48ef-b94f-b65180d69193/f8cb5055-73a1-4708-9add-8b73c04101c0"
+					(page "8")
+				)
+			)
+		)
+	)
+	(sheet
+		(at 25.4 66.04)
+		(size 21.59 3.81)
+		(fields_autoplaced yes)
+		(stroke
+			(width 0.1524)
+			(type solid)
+		)
+		(fill
+			(color 0 0 0 0.0000)
+		)
+		(property "Sheetname" "POTENC_connections"
+			(at 25.4 65.3284 0)
+			(effects
+				(font
+					(size 1.27 1.27)
+				)
+				(justify left bottom)
+			)
+		)
+		(property "Sheetfile" "potenc_connections.kicad_sch"
+			(at 25.4 70.4346 0)
+			(effects
+				(font
+					(size 1.27 1.27)
+				)
+				(justify left top)
+			)
+		)
+		(instances
+			(project "ARM-JL"
+				(path "/ea96555f-a650-48ef-b94f-b65180d69193/f8cb5055-73a1-4708-9add-8b73c04101c0"
+					(page "7")
+				)
+			)
+		)
+	)
+	(sheet
+		(at 25.4 35.56)
+		(size 21.59 3.81)
+		(fields_autoplaced yes)
+		(stroke
+			(width 0.1524)
+			(type solid)
+		)
+		(fill
+			(color 0 0 0 0.0000)
+		)
+		(property "Sheetname" "esp32"
+			(at 25.4 34.8484 0)
+			(effects
+				(font
+					(size 1.27 1.27)
+				)
+				(justify left bottom)
+			)
+		)
+		(property "Sheetfile" "esp32.kicad_sch"
+			(at 25.4 39.9546 0)
 			(effects
 				(font
@@
 	)
 	(sheet
-		(at 27.94 33.02)
-		(size 21.59 3.81)
-		(fields_autoplaced yes)
-		(stroke
-			(width 0.1524)
-			(type solid)
-		)
-		(fill
-			(color 0 0 0 0.0000)
-		)
-		(property "Sheetname" "esp32"
-			(at 27.94 32.3084 0)
-			(effects
-				(font
-					(size 1.27 1.27)
-				)
-				(justify left bottom)
-			)
-		)
-		(property "Sheetfile" "esp32.kicad_sch"
-			(at 27.94 37.4146 0)
-			(effects
-				(font
-					(size 1.27 1.27)
-				)
-				(justify left top)
-			)
-		)
-		(instances
-			(project "ARM-JL"
-				(path "/ea96555f-a650-48ef-b94f-b65180d69193/f8cb5055-73a1-4708-9add-8b73c04101c0"
-					(page "4")
-				)
-			)
+		(at 25.4 55.88)
+		(size 21.59 3.81)
+		(fields_autoplaced yes)
+		(stroke
+			(width 0.1524)
+			(type solid)
+		)
+		(fill
+			(color 0 0 0 0.0000)
+		)
+		(property "Sheetname" "canbus"
+			(at 25.4 55.1684 0)
+			(effects
+				(font
+					(size 1.27 1.27)
+				)
+				(justify left bottom)
+			)
+		)
+		(property "Sheetfile" "canbus.kicad_sch"
+			(at 25.4 60.2746 0)
+			(effects
+				(font
+					(size 1.27 1.27)
+				)
+				(justify left top)
+			)
+		)
+		(instances
+			(project "ARM-JL"
+				(path "/ea96555f-a650-48ef-b94f-b65180d69193/f8cb5055-73a1-4708-9add-8b73c04101c0"
+					(page "6")
+				)
+			)

Commit message: ARM-JL Drawing Done
Parts:
- added H1, H2, H3: MountingHole_Pad, MountingHole:MountingHole_3.2mm_M3_DIN965_Pad_TopBottom, symbol RoverLibrary:MountingHole_Pad
Connections:
- new net GND: H1.1, H2.1, H3.1

Commit message: ARM-JL Routing in progress
Parts:
- removed H2: MountingHole_Pad, MountingHole:MountingHole_3.2mm_M3_DIN965_Pad_TopBottom, symbol RoverLibrary:MountingHole_Pad
Other:
- note added: "Connectors"
- note added: "Mecanical Parts"
- note added: "Ordering notes"
- note added: "Stackup: JLC04162-H-7628 4 Layers External: 2oz/ft²"
- note added: "TODO"
- moved on the sheet: H1, H3
Changed lines of the file:
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@@
 		(comment 1 "Made by Philippe Michaud")
+	)
+	(rectangle
+		(start 132.08 12.7)
+		(end 193.04 46.99)
+		(stroke
+			(width 0.254)
+			(type default)
+		)
+		(fill
+			(type none)
+		)
+	)
+	(rectangle
+		(start 69.85 48.26)
+		(end 130.81 82.55)
+		(stroke
+			(width 0.254)
+			(type default)
+		)
+		(fill
+			(type none)
+		)
+	)
+	(rectangle
+		(start 69.85 12.7)
+		(end 130.81 46.99)
+		(stroke
+			(width 0.254)
+			(type default)
+		)
+		(fill
+			(type none)
+		)
+	)
+	(text "TODO"
+		(exclude_from_sim no)
+		(at 100.076 64.516 0)
+		(effects
+			(font
+				(size 6.35 6.35)
+				(thickness 1.27)
+				(bold yes)
+			)
+		)
+	)
+	(text "Mecanical Parts"
+		(exclude_from_sim no)
+		(at 70.358 14.224 0)
+		(effects
+			(font
+				(size 1.27 1.27)
+			)
+			(justify left)
+		)
+	)
+	(text "Stackup:\n	JLC04162-H-7628 \n    4 Layers\n    External: 2oz/ft²"
+		(exclude_from_sim no)
+		(at 134.62 19.304 0)
+		(effects
+			(font
+				(size 1.27 1.27)
+				(thickness 0.1588)
+			)
+			(justify left)
+		)
+	)
+	(text "Connectors"
+		(exclude_from_sim no)
+		(at 70.358 49.784 0)
+		(effects
+			(font
+				(size 1.27 1.27)
+			)
+			(justify left)
+		)
+	)
+	(text "Ordering notes"
+		(exclude_from_sim no)
+		(at 132.588 14.224 0)
+		(effects
+			(font
+				(size 1.27 1.27)
+			)
+			(justify left)
+		)
 	)
 	(symbol
 		(lib_id "power:GND")
-		(at 76.2 48.26 0)
+		(at 81.28 38.1 0)
 		(unit 1)
 		(exclude_from_sim no)
@@
 		(dnp no)
 		(property "Reference" "#PWR050"
-			(at 76.2 54.61 0)
+			(at 81.28 44.45 0)
 			(effects
 				(font
@@
 		)
 		(property "Value" "GND"
-			(at 76.2 52.578 0)
+			(at 81.28 42.418 0)
 			(effects
 				(font
@@
 		)
 		(property "Footprint" ""
-			(at 76.2 48.26 0)
+			(at 81.28 38.1 0)
 			(effects
 				(font
@@
 		)
 		(property "Datasheet" ""
-			(at 76.2 48.26 0)
+			(at 81.28 38.1 0)
 			(effects
 				(font
@@
 		)
 		(property "Description" "Power symbol creates a global label with name \"GND\" , ground"
-			(at 76.2 48.26 0)
+			(at 81.28 38.1 0)
 			(effects
 				(font
@@
 	(symbol
 		(lib_id "RoverLibrary:MountingHole_Pad")
-		(at 76.2 20.32 0)
+		(at 81.28 21.59 0)
 		(unit 1)
 		(exclude_from_sim yes)
@@
 		(fields_autoplaced yes)
 		(property "Reference" "H1"
-			(at 78.74 17.7799 0)
+			(at 83.82 19.0499 0)
 			(effects
 				(font
@@
 		)
 		(property "Value" "MountingHole_Pad"
-			(at 78.74 20.3199 0)
+			(at 83.82 21.5899 0)
 			(effects
 				(font
@@
 		)
 		(property "Footprint" "MountingHole:MountingHole_3.2mm_M3_DIN965_Pad_TopBottom"
-			(at 76.2 20.32 0)
+			(at 81.28 21.59 0)
 			(effects
 				(font
@@
 		)
 		(property "Datasheet" "~"
-			(at 76.2 20.32 0)
+			(at 81.28 21.59 0)
 			(effects
 				(font
@@
 		)
 		(property "Description" "Mounting Hole with connection"
-			(at 76.2 20.32 0)
+			(at 81.28 21.59 0)
 			(effects
 				(font
@@
 	)
 	(symbol
-		(lib_id "RoverLibrary:MountingHole_Pad")
-		(at 76.2 33.02 0)
-		(unit 1)
-		(exclude_from_sim yes)
-		(in_bom no)
-		(on_board yes)
-		(dnp no)
-		(fields_autoplaced yes)
-		(property "Reference" "H2"
-			(at 78.74 30.4799 0)
-			(effects
-				(font
-					(size 1.27 1.27)
-				)
-				(justify left)
-			)
-		)
-		(property "Value" "MountingHole_Pad"
-			(at 78.74 33.0199 0)
-			(effects
-				(font
-					(size 1.27 1.27)
-				)
-				(justify left)
-			)
-		)
-		(property "Footprint" "MountingHole:MountingHole_3.2mm_M3_DIN965_Pad_TopBottom"
-			(at 76.2 33.02 0)
-			(effects
-				(font
-					(size 1.27 1.27)
-				)
-				(hide yes)
-			)
-		)
-		(property "Datasheet" "~"
-			(at 76.2 33.02 0)
-			(effects
-				(font
-					(size 1.27 1.27)
-				)
-				(hide yes)
-			)
-		)
-		(property "Description" "Mounting Hole with connection"
-			(at 76.2 33.02 0)
-			(effects
-				(font
-					(size 1.27 1.27)
-				)
-				(hide yes)
-			)
-		)
-		(pin "1"
-		)
-		(instances
-			(project "ARM-JL"
-				(path "/ea96555f-a650-48ef-b94f-b65180d69193/f8cb5055-73a1-4708-9add-8b73c04101c0"
-					(reference "H2")
-					(unit 1)
-				)
-			)
-		)
-	)
-	(symbol
 		(lib_id "power:GND")
-		(at 76.2 22.86 0)
+		(at 81.28 24.13 0)
 		(unit 1)
 		(exclude_from_sim no)
@@
 		(dnp no)
 		(property "Reference" "#PWR022"
-			(at 76.2 29.21 0)
+			(at 81.28 30.48 0)
 			(effects
 				(font
@@
 		)
 		(property "Value" "GND"
-			(at 76.2 26.924 0)
+			(at 81.28 28.194 0)
 			(effects
 				(font
@@
 		)
 		(property "Footprint" ""
-			(at 76.2 22.86 0)
+			(at 81.28 24.13 0)
 			(effects
 				(font
@@
 		)
 		(property "Datasheet" ""
-			(at 76.2 22.86 0)
+			(at 81.28 24.13 0)
 			(effects
 				(font
@@
 		)
 		(property "Description" "Power symbol creates a global label with name \"GND\" , ground"
-			(at 76.2 22.86 0)
+			(at 81.28 24.13 0)
 			(effects
 				(font
@@
 	(symbol
 		(lib_id "RoverLibrary:MountingHole_Pad")
-		(at 76.2 45.72 0)
+		(at 81.28 35.56 0)
 		(unit 1)
 		(exclude_from_sim yes)
@@
 		(fields_autoplaced yes)
 		(property "Reference" "H3"
-			(at 78.74 43.1799 0)
+			(at 83.82 33.0199 0)
 			(effects
 				(font
@@
 		)
 		(property "Value" "MountingHole_Pad"
-			(at 78.74 45.7199 0)
+			(at 83.82 35.5599 0)
 			(effects
 				(font
@@
 		)
 		(property "Footprint" "MountingHole:MountingHole_3.2mm_M3_DIN965_Pad_TopBottom"
-			(at 76.2 45.72 0)
+			(at 81.28 35.56 0)
 			(effects
 				(font
@@
 		)
 		(property "Datasheet" "~"
-			(at 76.2 45.72 0)
+			(at 81.28 35.56 0)
 			(effects
 				(font
@@
 		)
 		(property "Description" "Mounting Hole with connection"
-			(at 76.2 45.72 0)
+			(at 81.28 35.56 0)
 			(effects
 				(font
@@
 					(unit 1)
 				)
-			)
-		)
-	)
-	(symbol
-		(lib_id "power:GND")
-		(at 76.2 35.56 0)
-		(unit 1)
-		(exclude_from_sim no)
-		(in_bom yes)
-		(on_board yes)
-		(dnp no)
-		(property "Reference" "#PWR049"
-			(at 76.2 41.91 0)
-			(effects
-				(font
-					(size 1.27 1.27)
-				)
-				(hide yes)
-			)
-		)
-		(property "Value" "GND"
-			(at 76.2 39.624 0)
-			(effects
-				(font
-					(size 1.27 1.27)
-				)
-			)
-		)
-		(property "Footprint" ""
-			(at 76.2 35.56 0)
-			(effects
-				(font
-					(size 1.27 1.27)
-				)
-				(hide yes)
-			)
-		)
-		(property "Datasheet" ""
-			(at 76.2 35.56 0)
-			(effects
-				(font
-					(size 1.27 1.27)
-				)
-				(hide yes)
-			)
-		)
-		(property "Description" "Power symbol creates a global label with name \"GND\" , ground"
-			(at 76.2 35.56 0)
-			(effects
-				(font
-					(size 1.27 1.27)
-				)
-				(hide yes)
-			)
-		)
-		(pin "1"
-		)
-		(instances
-			(project "ARM-JL"
-				(path "/ea96555f-a650-48ef-b94f-b65180d69193/f8cb5055-73a1-4708-9add-8b73c04101c0"
-					(reference "#PWR049")
-					(unit 1)
-				)

Commit message: ARM-JL REV0 done
Other:
- moved on the sheet: H1, H3
Changed lines of the file:
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@@
 	)
 	(rectangle
-		(start 132.08 12.7)
-		(end 193.04 46.99)
+		(start 135.89 12.446)
+		(end 196.85 46.736)
 		(stroke
 			(width 0.254)
@@
 	)
 	(rectangle
-		(start 69.85 48.26)
-		(end 130.81 82.55)
+		(start 73.66 48.26)
+		(end 134.62 82.55)
 		(stroke
 			(width 0.254)
@@
 	)
 	(rectangle
-		(start 69.85 12.7)
-		(end 130.81 46.99)
+		(start 73.66 12.7)
+		(end 134.62 46.99)
 		(stroke
 			(width 0.254)
@@
 	(text "TODO"
 		(exclude_from_sim no)
-		(at 100.076 64.516 0)
+		(at 103.886 64.516 0)
 		(effects
 			(font
@@
 	(text "Mecanical Parts"
 		(exclude_from_sim no)
-		(at 70.358 14.224 0)
+		(at 74.168 14.224 0)
 		(effects
 			(font
@@
 		)
 	)
-	(text "Stackup:\n	JLC04162-H-7628 \n    4 Layers\n    External: 2oz/ft²"
-		(exclude_from_sim no)
-		(at 134.62 19.304 0)
+	(text "Stackup:\n    JLC04162-H-7628 \n    4 Layers\n    External: 2oz/ft²"
+		(exclude_from_sim no)
+		(at 138.43 19.05 0)
 		(effects
 			(font
@@
 	(text "Connectors"
 		(exclude_from_sim no)
-		(at 70.358 49.784 0)
+		(at 74.168 49.784 0)
 		(effects
 			(font
@@
 	(text "Ordering notes"
 		(exclude_from_sim no)
-		(at 132.588 14.224 0)
+		(at 136.398 13.97 0)
 		(effects
 			(font
@@
 	(symbol
 		(lib_id "power:GND")
-		(at 81.28 38.1 0)
+		(at 86.36 38.1 0)
 		(unit 1)
 		(exclude_from_sim no)
@@
 		(dnp no)
 		(property "Reference" "#PWR050"
-			(at 81.28 44.45 0)
+			(at 86.36 44.45 0)
 			(effects
 				(font
@@
 		)
 		(property "Value" "GND"
-			(at 81.28 42.418 0)
+			(at 86.36 42.418 0)
 			(effects
 				(font
@@
 		)
 		(property "Footprint" ""
-			(at 81.28 38.1 0)
+			(at 86.36 38.1 0)
 			(effects
 				(font
@@
 		)
 		(property "Datasheet" ""
-			(at 81.28 38.1 0)
+			(at 86.36 38.1 0)
 			(effects
 				(font
@@
 		)
 		(property "Description" "Power symbol creates a global label with name \"GND\" , ground"
-			(at 81.28 38.1 0)
+			(at 86.36 38.1 0)
 			(effects
 				(font
@@
 	(symbol
 		(lib_id "RoverLibrary:MountingHole_Pad")
-		(at 81.28 21.59 0)
+		(at 86.36 21.59 0)
 		(unit 1)
 		(exclude_from_sim yes)
@@
 		(fields_autoplaced yes)
 		(property "Reference" "H1"
-			(at 83.82 19.0499 0)
+			(at 88.9 19.0499 0)
 			(effects
 				(font
@@
 		)
 		(property "Value" "MountingHole_Pad"
-			(at 83.82 21.5899 0)
+			(at 88.9 21.5899 0)
 			(effects
 				(font
@@
 		)
 		(property "Footprint" "MountingHole:MountingHole_3.2mm_M3_DIN965_Pad_TopBottom"
-			(at 81.28 21.59 0)
+			(at 86.36 21.59 0)
 			(effects
 				(font
@@
 		)
 		(property "Datasheet" "~"
-			(at 81.28 21.59 0)
+			(at 86.36 21.59 0)
 			(effects
 				(font
@@
 		)
 		(property "Description" "Mounting Hole with connection"
-			(at 81.28 21.59 0)
+			(at 86.36 21.59 0)
 			(effects
 				(font
@@
 	(symbol
 		(lib_id "power:GND")
-		(at 81.28 24.13 0)
+		(at 86.36 24.13 0)
 		(unit 1)
 		(exclude_from_sim no)
@@
 		(dnp no)
 		(property "Reference" "#PWR022"
-			(at 81.28 30.48 0)
+			(at 86.36 30.48 0)
 			(effects
 				(font
@@
 		)
 		(property "Value" "GND"
-			(at 81.28 28.194 0)
+			(at 86.36 28.194 0)
 			(effects
 				(font
@@
 		)
 		(property "Footprint" ""
-			(at 81.28 24.13 0)
+			(at 86.36 24.13 0)
 			(effects
 				(font
@@
 		)
 		(property "Datasheet" ""
-			(at 81.28 24.13 0)
+			(at 86.36 24.13 0)
 			(effects
 				(font
@@
 		)
 		(property "Description" "Power symbol creates a global label with name \"GND\" , ground"
-			(at 81.28 24.13 0)
+			(at 86.36 24.13 0)
 			(effects
 				(font
@@
 	(symbol
 		(lib_id "RoverLibrary:MountingHole_Pad")
-		(at 81.28 35.56 0)
+		(at 86.36 35.56 0)
 		(unit 1)
 		(exclude_from_sim yes)
@@
 		(fields_autoplaced yes)
 		(property "Reference" "H3"
-			(at 83.82 33.0199 0)
+			(at 88.9 33.0199 0)
 			(effects
 				(font
@@
 		)
 		(property "Value" "MountingHole_Pad"
-			(at 83.82 35.5599 0)
+			(at 88.9 35.5599 0)
 			(effects
 				(font
@@
 		)
 		(property "Footprint" "MountingHole:MountingHole_3.2mm_M3_DIN965_Pad_TopBottom"
-			(at 81.28 35.56 0)
+			(at 86.36 35.56 0)
 			(effects
 				(font
@@
 		)
 		(property "Datasheet" "~"
-			(at 81.28 35.56 0)
+			(at 86.36 35.56 0)
 			(effects
 				(font
@@
 		)
 		(property "Description" "Mounting Hole with connection"
-			(at 81.28 35.56 0)
-			(effects
-				(font
+			(at 86.36 35.56 0)
+			(effects
+				(font
