File: rover/2025/drive_J2/drive_J2.kicad_sch (KiCad schematic)
At the start: 53 parts, among them J1 USB_C_USB4105-GF-A, J2 XT30PW-F, J3 Eth-Horiz, J4 Eth-Horiz, J5 Conn_01x03, J6 Conn_01x02, J7 Jumper PWR, J8 Conn_01x03, J9 Conn_01x06, SW1 TS09-63-25-WT-160-SMT-TR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

Commit message: Design review
Parts:
- removed C14: 220nF, Capacitor_SMD:C_0805_2012Metric_Pad1.18x1.45mm_HandSolder, symbol Rover_LIB:C_0805
- removed C7: 100nF, Capacitor_SMD:C_0805_2012Metric_Pad1.18x1.45mm_HandSolder, symbol Rover_LIB:C_0805
- removed D4: G, LED_SMD:LED_0805_2012Metric_Pad1.15x1.40mm_HandSolder, symbol Rover_LIB:LED
- removed J7: Jumper PWR, Connector_PinHeader_2.54mm:PinHeader_2x03_P2.54mm_Vertical, symbol Connector_Generic:Conn_02x03_Odd_Even
- removed R9: 1k, Resistor_SMD:R_0805_2012Metric_Pad1.20x1.40mm_HandSolder, symbol Rover_LIB:R_0805
- removed U5: LD1086DT33TR, Package_TO_SOT_SMD:TO-252-2, symbol Rover_LIB:LDO-LD1086DT33TR
- added C15: 220nF, Capacitor_SMD:C_0805_2012Metric_Pad1.18x1.45mm_HandSolder, symbol Rover_LIB:C_0805
- added C16: 100nF, Capacitor_SMD:C_0805_2012Metric_Pad1.18x1.45mm_HandSolder, symbol Rover_LIB:C_0805
- added D5: B, LED_SMD:LED_0805_2012Metric_Pad1.15x1.40mm_HandSolder, symbol Rover_LIB:LED
- added J10: Jumper PWR, Connector_PinHeader_2.54mm:PinHeader_2x03_P2.54mm_Vertical, symbol Connector_Generic:Conn_02x03_Odd_Even
- added R10: 121, Resistor_SMD:R_0805_2012Metric_Pad1.20x1.40mm_HandSolder, symbol Rover_LIB:R_0805
- added R11: 1k, Resistor_SMD:R_0805_2012Metric_Pad1.20x1.40mm_HandSolder, symbol Rover_LIB:R_0805
- added U5: LDO-TLV74033PDBVR, Package_TO_SOT_SMD:SOT-23-5_HandSoldering, symbol Rover_LIB:LDO-TLV74033PDBVR
Connections:
- net +24V_Logic: now also J10.3 (Pin_3)
- net +24V_safe: now also J10.1 (Pin_1)
- net +3.3V: now also U5.5 (OUTPUT)
- net +5V: now also C12.1, C6.1, C16.1, J10.6 (Pin_6), R11.1, U5.1 (INPUT), U5.3 (EN)
- net +5V_USB: now also J10.5 (Pin_5)
- net CANH: no longer U6.7 (CANH)
- net CANH_M: now also R10.1
- net CANL: no longer U6.6 (CANL)
- net CANL_M: now also R10.2
- net GND: now also C15.2, C16.2, D5.1 (K), U5.2 (GND)
- removed net IN_LDO: C12.1, C6.1, U8.1 (INPUT)
- new net: C15.1, J10.2 (Pin_2), J10.4 (Pin_4), U8.1 (INPUT)
- new net: D5.2 (A), R11.2
- new net CAN_N: U6.6 (CANL)
- new net CAN_P: U6.7 (CANH)
Other:
- note removed: "LDO 5V"
- moved on the sheet: C12, C13, C6, D1, J5, J6, R4
