File: rover/Templates/ProjectTemplate/latest/ProjectTemplate.kicad_pcb (KiCad board)
At the start: 4 copper layers, 0 parts

Commit message: Project Template
Parts:
- added G***: LOGO, LOGO, F.Cu at (53.6, 34.0)
Other:
- board outline added: 100 x 100 mm
- board text added: "${PROJECTNAME} REV${REVISION} by: ${AUTHOR} ${CURRENT_DATE} ${GROUP_NAME} ${TEAM}"
Changed lines of the file:
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@@
 		(pad_to_mask_clearance 0)
 		(allow_soldermask_bridges_in_footprints no)
+		(grid_origin 10 10)
 		(pcbplotparams
 			(layerselection 0x00010fc_ffffffff)
@@
 		)
 	)
+	(property "AUTHOR" "<ENTER_AUTOR_HERE>")
+	(property "GROUP_NAME" "Robotique UdeS")
+	(property "REVISION" "0")
+	(property "TEAM" "ROVUS")
 	(net 0 "")
+	(footprint "LOGO"
+		(layer "F.Cu")
+		(at 53.6 34)
+		(property "Reference" "G***"
+			(at 4.760877 0 0)
+			(layer "F.SilkS")
+			(hide yes)
+			(effects
+				(font
+					(size 1.5 1.5)
+					(thickness 0.3)
+				)
+			)
+		)
+		(property "Value" "LOGO"
+			(at 0.075 0 0)
+			(layer "F.SilkS")
+			(hide yes)
+			(effects
+				(font
+					(size 1.5 1.5)
+					(thickness 0.3)
+				)
+			)
+		)
+		(property "Footprint" ""
+			(at 0 0 0)
+			(layer "F.Fab")
+			(hide yes)
+			(effects
+				(font
+					(size 1.27 1.27)
+					(thickness 0.15)
+				)
+			)
+		)
+		(property "Datasheet" ""
+			(at 0 0 0)
+			(layer "F.Fab")
+			(hide yes)
+			(effects
+				(font
+					(size 1.27 1.27)
+					(thickness 0.15)
+				)
+			)
+		)
+		(property "Description" ""
+			(at 0 0 0)
+			(layer "F.Fab")
+			(hide yes)
+			(effects
+				(font
+					(size 1.27 1.27)
+					(thickness 0.15)
+				)
+			)
+		)
+		(attr board_only exclude_from_pos_files exclude_from_bom)
+		(fp_poly
+			(pts
+				(xy 1.298057 -3.637995) (xy 1.425261 -3.612722) (xy 1.492187 -3.586602) (xy 1.602181 -3.514285)
+				(xy 1.71546 -3.415129) (xy 1.814516 -3.306214) (xy 1.880018 -3.208249) (xy 1.912906 -3.119794) (xy 1.938892 -3.007096)
+				(xy 1.948988 -2.930127) (xy 1.954073 -2.857676) (xy 1.954784 -2.793493) (xy 1.94808 -2.733393) (xy 1.930923 -2.673185)
+				(xy 1.900274 -2.608682) (xy 1.853095 -2.535694) (xy 1.786345 -2.450034) (xy 1.696987 -2.347513)
+				(xy 1.581981 -2.223943) (xy 1.438288 -2.075135) (xy 1.262869 -1.8969) (xy 1.052686 -1.685051) (xy 1.026485 -1.658683)
+				(xy 0.186824 -0.813679) (xy 1.015998 0.016637) (xy 1.227304 0.228669) (xy 1.403509 0.406961) (xy 1.547994 0.55572)
+				(xy 1.664142 0.679146) (xy 1.755334 0.781444) (xy 1.824953 0.866816) (xy 1.876381 0.939465) (xy 1.913001 1.003595)
+				(xy 1.938194 1.06341) (xy 1.955342 1.123111) (xy 1.967829 1.186903) (xy 1.970417 1.202722) (xy 1.970599 1.336463)
+				(xy 1.942391 1.471787) (xy 1.932311 1.505012) (xy 1.920252 1.536834) (xy 1.903302 1.570447) (xy 1.878548 1.609041)
+				(xy 1.843078 1.655808) (xy 1.793978 1.71394) (xy 1.728335 1.786629) (xy 1.643238 1.877067) (xy 1.535773 1.988444)
+				(xy 1.403028 2.123954) (xy 1.242089 2.286787) (xy 1.050045 2.480136) (xy 0.823981 2.707192) (xy 0.71677 2.814799)
+				(xy 0.505538 3.026044) (xy 0.303298 3.226849) (xy 0.113639 3.413745) (xy -0.059851 3.583264) (xy -0.213584 3.731935)
+				(xy -0.34397 3.856291) (xy -0.44742 3.952862) (xy -0.520345 4.018178) (xy -0.559158 4.048771) (xy -0.560599 4.049572)
+				(xy -0.704681 4.099396) (xy -0.868574 4.116742) (xy -1.027243 4.099289) (xy -1.045482 4.094539)
+				(xy -1.239538 4.012966) (xy -1.405684 3.887373) (xy -1.537541 3.723306) (xy -1.593439 3.618005)
+				(xy -1.632804 3.488052) (xy -1.648845 3.339463) (xy -1.641305 3.193121) (xy -1.609928 3.069913)
+				(xy -1.600415 3.049185) (xy -1.571533 3.010487) (xy -1.508445 2.938163) (xy -1.415335 2.836628)
+				(xy -1.296385 2.710296) (xy -1.155777 2.563581) (xy -0.997693 2.400896) (xy -0.826317 2.226657)
+				(xy -0.710879 2.110403) (xy 0.130544 1.266195) (xy -0.712228 0.421573) (xy -0.94251 0.189687) (xy -1.135291 -0.006897)
+				(xy -1.292307 -0.17004) (xy -1.415291 -0.301604) (xy -1.505981 -0.403449) (xy -1.566109 -0.477438)
+				(xy -1.597412 -0.525431) (xy -1.599806 -0.530686) (xy -1.634135 -0.664107) (xy -1.642624 -0.820591)
+				(xy -1.625669 -0.975958) (xy -1.590592 -1.091264) (xy -1.568676 -1.127699) (xy -1.526315 -1.182365)
+				(xy -1.461323 -1.257555) (xy -1.37151 -1.355561) (xy -1.25469 -1.478677) (xy -1.108674 -1.629195)
+				(xy -0.931276 -1.809408) (xy -0.720306 -2.02161) (xy -0.473579 -2.268093) (xy -0.357885 -2.383265)
+				(xy -0.122601 -2.616442) (xy 0.096161 -2.831587) (xy 0.29558 -3.026009) (xy 0.472839 -3.197017)
+				(xy 0.625117 -3.341918) (xy 0.749595 -3.458022) (xy 0.843454 -3.542638) (xy 0.903872 -3.593073)
+				(xy 0.922858 -3.605788) (xy 1.02574 -3.635239) (xy 1.157845 -3.645738)
+			)
+			(stroke
+				(width 0)
+				(type solid)
+			)
+			(fill solid)
+			(layer "F.SilkS")
+		)
+	)
+	(gr_line
+		(start 30 30)
+		(end 130 30)
+		(stroke
+			(width 0.05)
+			(type default)
+		)
+		(layer "Edge.Cuts")
+	)
+	(gr_line
+		(start 30 30)
+		(end 30 130)
+		(stroke
+			(width 0.05)
+			(type default)
+		)
+		(layer "Edge.Cuts")
+	)
+	(gr_line
+		(start 30 130)
+		(end 130 130)
+		(stroke
+			(width 0.05)
+			(type default)
+		)
+		(layer "Edge.Cuts")
+	)
+	(gr_line
+		(start 130 30)
+		(end 130 130)
+		(stroke
+			(width 0.05)
+			(type default)
+		)
+		(layer "Edge.Cuts")
+	)
+	(gr_text "${PROJECTNAME} REV${REVISION}\nby: ${AUTHOR}\n${CURRENT_DATE}\n${GROUP_NAME}\n${TEAM}"
+		(at 30.4 38.2 0)
+		(layer "F.SilkS")
+		(effects
+			(font
+				(size 1 1)
+				(thickness 0.2)
+				(bold yes)
+			)
+			(justify left bottom)
+		)
+	)
 )
