File: rover/Templates/ProjectTemplate/latest/ProjectTemplate.kicad_sch (KiCad schematic)
At the start: 7 parts

Commit message: Project Template
Other:
- company: (none) -> ${GROUP_NAME}
- title: <SET_PROJECT_NAME> -> ${PROJECTNAME}
Changed lines of the file:
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@@
 	(paper "A5")
 	(title_block
-		(title "<SET_PROJECT_NAME>")
-		(date "2025-02-07")
-		(rev "0")
-		(comment 1 "<SET_AUTHOR_NAME>")
+		(title "${PROJECTNAME}")
+		(date "2025-02-08")
+		(rev "${REVISION}")
+		(company "${GROUP_NAME}")
+		(comment 1 "${AUTHOR}")
 	)
 	(bus
