File: rover/2025/Selector/Selector.kicad_sch (KiCad schematic)
At the start: 5 parts, among them J1 XT30PW-M, J2 JST3_Pin, J3 JST6_Pin, P1 PHR-2

Commit message: Reversed switch holder
Parts:
- added D1, D2: BZV55B3V3, Diode_SMD:D_MiniMELF, symbol Diode:BZV55B3V3
- added J4, J5: JST3_Pin, Connector_JST:JST_XH_B3B-XH-AM_1x03_P2.50mm_Vertical, symbol rover_lib:CONN-JST-XH-B3B
- added R1, R2: 300, Resistor_SMD:R_0603_1608Metric_Pad0.98x0.95mm_HandSolder, symbol rover_lib:R_0603
Connections:
- net +24V: now also F1.2; no longer F1.1
- net E_STOP_IN: now also F1.1; no longer F1.2
- net GND: now also D1.2 (A), D2.2 (A), J4.2, J5.2
- net POS1 & 2: now also R2.2
- net POS2: now also R1.2
- net E_STOP_OUT: no longer names the net of J2.1, P1.1
- new net: D1.1 (K), J5.3, R1.1
- new net: D2.1 (K), J4.3, R2.1
Other:
- note added: "À vérifier : Current drawn by 3.3V load"
- moved on the sheet: F1

Commit message: Selector changes
Parts:
- removed R1, R2: 300, Resistor_SMD:R_0603_1608Metric_Pad0.98x0.95mm_HandSolder, symbol rover_lib:R_0603
- added R1, R4: 20k, symbol Device:R
- added R2, R3: 100k, symbol Device:R
- J1: footprint RoverFootprint:AMASS_XT30PW-M_1x02_P2.50mm_Horizontal -> Connector_AMASS:AMASS_XT30PW-M_1x02_P2.50mm_Horizontal
- P1: footprint PHR-2:JST_PHR-2 -> Connector_JST:JST_EH_B2B-EH-A_1x02_P2.50mm_Vertical
Connections:
- net E_STOP_IN is gone; now on net +24V: F1.1, P1.2
- net +24V: no longer F1.2, J1.2 (+)
- net GND: now also R1.2, R4.2; no longer J4.2, J5.2
- net POS1 & 2: now also R2.1
- net POS2: now also R3.1
- net at D1.1 (K), J5.3: now also R1.1, R3.2
- net at D2.1 (K), J4.3: now also R2.2, R4.1
- new net: F1.2, J1.2 (+)
Other:
- note added: "diode 3.3V à 500mW"
- note added: "pas supposé avoir des resisatnce ici pour allumer les del ?"
- note removed: "À vérifier : Current drawn by 3.3V load"
- moved on the sheet: F1, J5

Commit message: selector layout
Parts:
- F1: footprint RoverFootprint:FUSE_3568-20 -> Rover:FuseHolder-3588-20
- R1, R2, R3, R4: footprint (none) -> Resistor_SMD:R_0603_1608Metric
Other:
- note removed: "diode 3.3V à 500mW"
- note removed: "pas supposé avoir des resisatnce ici pour allumer les del ?"
Changed lines of the file:
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@@
 		)
 	)
-	(text "pas supposé avoir des resisatnce ici pour allumer les del ? "
-		(exclude_from_sim no)
-		(at 39.878 203.454 0)
+	(label "E_STOP, SELECTOR AND DEL"
+		(at 20.32 106.68 0)
+		(fields_autoplaced yes)
+		(effects
+			(font
+				(size 2.54 2.54)
+			)
+			(justify left bottom)
+		)
+	)
+	(label "INPUT FROM BMS"
+		(at 27.94 22.86 0)
+		(fields_autoplaced yes)
+		(effects
+			(font
+				(size 2.54 2.54)
+			)
+			(justify left bottom)
+		)
+	)
+	(global_label "POS1 & 2"
+		(shape input)
+		(at 106.68 127 180)
+		(fields_autoplaced yes)
 		(effects
 			(font
 				(size 1.27 1.27)
 			)
-		)
-	)
-	(text "diode 3.3V à 500mW\n"
-		(exclude_from_sim no)
-		(at 128.27 50.8 0)
+			(justify right)
+		)
+		(property "Intersheetrefs" "${INTERSHEET_REFS}"
+			(at 93.9582 127 0)
+			(effects
+				(font
+					(size 1.27 1.27)
+				)
+				(justify right)
+				(hide yes)
+			)
+		)
+	)
+	(global_label "POS2"
+		(shape input)
+		(at 104.14 69.85 180)
+		(fields_autoplaced yes)
 		(effects
 			(font
 				(size 1.27 1.27)
 			)
-		)
-	)
-	(label "E_STOP, SELECTOR AND DEL"
-		(at 20.32 106.68 0)
-		(fields_autoplaced yes)
-		(effects
-			(font
-				(size 2.54 2.54)
-			)
-			(justify left bottom)
-		)
-	)
-	(label "INPUT FROM BMS"
-		(at 27.94 22.86 0)
-		(fields_autoplaced yes)
-		(effects
-			(font
-				(size 2.54 2.54)
-			)
-			(justify left bottom)
+			(justify right)
+		)
+		(property "Intersheetrefs" "${INTERSHEET_REFS}"
+			(at 96.1353 69.85 0)
+			(effects
+				(font
+					(size 1.27 1.27)
+				)
+				(justify right)
+				(hide yes)
+			)
 		)
 	)
 	(global_label "POS1 & 2"
 		(shape input)
-		(at 106.68 127 180)
+		(at 48.26 161.29 0)
 		(fields_autoplaced yes)
 		(effects
@@
 				(size 1.27 1.27)
 			)
-			(justify right)
+			(justify left)
 		)
 		(property "Intersheetrefs" "${INTERSHEET_REFS}"
-			(at 93.9582 127 0)
-			(effects
-				(font
-					(size 1.27 1.27)
-				)
-				(justify right)
+			(at 60.9818 161.29 0)
+			(effects
+				(font
+					(size 1.27 1.27)
+				)
+				(justify left)
 				(hide yes)
 			)
@@
 	(global_label "POS2"
 		(shape input)
-		(at 104.14 69.85 180)
+		(at 48.26 156.21 0)
 		(fields_autoplaced yes)
 		(effects
@@
 				(size 1.27 1.27)
 			)
-			(justify right)
-		)
-		(property "Intersheetrefs" "${INTERSHEET_REFS}"
-			(at 96.1353 69.85 0)
-			(effects
-				(font
-					(size 1.27 1.27)
-				)
-				(justify right)
-				(hide yes)
-			)
-		)
-	)
-	(global_label "POS1 & 2"
-		(shape input)
-		(at 48.26 161.29 0)
-		(fields_autoplaced yes)
-		(effects
-			(font
-				(size 1.27 1.27)
-			)
-			(justify left)
-		)
-		(property "Intersheetrefs" "${INTERSHEET_REFS}"
-			(at 60.9818 161.29 0)
-			(effects
-				(font
-					(size 1.27 1.27)
-				)
-				(justify left)
-				(hide yes)
-			)
-		)
-	)
-	(global_label "POS2"
-		(shape input)
-		(at 48.26 156.21 0)
-		(fields_autoplaced yes)
-		(effects
-			(font
-				(size 1.27 1.27)
-			)
 			(justify left)
 		)
@@
 			)
 		)
-		(property "Footprint" ""
+		(property "Footprint" "Resistor_SMD:R_0603_1608Metric"
 			(at 115.57 128.778 90)
 			(effects
@@
 			)
 		)
-		(property "Footprint" ""
+		(property "Footprint" "Resistor_SMD:R_0603_1608Metric"
 			(at 120.142 137.16 90)
 			(effects
@@
 			)
 		)
-		(property "Footprint" ""
+		(property "Footprint" "Resistor_SMD:R_0603_1608Metric"
 			(at 117.602 80.01 90)
 			(effects
@@
 			)
 		)
-		(property "Footprint" ""
+		(property "Footprint" "Resistor_SMD:R_0603_1608Metric"
 			(at 113.03 71.628 90)
 			(effects
@@
 			)
 		)
-		(property "Footprint" "RoverFootprint:FUSE_3568-20"
+		(property "Footprint" "Rover:FuseHolder-3588-20"
 			(at 41.148 59.69 90)
 			(effects

Commit message: selector layout
Changed lines of the file:
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@@
+		)
+	)
+	(label "LED_GREEN"
+		(at 41.91 170.18 0)
+		(fields_autoplaced yes)
+		(effects
+			(font
+				(size 1.27 1.27)
+			)
+			(justify left bottom)
 		)
 	)

Commit message: ARM-JL Drawing Done
Parts:
- added R5: k, Resistor_SMD:R_0805_2012Metric_Pad1.20x1.40mm_HandSolder, symbol rover_lib:R_0805
- F1: value FuseHolder -> 2A; footprint Rover:FuseHolder-3588-20 -> RoverFootprint:FUSE_3568-20
- J1: footprint Connector_AMASS:AMASS_XT30PW-M_1x02_P2.50mm_Horizontal -> RoverFootprint:AMASS_XT30PW-M_1x02_P2.50mm_Horizontal
Changed lines of the file:
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@@
 	(label "E_STOP, SELECTOR AND DEL"
 		(at 20.32 106.68 0)
-		(fields_autoplaced yes)
 		(effects
 			(font
@@
 	(label "LED_GREEN"
 		(at 41.91 170.18 0)
-		(fields_autoplaced yes)
 		(effects
 			(font
@@
 	(label "INPUT FROM BMS"
 		(at 27.94 22.86 0)
-		(fields_autoplaced yes)
 		(effects
 			(font
@@
 	)
 	(symbol
+		(lib_id "rover_lib:R_0805")
+		(at 111.76 137.16 0)
+		(unit 1)
+		(exclude_from_sim no)
+		(in_bom yes)
+		(on_board yes)
+		(dnp no)
+		(property "Reference" "R5"
+			(at 113.284 135.382 0)
+			(do_not_autoplace yes)
+			(effects
+				(font
+					(size 1.27 1.27)
+				)
+				(justify left)
+			)
+		)
+		(property "Value" "k"
+			(at 113.284 137.16 0)
+			(do_not_autoplace yes)
+			(effects
+				(font
+					(size 1.27 1.27)
+				)
+				(justify left)
+			)
+		)
+		(property "Footprint" "Resistor_SMD:R_0805_2012Metric_Pad1.20x1.40mm_HandSolder"
+			(at 104.14 137.16 90)
+			(effects
+				(font
+					(size 1.27 1.27)
+				)
+				(hide yes)
+			)
+		)
+		(property "Datasheet" ""
+			(at 111.76 137.16 90)
+			(do_not_autoplace yes)
+			(effects
+				(font
+					(size 1.27 1.27)
+				)
+				(hide yes)
+			)
+		)
+		(property "Description" "Resistor"
+			(at 111.76 148.59 0)
+			(effects
+				(font
+					(size 1.27 1.27)
+				)
+				(hide yes)
+			)
+		)
+		(property "Digikey" ""
+			(at 111.76 137.16 0)
+			(do_not_autoplace yes)
+			(effects
+				(font
+					(size 1.27 1.27)
+				)
+				(hide yes)
+			)
+		)
+		(property "Package" "0805"
+			(at 113.284 138.938 0)
+			(do_not_autoplace yes)
+			(effects
+				(font
+					(size 1.27 1.27)
+				)
+				(justify left)
+			)
+		)
+		(pin "1"
+		)
+		(pin "2"
+		)
+		(instances
+			(project ""
+				(path "/59a8ef21-cb28-4a01-85e5-f4611a966f3e"
+					(reference "R5")
+					(unit 1)
+				)
+			)
+		)
+	)
+	(symbol
 		(lib_id "Device:R")
 		(at 115.57 127 90)
@@
 		(on_board yes)
 		(dnp no)
-		(fields_autoplaced yes)
 		(property "Reference" "F1"
-			(at 41.91 57.1499 0)
+			(at 40.64 58.42 0)
 			(effects
 				(font
@@
 			)
 		)
-		(property "Value" "FuseHolder"
-			(at 41.91 59.6899 0)
+		(property "Value" "2A"
+			(at 40.64 60.96 0)
 			(effects
 				(font
@@
 			)
 		)
-		(property "Footprint" "Rover:FuseHolder-3588-20"
+		(property "Footprint" "RoverFootprint:FUSE_3568-20"
 			(at 41.148 59.69 90)
 			(effects
@@
 			)
 		)
-		(property "Description" "Fuse"
+		(property "Description" "Fuseholder through hole, 30A max"
 			(at 39.37 59.69 0)
 			(effects
@@
 				)
 				(justify right)
+				(hide yes)
 			)
 		)
@@
 			)
 		)
-		(property "Footprint" "Connector_AMASS:AMASS_XT30PW-M_1x02_P2.50mm_Horizontal"
+		(property "Footprint" "RoverFootprint:AMASS_XT30PW-M_1x02_P2.50mm_Horizontal"
 			(at 29.21 39.37 0)
 			(effects

Commit message: JST: Change JST 2 pin
Using the RoverLib One
Parts:
- removed P1: PHR-2, Connector_JST:JST_EH_B2B-EH-A_1x02_P2.50mm_Vertical, symbol Jst_2_pin:PHR-2
- added J6: JST2_Pin, RoverFootprint:2-pins-JST_XH_B2B-XH-A_1x02_P2.50mm_Vertical, symbol rover_lib:CONN-JST-XH-B2B
Connections:
- net +24V: now also J6.1
- net at J2.1: now also J6.2
Changed lines of the file:
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@@
-	(wire
-		(pts
-			(xy 39.37 128.27) (xy 37.084 128.27)
-		)
-		(stroke
-			(width 0)
-			(type default)
-		)
-	)
 	(wire
 		(pts
@@
 	(wire
 		(pts
+			(xy 31.75 132.08) (xy 50.8 132.08)
+		)
+		(stroke
+			(width 0)
+			(type default)
+		)
+	)
+	(wire
+		(pts
 			(xy 134.62 142.24) (xy 134.62 144.78)
 		)
@@
 	(wire
 		(pts
-			(xy 50.8 130.81) (xy 50.8 152.4)
+			(xy 50.8 132.08) (xy 50.8 152.4)
 		)
 		(stroke
@@
 	(wire
 		(pts
+			(xy 31.75 129.54) (xy 45.72 129.54)
+		)
+		(stroke
+			(width 0)
+			(type default)
+		)
+	)
+	(wire
+		(pts
 			(xy 31.75 152.4) (xy 50.8 152.4)
 		)
@@
 	(wire
 		(pts
-			(xy 39.37 125.73) (xy 45.72 125.73)
-		)
-		(stroke
-			(width 0)
-			(type default)
-		)
-	)
-	(wire
-		(pts
 			(xy 41.91 183.515) (xy 32.385 183.515)
 		)
@@
 	(wire
 		(pts
-			(xy 37.084 130.81) (xy 50.8 130.81)
-		)
-		(stroke
-			(width 0)
-			(type default)
-		)
-	)
-	(wire
-		(pts
 			(xy 53.34 49.53) (xy 53.34 50.8)
 		)
@@
 	(wire
 		(pts
-			(xy 39.37 125.73) (xy 39.37 128.27)
+			(xy 45.72 125.73) (xy 45.72 129.54)
 		)
 		(stroke
@@
 	(label "E_STOP, SELECTOR AND DEL"
 		(at 20.32 106.68 0)
+		(fields_autoplaced yes)
 		(effects
 			(font
@@
 	(label "LED_GREEN"
 		(at 41.91 170.18 0)
+		(fields_autoplaced yes)
 		(effects
 			(font
@@
 	(label "INPUT FROM BMS"
 		(at 27.94 22.86 0)
+		(fields_autoplaced yes)
 		(effects
 			(font
@@
 		)
 		(instances
-			(project ""
+			(project "Selector"
 				(path "/59a8ef21-cb28-4a01-85e5-f4611a966f3e"
 					(reference "R5")
@@
 	)
 	(symbol
-		(lib_id "Jst_2_pin:PHR-2")
-		(at 27.94 129.54 180)
-		(unit 1)
-		(exclude_from_sim no)
-		(in_bom yes)
-		(on_board yes)
-		(dnp no)
-		(fields_autoplaced yes)
-		(property "Reference" "P1"
-			(at 28.829 120.65 0)
-			(effects
-				(font
-					(size 1.27 1.27)
-				)
-			)
-		)
-		(property "Value" "PHR-2"
-			(at 28.829 123.19 0)
-			(effects
-				(font
-					(size 1.27 1.27)
-				)
-			)
-		)
-		(property "Footprint" "Connector_JST:JST_EH_B2B-EH-A_1x02_P2.50mm_Vertical"
-			(at 27.94 129.54 0)
-			(effects
-				(font
-					(size 1.27 1.27)
-				)
-				(justify bottom)
-				(hide yes)
-			)
-		)
-		(property "Datasheet" ""
-			(at 27.94 129.54 0)
-			(effects
-				(font
-					(size 1.27 1.27)
-				)
-				(hide yes)
-			)
-		)
-		(property "Description" ""
-			(at 27.94 129.54 0)
-			(effects
-				(font
-					(size 1.27 1.27)
-				)
-				(hide yes)
-			)
-		)
-		(property "MF" "JST Sales"
-			(at 27.94 129.54 0)
-			(effects
-				(font
-					(size 1.27 1.27)
-				)
-				(justify bottom)
-				(hide yes)
-			)
-		)
-		(property "Description_1" "\n                        \n                            2 Rectangular Connectors - Housings Receptacle Natural 0.079 (2.00mm)\n                        \n"
-			(at 27.94 129.54 0)
-			(effects
-				(font
-					(size 1.27 1.27)
-				)
-				(justify bottom)
-				(hide yes)
-			)
-		)
-		(property "Package" "Custom Package JST Sales"
-			(at 27.94 129.54 0)
-			(effects
-				(font
-					(size 1.27 1.27)
-				)
-				(justify bottom)
-				(hide yes)
-			)
-		)
-		(property "Price" "None"
-			(at 27.94 129.54 0)
-			(effects
-				(font
-					(size 1.27 1.27)
-				)
-				(justify bottom)
-				(hide yes)
-			)
-		)
-		(property "Check_prices" "https://www.snapeda.com/parts/PHR-2/JST/view-part/?ref=eda"
-			(at 27.94 129.54 0)
-			(effects
-				(font
-					(size 1.27 1.27)
-				)
-				(justify bottom)
-				(hide yes)
-			)
-		)
-		(property "SnapEDA_Link" "https://www.snapeda.com/parts/PHR-2/JST/view-part/?ref=snap"
-			(at 27.94 129.54 0)
-			(effects
-				(font
-					(size 1.27 1.27)
-				)
-				(justify bottom)
-				(hide yes)
-			)
-		)
-		(property "MP" "PHR-2"
-			(at 27.94 129.54 0)
-			(effects
-				(font
-					(size 1.27 1.27)
-				)
-				(justify bottom)
-				(hide yes)
-			)
-		)
-		(property "Availability" "In Stock"
-			(at 27.94 129.54 0)
-			(effects
-				(font
-					(size 1.27 1.27)
-				)
-				(justify bottom)
-				(hide yes)
-			)
-		)
-		(property "MANUFACTURER" "JST"
-			(at 27.94 129.54 0)
-			(effects
-				(font
-					(size 1.27 1.27)
-				)
-				(justify bottom)
-				(hide yes)
-			)
-		)
-		(pin "1"
-		)
-		(pin "2"
-		)
-		(instances
-			(project ""
-				(path "/59a8ef21-cb28-4a01-85e5-f4611a966f3e"
-					(reference "P1")
-					(unit 1)
-				)
-			)
-		)
-	)
-	(symbol
 		(lib_id "power:GND")
 		(at 45.72 187.96 0)
@@
 		)
 		(instances
-			(project ""
+			(project "Selector"
 				(path "/59a8ef21-cb28-4a01-85e5-f4611a966f3e"
 					(reference "#PWR04")
@@
 		)
 		(instances
-			(project ""
+			(project "Selector"
 				(path "/59a8ef21-cb28-4a01-85e5-f4611a966f3e"
 					(reference "J2")
@@
 		)
 		(instances
-			(project ""
+			(project "Selector"
 				(path "/59a8ef21-cb28-4a01-85e5-f4611a966f3e"
 					(reference "#PWR06")
@@
 		)
 		(instances
-			(project ""
+			(project "Selector"
 				(path "/59a8ef21-cb28-4a01-85e5-f4611a966f3e"
 					(reference "R1")
@@
 		)
 		(instances
-			(project ""
+			(project "Selector"
 				(path "/59a8ef21-cb28-4a01-85e5-f4611a966f3e"
 					(reference "#PWR02")
@@
 		)
 		(instances
-			(project ""
+			(project "Selector"
 				(path "/59a8ef21-cb28-4a01-85e5-f4611a966f3e"
 					(reference "D1")
@@
 	)
 	(symbol
+		(lib_id "rover_lib:CONN-JST-XH-B2B")
+		(at 28.575 126.365 0)
+		(unit 1)
+		(exclude_from_sim no)
+		(in_bom yes)
+		(on_board yes)
+		(dnp no)
+		(fields_autoplaced yes)
+		(property "Reference" "J6"
+			(at 27.94 123.19 0)
+			(effects
+				(font
+					(size 1.27 1.27)
+				)
+			)
+		)
+		(property "Value" "JST2_Pin"
+			(at 27.94 125.73 0)
+			(effects
+				(font
+					(size 1.27 1.27)
+				)
+			)
+		)
+		(property "Footprint" "RoverFootprint:2-pins-JST_XH_B2B-XH-A_1x02_P2.50mm_Vertical"
+			(at 28.575 126.365 0)
+			(effects
+				(font
+					(size 1.27 1.27)
+				)
+				(hide yes)
+			)
+		)
+		(property "Datasheet" ""
+			(at 28.575 126.365 0)
+			(effects
+				(font
+					(size 1.27 1.27)
+				)
+				(hide yes)
+			)
+		)
+		(property "Description" ""
+			(at 28.575 126.365 0)
+			(effects
+				(font
+					(size 1.27 1.27)
+				)
+				(hide yes)
+			)
+		)
+		(pin "2"
+		)
+		(pin "1"
+		)
+		(instances
+			(project "Selector"
+				(path "/59a8ef21-cb28-4a01-85e5-f4611a966f3e"
+					(reference "J6")
+					(unit 1)
+				)
+			)
+		)
+	)
+	(symbol
 		(lib_id "rover_lib:CONN-JST-XH-B6B")
 		(at 29.21 175.26 0)
@@
 		)
 		(instances
-			(project ""
+			(project "Selector"
 				(path "/59a8ef21-cb28-4a01-85e5-f4611a966f3e"
 					(reference "J3")
@@
 		)
 		(instances
-			(project ""
+			(project "Selector"
 				(path "/59a8ef21-cb28-4a01-85e5-f4611a966f3e"
 					(reference "#PWR03")
@@
 		)
 		(instances
-			(project ""
+			(project "Selector"
 				(path "/59a8ef21-cb28-4a01-85e5-f4611a966f3e"
 					(reference "F1")
@@
 		)
 		(instances
-			(project ""
+			(project "Selector"
 				(path "/59a8ef21-cb28-4a01-85e5-f4611a966f3e"
 					(reference "#PWR01")
@@
 		)
 		(instances
-			(project ""
+			(project "Selector"
 				(path "/59a8ef21-cb28-4a01-85e5-f4611a966f3e"
 					(reference "J1")

Commit message: small selector updates
Parts:
- removed D1, D2: BZV55B3V3, Diode_SMD:D_MiniMELF, symbol Diode:BZV55B3V3
- removed J2: JST3_Pin, Connector_JST:JST_XH_B3B-XH-AM_1x03_P2.50mm_Vertical, symbol rover_lib:CONN-JST-XH-B3B
- removed R5: k, Resistor_SMD:R_0805_2012Metric_Pad1.20x1.40mm_HandSolder, symbol rover_lib:R_0805
- added D1, D3: BZV55B5V6, Diode_SMD:D_MiniMELF, symbol Diode:BZV55B5V6
- added J2: JST4_Pin, Connector_JST:JST_XH_B4B-XH-A_1x04_P2.50mm_Vertical, symbol rover_lib:CONN-JST-XH-B4B
- R1, R2, R3, R4: footprint Resistor_SMD:R_0603_1608Metric -> Resistor_SMD:R_0805_2012Metric
Connections:
- net +24V: now also F1.2; no longer F1.1
- net GND: now also D1.2 (A), D3.2 (A)
- net POS1 & 2: now also J2.3
- net POS2: now also J2.2
- net at J4.3, R2.2, R4.1: now also D1.1 (K)
- net ESTOP TO SELECTOR: now reaches J6.2
- net ESTOP TO SELECTOR: now also J2.1
- net at J5.3, R1.1, R3.2: now also D3.1 (K)
- net at J1.2 (+): now also F1.1; no longer F1.2
Other:
- note added: "Voltage range of lipo 6s : 21 - 25 V Safety range of chip input voltage : 2.1 - 5.3 V Zener diode breakdown voltage : 5.6 V"
- moved on the sheet: F1, J3, J6

Commit message: Selector ready for update
Parts:
- removed J1: XT30PW-M, RoverFootprint:AMASS_XT30PW-M_1x02_P2.50mm_Horizontal, symbol rover_lib:XT30PW-M
- added H2, H3: MountingHole_Pad, MountingHole:MountingHole_3.2mm_M3_DIN965_Pad_TopBottom, symbol rover_lib:MountingHole_Pad
- added U1: XT60PW-M, RoverFootprint:AMASS_XT60PW-M_1x02_P7.20mm_Horizontal, symbol rover_lib:XT60PW-M
Connections:
- net GND: now also H2.1, H3.1, U1.1 (-)
- net at F1.1: now also U1.2 (+)
- net ESTOP TO SELECTOR: no longer names the net of J2.1, J6.2
Other:
- note added: "Voltage range of lipo 6s : 21 - 25 V Safety range of chip input voltage : 2.1 - 5.3 V Range obtained from voltage divider : 3.5 - 4.16 V Zener diode breakdown voltage : 5.6 V"
- note removed: "Voltage range of lipo 6s : 21 - 25 V Safety range of chip input voltage : 2.1 - 5.3 V Zener diode breakdown voltage : 5.6 V"
