File: rover/2025/DriveJ2/latest/drive_J2.kicad_sch (KiCad schematic)
At the start: 54 parts, among them J1 USB_C_USB4105-GF-A, J10 Jumper PWR, J2 XT30PW-F, J3 Eth-Horiz, J4 Eth-Horiz, J5 Conn_01x03, J6 Conn_01x02, J8 Conn_01x03, J9 Conn_01x06, SW1 TS09-63-25-WT-160-SMT-TR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

Commit message: Final changes on connector + cleaning directory
Parts:
- F1: PACKAGE (none) -> THT
- J8: footprint Connector_JST:JST_PH_S3B-PH-K_1x03_P2.00mm_Horizontal -> Connector_JST:JST_PH_B3B-PH-K_1x03_P2.00mm_Vertical
- J9: footprint Connector_JST:JST_PH_S6B-PH-K_1x06_P2.00mm_Horizontal -> Connector_JST:JST_PH_B6B-PH-K_1x06_P2.00mm_Vertical
- U2: STATUS TO BE VERIFIED -> APPROVED
Other:
- moved on the sheet: F1

Commit message: Upgraded version of DriveJ2
Parts:
- removed SW1, SW2, SW3, SW4: TS09-63-25-WT-160-SMT-TR, Button_Switch_SMD:SW_DIP_SPSTx01_Slide_6.7x4.1mm_W8.61mm_P2.54mm_LowProfile, symbol Rover_LIB:PushButton-TS09-63-25-WT-160-SMT-TR
- added C14, C7: 100nF, Capacitor_SMD:C_0805_2012Metric_Pad1.18x1.45mm_HandSolder, symbol Rover_LIB:C_0805
- added SW1, SW2, SW3, SW4: SW-PTS815SJM250SMTRLFS, RoverFootprint:SW-PTS815 SJM250SMTRLFS, symbol Rover_LIB:SW-PTS815SJM250SMTRLFS
Connections:
- net EN_PB: now also SW1.4
- net GND: now also C14.1, C7.1, SW1.1, SW1.2, SW2.1, SW2.2, SW3.1, SW3.2, SW4.1, SW4.2
- net GPIO_0: now also SW2.4
- net Jog+: now also U2.19 (IO11), C14.2, SW3.4; no longer U2.18 (IO10)
- net Jog-: now also U2.18 (IO10), C7.2, SW4.4; no longer U2.19 (IO11)
Other:
- moved on the sheet: R7, R8
