File: rover/2025/Regulator/latest/Regulator.kicad_sch (KiCad schematic)
At the start: 31 parts, among them J1 ETH-RJHSE508102, J2 Conn_01x01_Pin, J3 Conn_01x01_Pin, J4 Conn_01x01_Pin, J5 Conn_01x01_Pin, J6 ETH-RJHSE5081, U1 DC_DC-AP64501

Commit message: Last touch before order for ARMJL, Regulator and DDB + start of J345
Parts:
- R4, R5: value 5.1k -> 1k
Changed lines of the file:
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@@
 			)
 		)
-		(property "Value" "5.1k"
+		(property "Value" "1k"
 			(at 71.12 126.9999 0)
 			(effects
@@
 			)
 		)
-		(property "Value" "5.1k"
+		(property "Value" "1k"
 			(at 71.12 101.5999 0)
 			(effects

Commit message: Regulator Ready to order
Parts:
- C10: value 100uF -> (TBD)
- C11: value 100uF (Opt) -> (TBD)
- C9: value (Opt) -> (TBD)
- J2, J3, J4, J5: now left out of the parts list
- L1, R1, R3: value ~ -> (TBD)
- R4, R5: value 1k -> 5.1k
- R6: value 22.1k -> 5.1k
Changed lines of the file:
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@@
 			)
 		)
-		(property "Value" "(Opt)"
+		(property "Value" "(TBD)"
 			(at 125.984 64.77 0)
 			(effects
@@
 			)
 		)
-		(property "Value" "1k"
+		(property "Value" "5.1k"
 			(at 71.12 126.9999 0)
 			(effects
@@
 			)
 		)
-		(property "Value" "~"
+		(property "Value" "(TBD)"
 			(at 113.03 57.1499 0)
 			(effects
@@
 			)
 		)
-		(property "Value" "22.1k"
+		(property "Value" "5.1k"
 			(at 171.45 124.4599 0)
 			(effects
@@
 		(unit 1)
 		(exclude_from_sim no)
-		(in_bom yes)
+		(in_bom no)
 		(on_board yes)
 		(dnp no)
@@
 			)
 		)
-		(property "Value" "1k"
+		(property "Value" "5.1k"
 			(at 71.12 101.5999 0)
 			(effects
@@
 			)
 		)
-		(property "Value" "~"
+		(property "Value" "(TBD)"
 			(at 142.24 46.9899 0)
 			(effects
@@
 		(unit 1)
 		(exclude_from_sim no)
-		(in_bom yes)
+		(in_bom no)
 		(on_board yes)
 		(dnp no)
@@
 			)
 		)
-		(property "Value" "100uF (Opt)"
+		(property "Value" "(TBD)"
 			(at 54.864 39.37 0)
 			(effects
@@
 		(unit 1)
 		(exclude_from_sim no)
-		(in_bom yes)
+		(in_bom no)
 		(on_board yes)
 		(dnp no)
@@
 			)
 		)
-		(property "Value" "100uF"
+		(property "Value" "(TBD)"
 			(at 190.5 46.1009 0)
 			(effects
@@
 		(unit 1)
 		(exclude_from_sim no)
-		(in_bom yes)
+		(in_bom no)
 		(on_board yes)
 		(dnp no)
@@
 			)
 		)
-		(property "Value" "~"
-			(at 119.38 39.624 90)
+		(property "Value" "(TBD)"
+			(at 119.38 43.434 90)
 			(effects
 				(font

Commit message: PCBs ordered
Parts:
- removed C2: 22uF, Capacitor_SMD:C_0805_2012Metric_Pad1.18x1.45mm_HandSolder, symbol Device:C
- C1, C5, C6, C7: footprint Capacitor_SMD:C_0805_2012Metric_Pad1.18x1.45mm_HandSolder -> Capacitor_SMD:C_1210_3225Metric_Pad1.33x2.70mm_HandSolder
- C10, C11: value (TBD) -> 100uF
- R6: footprint Resistor_SMD:R_0805_2012Metric -> Resistor_SMD:R_0805_2012Metric_Pad1.20x1.40mm_HandSolder
Other:
- moved on the sheet: C10
Changed lines of the file:
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@@
 	)
 	(junction
+		(at 175.26 41.91)
+		(diameter 0)
+		(color 0 0 0 0)
+	)
+	(junction
 		(at 31.75 139.7)
 		(diameter 0)
@@
 	)
 	(junction
-		(at 186.69 41.91)
-		(diameter 0)
-		(color 0 0 0 0)
-	)
-	(junction
 		(at 152.4 67.31)
 		(diameter 0)
@@
 	)
 	(junction
-		(at 173.99 41.91)
-		(diameter 0)
-		(color 0 0 0 0)
-	)
-	(junction
-		(at 173.99 67.31)
-		(diameter 0)
-		(color 0 0 0 0)
-	)
-	(junction
 		(at 104.14 58.42)
 		(diameter 0)
@@
 	(wire
 		(pts
-			(xy 186.69 67.31) (xy 173.99 67.31)
-		)
-		(stroke
-			(width 0)
-			(type default)
-		)
-	)
-	(wire
-		(pts
 			(xy 78.74 41.91) (xy 81.28 41.91)
 		)
@@
 	(wire
 		(pts
-			(xy 186.69 49.53) (xy 186.69 67.31)
+			(xy 175.26 49.53) (xy 175.26 67.31)
 		)
 		(stroke
@@
 	(wire
 		(pts
-			(xy 68.58 41.91) (xy 68.58 34.29)
+			(xy 175.26 41.91) (xy 199.39 41.91)
 		)
 		(stroke
@@
 	(wire
 		(pts
-			(xy 16.51 93.98) (xy 25.4 93.98)
+			(xy 68.58 41.91) (xy 68.58 34.29)
 		)
 		(stroke
@@
 	(wire
 		(pts
-			(xy 52.07 67.31) (xy 68.58 67.31)
+			(xy 16.51 93.98) (xy 25.4 93.98)
 		)
 		(stroke
@@
 	(wire
 		(pts
-			(xy 130.81 41.91) (xy 127 41.91)
+			(xy 52.07 67.31) (xy 68.58 67.31)
 		)
 		(stroke
@@
 	(wire
 		(pts
-			(xy 104.14 67.31) (xy 110.49 67.31)
+			(xy 130.81 41.91) (xy 127 41.91)
 		)
 		(stroke
@@
 	(wire
 		(pts
-			(xy 128.27 109.22) (xy 135.89 109.22)
+			(xy 104.14 67.31) (xy 110.49 67.31)
 		)
 		(stroke
@@
 	(wire
 		(pts
-			(xy 163.83 41.91) (xy 173.99 41.91)
+			(xy 128.27 109.22) (xy 135.89 109.22)
 		)
 		(stroke
@@
 	(wire
 		(pts
-			(xy 186.69 41.91) (xy 199.39 41.91)
+			(xy 163.83 41.91) (xy 175.26 41.91)
 		)
 		(stroke
@@
 	(wire
 		(pts
-			(xy 173.99 41.91) (xy 186.69 41.91)
-		)
-		(stroke
-			(width 0)
-			(type default)
-		)
-	)
-	(wire
-		(pts
 			(xy 152.4 41.91) (xy 163.83 41.91)
 		)
@@
 	(wire
 		(pts
-			(xy 163.83 67.31) (xy 173.99 67.31)
-		)
-		(stroke
-			(width 0)
-			(type default)
-		)
-	)
-	(wire
-		(pts
-			(xy 173.99 67.31) (xy 173.99 49.53)
+			(xy 163.83 67.31) (xy 175.26 67.31)
 		)
 		(stroke
@@
 			)
 		)
-		(property "Datasheet" "~"
+		(property "Datasheet" "C9"
 			(at 123.19 63.5 0)
 			(effects
@@
 			)
 		)
-		(property "Datasheet" "~"
+		(property "Datasheet" "R3"
 			(at 110.49 55.88 0)
 			(effects
@@
 			)
 		)
-		(property "Footprint" "Resistor_SMD:R_0805_2012Metric"
+		(property "Footprint" "Resistor_SMD:R_0805_2012Metric_Pad1.20x1.40mm_HandSolder"
 			(at 167.132 123.19 90)
 			(effects
@@
 			)
 		)
-		(property "Footprint" "Capacitor_SMD:C_0805_2012Metric_Pad1.18x1.45mm_HandSolder"
+		(property "Footprint" "Capacitor_SMD:C_1210_3225Metric_Pad1.33x2.70mm_HandSolder"
 			(at 151.4348 41.91 0)
 			(effects
@@
 			)
 		)
-		(property "Datasheet" "~"
+		(property "Datasheet" "R1"
 			(at 139.7 45.72 0)
 			(effects
@@
 			)
 		)
-		(property "Footprint" "Capacitor_SMD:C_0805_2012Metric_Pad1.18x1.45mm_HandSolder"
+		(property "Footprint" "Capacitor_SMD:C_1210_3225Metric_Pad1.33x2.70mm_HandSolder"
 			(at 69.5452 41.91 0)
 			(effects
@@
 			)
 		)
-		(property "Footprint" "Capacitor_SMD:C_0805_2012Metric_Pad1.18x1.45mm_HandSolder"
+		(property "Footprint" "Capacitor_SMD:C_1210_3225Metric_Pad1.33x2.70mm_HandSolder"
 			(at 162.8648 41.91 0)
 			(effects
@@
 	)
 	(symbol
-		(lib_id "Device:C")
-		(at 173.99 45.72 180)
-		(unit 1)
-		(exclude_from_sim no)
-		(in_bom yes)
-		(on_board yes)
-		(dnp no)
-		(property "Reference" "C2"
-			(at 176.784 44.45 0)
-			(effects
-				(font
-					(size 1.27 1.27)
-				)
-				(justify right)
-			)
-		)
-		(property "Value" "22uF"
-			(at 176.784 46.99 0)
-			(effects
-				(font
-					(size 1.27 1.27)
-				)
-				(justify right)
-			)
-		)
-		(property "Footprint" "Capacitor_SMD:C_0805_2012Metric_Pad1.18x1.45mm_HandSolder"
-			(at 173.0248 41.91 0)
-			(effects
-				(font
-					(size 1.27 1.27)
-				)
-				(hide yes)
-			)
-		)
-		(property "Datasheet" "~"
-			(at 173.99 45.72 0)
-			(effects
-				(font
-					(size 1.27 1.27)
-				)
-				(hide yes)
-			)
-		)
-		(property "Description" "Unpolarized capacitor"
-			(at 173.99 45.72 0)
-			(effects
-				(font
-					(size 1.27 1.27)
-				)
-				(hide yes)
-			)
-		)
-		(pin "1"
-		)
-		(pin "2"
-		)
-		(instances
-			(project "regulator_5v"
-				(path "/fc17f381-1fc7-4ef2-b341-b694691f02ec"
-					(reference "C2")
-					(unit 1)
-				)
-			)
-		)
-	)
-	(symbol
 		(lib_id "power:GND")
 		(at 135.89 120.65 0)
@@
 			)
 		)
-		(property "Value" "(TBD)"
+		(property "Value" "100uF"
 			(at 54.864 39.37 0)
 			(effects
@@
 			)
 		)
-		(property "Datasheet" "~"
+		(property "Datasheet" ""
 			(at 52.07 38.1 0)
 			(effects
@@
 			)
 		)
-		(property "Footprint" "Capacitor_SMD:C_0805_2012Metric_Pad1.18x1.45mm_HandSolder"
+		(property "Footprint" "Capacitor_SMD:C_1210_3225Metric_Pad1.33x2.70mm_HandSolder"
 			(at 79.7052 41.91 0)
 			(effects
@@
 	(symbol
 		(lib_id "Device:C_Polarized")
-		(at 186.69 45.72 0)
+		(at 175.26 45.72 0)
 		(unit 1)
 		(exclude_from_sim no)
@@
 		(fields_autoplaced yes)
 		(property "Reference" "C10"
-			(at 190.5 43.5609 0)
+			(at 179.07 43.5609 0)
 			(effects
 				(font
@@
 			)
 		)
-		(property "Value" "(TBD)"
-			(at 190.5 46.1009 0)
+		(property "Value" "100uF"
+			(at 179.07 46.1009 0)
 			(effects
 				(font
@@
 		)
 		(property "Footprint" "Capacitor_SMD:CP_Elec_6.3x7.7"
-			(at 187.6552 49.53 0)
+			(at 176.2252 49.53 0)
 			(effects
 				(font
@@
 			)
 		)
-		(property "Datasheet" "~"
-			(at 186.69 45.72 0)
+		(property "Datasheet" ""
+			(at 175.26 45.72 0)
 			(effects
 				(font
@@
 		)
 		(property "Description" "Polarized capacitor"
-			(at 186.69 45.72 0)
+			(at 175.26 45.72 0)
 			(effects
 				(font
@@
 			)
 		)
-		(property "Datasheet" "~"
+		(property "Datasheet" "L1"
 			(at 119.38 41.91 0)
 			(effects
