File: rover/2025/ArmJ345/latest/aux.kicad_sch (KiCad schematic)
At the start: 20 parts, among them J11 Conn_01x04_MountingPin, J12 Conn_01x02_MountingPin, J13 Conn_01x02_MountingPin, J14 Conn_01x03_MountingPin, SW3 SW-PTS815SJM250SMTRLFS, SW4 SW-PTS815SJM250SMTRLFS, SW5 SW-PTS815SJM250SMTRLFS, SW6 SW-PTS815SJM250SMTRLFS, SW7 SW-PTS815SJM250SMTRLFS, SW8 SW-PTS815SJM250SMTRLFS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

Commit message: Layout armj345
Parts:
- removed J12: Conn_01x02_MountingPin, Connector_JST:JST_PH_S2B-PH-SM4-TB_1x02-1MP_P2.00mm_Horizontal, symbol Connector_Generic_MountingPin:Conn_01x02_MountingPin
- removed R20: 10k, Resistor_SMD:R_0805_2012Metric_Pad1.20x1.40mm_HandSolder, symbol RoverLibrary:R_0805
Connections:
- no-connect marks 4 -> 3
