File: rover/2025/CommBMS/latest/Board.kicad_sch (KiCad schematic)
At the start: 0 parts

Commit message: Comm_bms2
Parts:
- added C1, C10, C2, C4, C6: 100nF, Capacitor_SMD:C_0805_2012Metric_Pad1.18x1.45mm_HandSolder, symbol RoverLibrary:C_0805
- added C11: 1uF, Capacitor_SMD:C_0805_2012Metric_Pad1.18x1.45mm_HandSolder, symbol RoverLibrary:C_0805
- added C3, C5, C7: 10uF, Capacitor_SMD:C_0805_2012Metric_Pad1.18x1.45mm_HandSolder, symbol RoverLibrary:C_0805
- added C8, C9: 22uF, Capacitor_SMD:C_0805_2012Metric_Pad1.18x1.45mm_HandSolder, symbol RoverLibrary:C_0805
- added D1: R, LED_SMD:LED_0805_2012Metric_Pad1.15x1.40mm_HandSolder, symbol RoverLibrary:LED
- added D2: G, LED_SMD:LED_0805_2012Metric_Pad1.15x1.40mm_HandSolder, symbol Device:LED
- added J1, J2: Eth-Horiz-54601-908WPLF, RoverFootprint:Ethernet_Horizontal, symbol RoverLibrary:Eth-Horiz-54601-908WPLF
- added J3: USB_C_USB4105-GF-A, Connector_USB:USB_C_Receptacle_GCT_USB4105-xx-A_16P_TopMnt_Horizontal, symbol RoverLibrary:USB_C_USB4105-GF-A
- added J4: 39301080, RoverFootprint:Molex_Mini-Fit_Jr_5569-08A2_2x04_P4.20mm_Horizontal, symbol RoverLibrary:CONN-MOLEX_8PIN-39301080
- added R1, R2: 1k, Resistor_SMD:R_0805_2012Metric_Pad1.20x1.40mm_HandSolder, symbol RoverLibrary:R_0805
- added R3, R4: 5k1, Resistor_SMD:R_0805_2012Metric_Pad1.20x1.40mm_HandSolder, symbol RoverLibrary:R_0805
- added R5, R6: 0, Resistor_SMD:R_0805_2012Metric_Pad1.20x1.40mm_HandSolder, symbol RoverLibrary:R_0805
- added R7: 10k, Resistor_SMD:R_0805_2012Metric_Pad1.20x1.40mm_HandSolder, symbol RoverLibrary:R_0805
- added SW1, SW2: TS09-63-25-WT-160-SMT-TR, RoverFootprint:SW-PTS815 SJM250SMTRLFS, symbol RoverLibrary:SW-PTS815SJM250SMTRLFS
- added U1, U4: SN65HVD232Q, Package_SO:SOIC-8_3.9x4.9mm_P1.27mm, symbol RoverLibrary:CAN-Transceiver-SN65HVD232
- added U2: TVS, Package_SO:SOIC-8_3.9x4.9mm_P1.27mm, symbol RoverLibrary:TVS-SMDB03CE3/TR7TR-ND
- added U5: ESP32-S3-WROOM-1, RF_Module:ESP32-S3-WROOM-1U, symbol RoverLibrary:ESP32-S3-WROVER
- added U6: LDO-AZ1117CH2-3.3TRG1, Package_TO_SOT_SMD:SOT-223-3_TabPin2, symbol RoverLibrary:LDO-AZ1117CH2-3.3TRG1
- added U7: AXP1T34, Package_TO_SOT_SMD:SOT-353_SC-70-5, symbol RoverLibrary:Level_shifter-AXP1T34
Connections:
- new net: J1.3, J2.3
- new net: J1.4, J2.4
- new net: D1.2 (A), R1.1
- new net: R5.2, U7.1 (Vcci)
- new net: J3.A5 (CC1), R3.1
- new net: J3.B5 (CC2), R4.1
- new net: D2.2 (A), R2.1
- new net: R6.2, U7.2 (INPUT)
- new net +3.3V: C10.1, C3.1, C4.1, C5.1, C6.1, C8.1, C9.1, R2.2, R7.1, U1.3 (VCC), U4.3 (VCC), U5.2 (3V3), U6.3 (OUTPUT), U7.5 (Vcco)
- new net +5V_USB: C7.1, J3.A4 (VBUS), J3.A9 (VBUS), J3.B4 (VBUS), J3.B9 (VBUS), R5.1, U2.3, U6.1 (INPUT)
- new net 5V_USB: J1.5, J1.7, J2.5, J2.7
- new net CANH: J1.1 (CANH), J2.1 (CANH), U1.7 (CANH)
- new net CANH_B: J4.1, U4.7 (CANH)
- new net CANL: J1.2 (CANL), J2.2 (CANL), U1.6 (CANL)
- new net CANL_B: J4.2, U4.6 (CANL)
- new net EN_PB: C1.2, C11.1, R7.2, SW1.4, U5.3 (EN)
- new net GND: C1.1, C10.2, C11.2, C2.1, C3.2, C4.2, C5.2, C6.2, C7.2, C8.2, C9.2, D1.1 (K), D2.1 (K), J1.6, J1.8, J2.6, J2.8, J3.A1 (GND), J3.A12 (GND), J3.B1 (GND), J3.B12 (GND), J3.S1 (SHIELD), J4.7, R3.2, R4.2, SW1.1, SW1.2, SW2.1, SW2.2, U1.2 (GND), U1.8 (S), U2.5, U2.6, U2.7, U2.8, U4.2 (GND), U4.8 (S), U5.1 (GND), U5.40 (GND), U5.41 (GND), U6.2 (GND), U7.3 (GND)
- new net GPIO_0: C2.2, SW2.4, U5.27 (IO0-BOOT)
- new net LED_BUILDIN: R1.2, U5.5 (IO5)
- new net PWM_3V: U5.33 (IO40), U7.4 (OUTPUT)
- new net PWM_5V: J4.6, R6.1
- new net PWM_EN: J4.8, U5.34 (IO41)
- new net RXB: U4.4 (RXD), U5.36 (RXD0)
- new net RXC: U1.4 (RXD), U5.24 (IO47)
- new net TXB: U4.1 (TXD), U5.37 (TXD0)
- new net TXC: U1.1 (TXD), U5.25 (IO48)
- new net USB_N: J3.A7 (D-), J3.B7 (D-), U2.2, U5.13 (IO19-USB_N)
- new net USB_P: J3.A6 (D+), J3.B6 (D+), U2.1, U5.14 (IO20-USB-P)
- no-connect marks 0 -> 34
Other:
- note added: "BMS CAN Transceiver"
- note added: "BMS Connector"
- note added: "Boot ESP32 Button"
- note added: "CAN Transceiver"
- note added: "Data Connectors"
- note added: "ESP LDO"
- note added: "ESP32"
- note added: "Enable ESP32 Button"
- note added: "LED Build In"
- note added: "PWM LEVEL DOWN"
- note added: "USB Port ESP32"

Commit message: Little update
Connections:
- net USB_N: now also U2.1; no longer U2.2
- net USB_P: now also U2.2; no longer U2.1
Changed lines of the file:
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@@
-	)
-	(junction
-		(at 68.58 80.01)
-		(diameter 0)
-		(color 0 0 0 0)
 	)
 	(junction
@@
 	)
 	(junction
+		(at 68.58 74.93)
+		(diameter 0)
+		(color 0 0 0 0)
+	)
+	(junction
 		(at 52.07 74.93)
 		(diameter 0)
@@
 	)
 	(junction
+		(at 66.04 80.01)
+		(diameter 0)
+		(color 0 0 0 0)
+	)
+	(junction
 		(at 76.2 36.83)
 		(diameter 0)
@@
 	)
 	(junction
-		(at 66.04 74.93)
-		(diameter 0)
-		(color 0 0 0 0)
-	)
-	(junction
 		(at 43.18 26.67)
 		(diameter 0)
@@
 	(wire
 		(pts
-			(xy 66.04 74.93) (xy 76.2 74.93)
+			(xy 52.07 74.93) (xy 68.58 74.93)
 		)
 		(stroke
@@
 	(wire
 		(pts
+			(xy 66.04 80.01) (xy 66.04 81.28)
+		)
+		(stroke
+			(width 0)
+			(type default)
+		)
+	)
+	(wire
+		(pts
 			(xy 87.63 59.69) (xy 91.44 59.69)
 		)
@@
 	(wire
 		(pts
+			(xy 66.04 80.01) (xy 76.2 80.01)
+		)
+		(stroke
+			(width 0)
+			(type default)
+		)
+	)
+	(wire
+		(pts
 			(xy 49.53 74.93) (xy 52.07 74.93)
 		)
@@
 	(wire
 		(pts
-			(xy 66.04 74.93) (xy 66.04 81.28)
-		)
-		(stroke
-			(width 0)
-			(type default)
-		)
-	)
-	(wire
-		(pts
 			(xy 26.67 100.33) (xy 34.29 100.33)
 		)
@@
 	(wire
 		(pts
-			(xy 68.58 80.01) (xy 68.58 81.28)
-		)
-		(stroke
-			(width 0)
-			(type default)
-		)
-	)
-	(wire
-		(pts
 			(xy 41.91 193.04) (xy 46.99 193.04)
 		)
@@
 	(wire
 		(pts
+			(xy 68.58 74.93) (xy 68.58 81.28)
+		)
+		(stroke
+			(width 0)
+			(type default)
+		)
+	)
+	(wire
+		(pts
 			(xy 26.67 97.79) (xy 26.67 100.33)
 		)
@@
 	(wire
 		(pts
-			(xy 68.58 80.01) (xy 76.2 80.01)
-		)
-		(stroke
-			(width 0)
-			(type default)
-		)
-	)
-	(wire
-		(pts
 			(xy 219.71 198.12) (xy 219.71 199.39)
 		)
@@
 	(wire
 		(pts
-			(xy 52.07 74.93) (xy 66.04 74.93)
-		)
-		(stroke
-			(width 0)
-			(type default)
-		)
-	)
-	(wire
-		(pts
 			(xy 240.03 179.07) (xy 240.03 182.88)
 		)
@@
 	(wire
 		(pts
-			(xy 52.07 80.01) (xy 68.58 80.01)
+			(xy 52.07 80.01) (xy 66.04 80.01)
 		)
 		(stroke
@@
 		)
 		(stroke
+			(width 0)
+			(type default)
+		)
+	)
+	(wire
+		(pts
+			(xy 68.58 74.93) (xy 76.2 74.93)
+		)
+		(stroke

Commit message: ouep
Parts:
- removed R5, R6: 0, Resistor_SMD:R_0805_2012Metric_Pad1.20x1.40mm_HandSolder, symbol RoverLibrary:R_0805
- removed U4: SN65HVD232Q, Package_SO:SOIC-8_3.9x4.9mm_P1.27mm, symbol RoverLibrary:CAN-Transceiver-SN65HVD232
- added C12: 1n, Capacitor_SMD:C_0805_2012Metric_Pad1.18x1.45mm_HandSolder, symbol RoverLibrary:C_0805
- added C13, C14: 100nF, Capacitor_SMD:C_0805_2012Metric_Pad1.18x1.45mm_HandSolder, symbol RoverLibrary:C_0805
- added D3: CVJ10F30, DiodeSchott:UFV_TOS-L, symbol RoverLibrary:Diode_Schottchy_CVJ10F30
- added R5, R6: 0, Resistor_SMD:R_0603_1608Metric_Pad0.98x0.95mm_HandSolder, symbol RoverLibrary:R_0603
- added U3: LDO-LM7805MPX/NOPB, Package_TO_SOT_SMD:TO-263-3_TabPin2, symbol RoverLibrary:LDO-LM340SX-5.0/NOPB
- added U4: SP3485EN, Package_SO:SOIC-8_3.9x4.9mm_P1.27mm, symbol RoverLibrary:RS485_Transceiver-SP3485EN
- C8, C9: value 22uF -> 10uF
Connections:
- net +3.3V: now also U4.8 (VCC)
- net +5V_USB: now also D3.3; no longer C7.1, U6.1 (INPUT)
- net GND: now also U2.4, C12.2, C13.2, C14.2, U3.2 (GND), U4.5 (GND); no longer J3.S1 (SHIELD)
- net LED_BUILDIN: now also U5.39 (IO1); no longer U5.5 (IO5)
- net PWM_3V: now also U5.11 (IO18); no longer U5.33 (IO40)
- net PWM_5V: now also R6.1
- net PWM_EN: now also U5.10 (IO17); no longer U5.34 (IO41)
- net RXB: now also U5.18 (IO10), U4.1 (RXD); no longer U5.36 (RXD0)
- net RXC: now also U5.25 (IO48); no longer U5.24 (IO47)
- net TXB: now also U5.17 (IO9), U4.4 (TXD); no longer U5.37 (TXD0)
- net TXC: now also U5.24 (IO47); no longer U5.25 (IO48)
- net at J2.3: no longer J1.3
- net at J2.4: no longer J1.4
- net at U7.1 (Vcci): now also R5.2
- net at U7.2 (INPUT): now also R6.2
- net RE: now reaches U5.19 (IO11)
- net RE: now also U4.2 (RE)
- net DE: now reaches U5.20 (IO12)
- net DE: now also U4.3 (DE)
- net 5V_USB renamed +24V_ETH
- net +24V_ETH: now also C13.1, U3.1 (INPUT)
- net CANH_B renamed BMS_A
- net BMS_A: now also U4.6 (A)
- net CANL_B renamed BMS_B
- net BMS_B: now also U4.7 (B)
- new net: C12.1, J3.S1 (SHIELD)
- new net: C14.1, D3.1, U3.3 (OUTPUT)
- new net +5V: C7.1, D3.4, D3.5, R5.1, U6.1 (INPUT)
- no-connect marks 34 -> 35
Other:
- note added: "Eth connector"
- note added: "RS485 Transceiver"
- note removed: "BMS CAN Transceiver"
- note removed: "Data Connectors"
- moved on the sheet: C7, C8, D2, J1, J2, J4, R2, U2, U7

Commit message: commBMS modif
Parts:
- removed C13, C14: 100nF, Capacitor_SMD:C_0805_2012Metric_Pad1.18x1.45mm_HandSolder, symbol RoverLibrary:C_0805
- removed U3: LDO-LM7805MPX/NOPB, Package_TO_SOT_SMD:TO-263-3_TabPin2, symbol RoverLibrary:LDO-LM340SX-5.0/NOPB
- removed U6: LDO-AZ1117CH2-3.3TRG1, Package_TO_SOT_SMD:SOT-223-3_TabPin2, symbol RoverLibrary:LDO-AZ1117CH2-3.3TRG1
- added U3: LDO-LM7805MPX/NOPB, Package_TO_SOT_SMD:TO-263-3_TabPin2, symbol RoverLibrary:LDO-LM1084ISX-3.3/NOPB
- J4: footprint RoverFootprint:Molex_Mini-Fit_Jr_5569-08A2_2x04_P4.20mm_Horizontal -> Connector_Molex:Molex_Mini-Fit_Jr_5569-08A2_2x04_P4.20mm_Horizontal
Connections:
- net +24V_ETH: now also D3.1
- net +3.3V: now also U3.2 (OUTPUT)
- net GND: now also U3.1 (GND)
- net +5V_BMS: now reaches J4.5
- net +5V_BMS: now also R5.1
- net +5V: no longer names the net of C7.1, D3.4, D3.5
- net +5V: now also U3.3 (INPUT); no longer R5.1
- net PWM_EN renamed DIN2
- no-connect marks 35 -> 34
Other:
- moved on the sheet: C7, C8, D2, D3, R2

Commit message: 3D
Parts:
- D3: footprint DiodeSchott:UFV_TOS-L -> RoverFootprint:Diode_schottky-CVJ10F30
- J4: value 39301080 -> CONN-MOLEX_8PIN-39301080; footprint Connector_Molex:Molex_Mini-Fit_Jr_5569-08A2_2x04_P4.20mm_Horizontal -> RoverFootprint:CONN-MOLEX_8PIN-39301080
Changed lines of the file:
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@@
 			)
 		)
-		(property "Value" "39301080"
+		(property "Value" "CONN-MOLEX_8PIN-39301080"
 			(at 102.87 142.2399 0)
 			(effects
@@
 				)
 				(justify left)
+				(hide yes)
 			)
 		)
-		(property "Footprint" "Connector_Molex:Molex_Mini-Fit_Jr_5569-08A2_2x04_P4.20mm_Horizontal"
+		(property "Footprint" "RoverFootprint:CONN-MOLEX_8PIN-39301080"
 			(at 97.282 153.924 0)
 			(effects
@@
 			)
 		)
-		(property "Footprint" "DiodeSchott:UFV_TOS-L"
+		(property "Footprint" "RoverFootprint:Diode_schottky-CVJ10F30"
 			(at 61.214 250.444 0)
 			(effects

Commit message: BOM digikey
Parts:
- J1, J2: value Eth-Horiz-54601-908WPLF -> Eth-Horiz
- SW1, SW2: value TS09-63-25-WT-160-SMT-TR -> SW-PTS815SJM250SMTRLFS; Digikey https://www.digikey.ca/en/products/detail/same-sky-formerly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 -> (none); STATUS APPROVED -> (none)
- U1: value SN65HVD232Q -> SN65HVD232
- U5: value ESP32-S3-WROOM-1 -> ESP32-S3-WROVER
