File: rover/2025/CommBMS/latest/CommBMS.kicad_sch (KiCad schematic)
At the start: 7 parts

Commit message: Comm_bms2
Parts:
- added G1, G3: CONN_MOLEX, symbol RoverLibrary:Off Board Part
- added G10, G11, G12, G13, G14, G15, G16, G17, G18, G2, G4, G5, G6, G7, G8, G9: CRIMP, symbol RoverLibrary:Off Board Part
Other:
- note added: "3.3V"
- note added: "5V"
- note added: "CAN"
- note added: "CAN/RS485"
- note added: "PWM"

Commit message: commBMS modif
Parts:
- removed FID1, FID2, FID3: Fiducial, symbol Mechanical:Fiducial
Other:
- note added: "24V"
- note added: "RS485"
- note removed: "5V"
- note removed: "CAN/RS485"
Changed lines of the file:
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@@
 		)
 	)
-	(text "CAN/RS485"
+	(text "RS485"
 		(exclude_from_sim no)
 		(at 127 50.038 0)
@@
 		)
 	)
-	(text "5V"
+	(text "24V"
 		(exclude_from_sim no)
 		(at 76.962 57.404 0)
@@
 		)
 	)
-	(text "5V"
+	(text "24V"
 		(exclude_from_sim no)
 		(at 76.454 43.688 0)
@@
 	)
 	(symbol
-		(lib_id "Mechanical:Fiducial")
-		(at 114.3 120.65 0)
-		(unit 1)
-		(exclude_from_sim yes)
-		(in_bom no)
-		(on_board yes)
-		(dnp no)
-		(fields_autoplaced yes)
-		(property "Reference" "FID3"
-			(at 116.84 119.3799 0)
-			(effects
-				(font
-					(size 1.27 1.27)
-				)
-				(justify left)
-			)
-		)
-		(property "Value" "Fiducial"
-			(at 116.84 121.9199 0)
-			(effects
-				(font
-					(size 1.27 1.27)
-				)
-				(justify left)
-			)
-		)
-		(property "Footprint" ""
-			(at 114.3 120.65 0)
-			(effects
-				(font
-					(size 1.27 1.27)
-				)
-				(hide yes)
-			)
-		)
-		(property "Datasheet" "~"
-			(at 114.3 120.65 0)
-			(effects
-				(font
-					(size 1.27 1.27)
-				)
-				(hide yes)
-			)
-		)
-		(property "Description" "Fiducial Marker"
-			(at 114.3 120.65 0)
-			(effects
-				(font
-					(size 1.27 1.27)
-				)
-				(hide yes)
-			)
-		)
-		(instances
-			(project "ProjectTemplate"
-				(path "/a4fa9b30-7b48-474a-bdaa-0d7a6d26a697"
-					(reference "FID3")
-					(unit 1)
-				)
-			)
-		)
-	)
-	(symbol
 		(lib_id "RoverLibrary:Off Board Part")
 		(at 30.48 90.17 0)
@@
 	)
 	(symbol
-		(lib_id "Mechanical:Fiducial")
-		(at 114.3 107.95 0)
-		(unit 1)
-		(exclude_from_sim yes)
-		(in_bom no)
-		(on_board yes)
-		(dnp no)
-		(fields_autoplaced yes)
-		(property "Reference" "FID1"
-			(at 116.84 106.6799 0)
-			(effects
-				(font
-					(size 1.27 1.27)
-				)
-				(justify left)
-			)
-		)
-		(property "Value" "Fiducial"
-			(at 116.84 109.2199 0)
-			(effects
-				(font
-					(size 1.27 1.27)
-				)
-				(justify left)
-			)
-		)
-		(property "Footprint" ""
-			(at 114.3 107.95 0)
-			(effects
-				(font
-					(size 1.27 1.27)
-				)
-				(hide yes)
-			)
-		)
-		(property "Datasheet" "~"
-			(at 114.3 107.95 0)
-			(effects
-				(font
-					(size 1.27 1.27)
-				)
-				(hide yes)
-			)
-		)
-		(property "Description" "Fiducial Marker"
-			(at 114.3 107.95 0)
-			(effects
-				(font
-					(size 1.27 1.27)
-				)
-				(hide yes)
-			)
-		)
-		(instances
-			(project ""
-				(path "/a4fa9b30-7b48-474a-bdaa-0d7a6d26a697"
-					(reference "FID1")
-					(unit 1)
-				)
-			)
-		)
-	)
-	(symbol
 		(lib_id "RoverLibrary:Off Board Part")
 		(at 30.48 78.74 0)
@@
 					(unit 1)
 				)
-			)
-		)
-	)
-	(symbol
-		(lib_id "Mechanical:Fiducial")
-		(at 114.3 114.3 0)
-		(unit 1)
-		(exclude_from_sim yes)
-		(in_bom no)
-		(on_board yes)
-		(dnp no)
-		(fields_autoplaced yes)
-		(property "Reference" "FID2"
-			(at 116.84 113.0299 0)
-			(effects
-				(font
-					(size 1.27 1.27)
-				)
-				(justify left)
-			)
-		)
-		(property "Value" "Fiducial"
-			(at 116.84 115.5699 0)
-			(effects
-				(font
-					(size 1.27 1.27)
-				)
-				(justify left)
-			)
-		)
-		(property "Footprint" ""
-			(at 114.3 114.3 0)
-			(effects
-				(font
-					(size 1.27 1.27)
-				)
-				(hide yes)
-			)
-		)
-		(property "Datasheet" "~"
-			(at 114.3 114.3 0)
-			(effects
-				(font
-					(size 1.27 1.27)
-				)
-				(hide yes)
-			)
-		)
-		(property "Description" "Fiducial Marker"
-			(at 114.3 114.3 0)
-			(effects
-				(font
-					(size 1.27 1.27)
-				)
-				(hide yes)
-			)
-		)
-		(instances
-			(project "ProjectTemplate"
-				(path "/a4fa9b30-7b48-474a-bdaa-0d7a6d26a697"
-					(reference "FID2")
-					(unit 1)
-				)

Commit message: BOM digikey
Parts:
- G1: Digikey TODO -> https://www.digikey.com/en/products/detail/molex/0039012080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
- G5: Digikey TODO -> https://www.digikey.com/en/products/detail/molex/0039000038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
