File: rover/2025/GasConnBrd/Ref_board/Ref_board/Ref_board.kicad_sch (KiCad schematic)
At the start: 36 parts, among them J3 Eth-Horiz, J6 Eth-Horiz, J7 USB_C_USB4145-GCT, SW3 TS09-63-25-WT-160-SMT-TR, SW4 TS09-63-25-WT-160-SMT-TR, U10 LDO-TLV74033PDBVR, U11 DC_DC-AP64501, U3 SN65HVD232, U7 LDO-TLV74033PDBVR, U8 ESP32-S3-WROVER, U9 TVS

Commit message: Esp+Pwr_Added
Parts:
- removed C17: 10uF, Capacitor_SMD:C_0805_2012Metric_Pad1.18x1.45mm_HandSolder, symbol RoverLibrary:C-100nF
- removed C18, C19, C24, C25, C26: 10uF, Capacitor_SMD:C_0805_2012Metric_Pad1.18x1.45mm_HandSolder, symbol RoverLibrary:C_0805
- removed C2, C20, C23: 100nF, Capacitor_SMD:C_0805_2012Metric_Pad1.18x1.45mm_HandSolder, symbol RoverLibrary:C-100nF
- removed C21: 1uF, Capacitor_SMD:C_0805_2012Metric_Pad1.18x1.45mm_HandSolder, symbol RoverLibrary:C-1uF
- removed C22: 10uF, Capacitor_SMD:C_0805_2012Metric_Pad1.18x1.45mm_HandSolder, symbol RoverLibrary:C-22uF
- removed C27: 10nF, Capacitor_SMD:C_0805_2012Metric_Pad1.18x1.45mm_HandSolder, symbol RoverLibrary:C_0805
- removed C28: 100nF, Capacitor_SMD:C_0805_2012Metric_Pad1.18x1.45mm_HandSolder, symbol RoverLibrary:C_0805
- removed C29: 2.7nF, Capacitor_SMD:C_0805_2012Metric_Pad1.18x1.45mm_HandSolder, symbol RoverLibrary:C_0805
- removed C30, C31, C32: 22uF, Capacitor_SMD:C_0805_2012Metric_Pad1.18x1.45mm_HandSolder, symbol RoverLibrary:C_0805
- removed D4: CVJ10F30, RoverFootprint:Diode_schottky-CVJ10F30, symbol RoverLibrary:Diode_Schottchy_CVJ10F30
- removed D5: B, LED_SMD:LED_0805_2012Metric_Pad1.15x1.40mm_HandSolder, symbol RoverLibrary:LED
- removed J3, J6: Eth-Horiz, RoverFootprint:Ethernet_Horizontal, symbol RoverLibrary:Eth-Horiz-54601-908WPLF
- removed J7: USB_C_USB4145-GCT, RoverFootprint:USB4145_GCT, symbol RoverLibrary:USB_C_USB4145-03-C
- removed L2: 3.6uH, RoverFootprint:L_3.6u_ASPI-6045S-3R6N-T, symbol RoverLibrary:L_3.6u_ASPI-6045S-3R6N-T
- removed R10: 22.1k, Resistor_SMD:R_0805_2012Metric_Pad1.20x1.40mm_HandSolder, symbol RoverLibrary:R_0805
- removed R6: 1k, Resistor_SMD:R_0805_2012Metric_Pad1.20x1.40mm_HandSolder, symbol RoverLibrary:R-1k
- removed R7: 10k, Resistor_SMD:R_0805_2012Metric_Pad1.20x1.40mm_HandSolder, symbol RoverLibrary:R-10k
- removed R8: 15.8k, Resistor_SMD:R_0805_2012Metric_Pad1.20x1.40mm_HandSolder, symbol RoverLibrary:R_0805
- removed R9: 115k, Resistor_SMD:R_0805_2012Metric_Pad1.20x1.40mm_HandSolder, symbol RoverLibrary:R_0805
- removed SW3, SW4: TS09-63-25-WT-160-SMT-TR, Button_Switch_SMD:SW_DIP_SPSTx01_Slide_6.7x4.1mm_W8.61mm_P2.54mm_LowProfile, symbol RoverLibrary:PushButton-TS09-63-25-WT-160-SMT-TR
- removed U10, U7: LDO-TLV74033PDBVR, Package_TO_SOT_SMD:SOT-23-5_HandSoldering, symbol RoverLibrary:LDO-TLV74033PDBVR
- removed U11: DC_DC-AP64501, Package_SO:SOIC-8-1EP_3.9x4.9mm_P1.27mm_EP2.29x3mm, symbol RoverLibrary:DC_DC-AP64501
- removed U3: SN65HVD232, Package_SO:SOIC-8_3.9x4.9mm_P1.27mm, symbol RoverLibrary:CAN-Transceiver-SN65HVD232
- removed U8: ESP32-S3-WROVER, RF_Module:ESP32-S3-WROOM-1U, symbol RoverLibrary:ESP32-S3-WROVER
- removed U9: TVS, Package_SO:SOIC-8_3.9x4.9mm_P1.27mm, symbol RoverLibrary:TVS-SMDB03CE3/TR7TR-ND
- added C1, C4, C8: 100nF, Capacitor_SMD:C_0805_2012Metric_Pad1.18x1.45mm_HandSolder, symbol RoverLibrary:C-100nF
- added C10, C5, C6: 10uF, Capacitor_SMD:C_0805_2012Metric_Pad1.18x1.45mm_HandSolder, symbol RoverLibrary:C_0805
- added C11: 10nF, Capacitor_SMD:C_0805_2012Metric_Pad1.18x1.45mm_HandSolder, symbol RoverLibrary:C_0805
- added C12: 100nF, Capacitor_SMD:C_0805_2012Metric_Pad1.18x1.45mm_HandSolder, symbol RoverLibrary:C_0805
- added C13: 2.7nF, Capacitor_SMD:C_0805_2012Metric_Pad1.18x1.45mm_HandSolder, symbol RoverLibrary:C_0805
- added C14, C15, C16: 22uF, Capacitor_SMD:C_0805_2012Metric_Pad1.18x1.45mm_HandSolder, symbol RoverLibrary:C_0805
- added C3: 10uF, Capacitor_SMD:C_0805_2012Metric_Pad1.18x1.45mm_HandSolder, symbol RoverLibrary:C-100nF
- added C7: 1uF, Capacitor_SMD:C_0805_2012Metric_Pad1.18x1.45mm_HandSolder, symbol RoverLibrary:C-1uF
- added C9: 10uF, Capacitor_SMD:C_0805_2012Metric_Pad1.18x1.45mm_HandSolder, symbol RoverLibrary:C-22uF
- added D2: CVJ10F30, RoverFootprint:Diode_schottky-CVJ10F30, symbol RoverLibrary:Diode_Schottchy_CVJ10F30
- added D3: B, LED_SMD:LED_0805_2012Metric_Pad1.15x1.40mm_HandSolder, symbol RoverLibrary:LED
- added G1: PHR-6, symbol RoverLibrary:Off Board Part
- added G2: JUMPER 2PINS (QPC02SXGN-RC), symbol RoverLibrary:Off Board Part
- added H1, H2, H3, H4: MountingHole_Pad, MountingHole:MountingHole_3.2mm_M3_DIN965_Pad_TopBottom, symbol RoverLibrary:MountingHole_Pad
- added J1, J2: Eth-Horiz, RoverFootprint:Ethernet_Horizontal, symbol RoverLibrary:Eth-Horiz-54601-908WPLF
- added J4: JST6_Pin, Connector_JST:JST_PH_B6B-PH-K_1x06_P2.00mm_Vertical, symbol RoverLibrary:CONN-JST-XH-B6B
- added J5: USB_C_USB4145-GCT, RoverFootprint:USB4145_GCT, symbol RoverLibrary:USB_C_USB4145-03-C
- added L1: 3.6uH, RoverFootprint:L_3.6u_ASPI-6045S-3R6N-T, symbol RoverLibrary:L_3.6u_ASPI-6045S-3R6N-T
- added R1: 10k, Resistor_SMD:R_0805_2012Metric_Pad1.20x1.40mm_HandSolder, symbol RoverLibrary:R-10k
- added R2: 15.8k, Resistor_SMD:R_0805_2012Metric_Pad1.20x1.40mm_HandSolder, symbol RoverLibrary:R_0805
- added R3: 115k, Resistor_SMD:R_0805_2012Metric_Pad1.20x1.40mm_HandSolder, symbol RoverLibrary:R_0805
- added R4: 1k, Resistor_SMD:R_0805_2012Metric_Pad1.20x1.40mm_HandSolder, symbol RoverLibrary:R-1k
- added R5: 22.1k, Resistor_SMD:R_0805_2012Metric_Pad1.20x1.40mm_HandSolder, symbol RoverLibrary:R_0805
- added SW1, SW2: TS09-63-25-WT-160-SMT-TR, Button_Switch_SMD:SW_DIP_SPSTx01_Slide_6.7x4.1mm_W8.61mm_P2.54mm_LowProfile, symbol RoverLibrary:PushButton-TS09-63-25-WT-160-SMT-TR
- added U1: SN65HVD232, Package_SO:SOIC-8_3.9x4.9mm_P1.27mm, symbol RoverLibrary:CAN-Transceiver-SN65HVD232
- added U2: ESP32-S3-WROVER, RF_Module:ESP32-S3-WROOM-1U, symbol RoverLibrary:ESP32-S3-WROVER
- added U4: LDO-TLV74033PDBVR, Package_TO_SOT_SMD:SOT-23-5_HandSoldering, symbol RoverLibrary:LDO-TLV74033PDBVR
- added U5: TVS, Package_SO:SOIC-8_3.9x4.9mm_P1.27mm, symbol RoverLibrary:TVS-SMDB03CE3/TR7TR-ND
- added U6: DC_DC-AP64501, Package_SO:SOIC-8-1EP_3.9x4.9mm_P1.27mm_EP2.29x3mm, symbol RoverLibrary:DC_DC-AP64501
Connections:
- net +24V: now also C10.1, J1.5, J1.7, J2.5, J2.7, U6.2 (V_{in}), U6.3 (EN)
- net +3.3V: now also C3.1, C4.1, C5.1, C8.2, C9.1, R1.1, U1.3 (VCC), U2.2 (3V3), U4.5 (OUTPUT)
- net +5V: now also C6.1, D2.4, D2.5, J4.1, U4.1 (INPUT), U4.3 (EN)
- net +5V_ETH: now also C14.1, C15.1, C16.1, D2.3, L1.2, R3.1
- net +5V_USB: now also D2.1, J5.A4 (VBUS), J5.A9 (VBUS), J5.B4 (VBUS), J5.B9 (VBUS), U5.1
- net CAN_N: now also J1.2 (CANL), J2.2 (CANL), U1.6 (CANL)
- net CAN_P: now also J1.1 (CANH), J2.1 (CANH), U1.7 (CANH)
- net EN_ESP: now also C1.1, C7.1, R1.2, SW1.1, U2.3 (EN)
- net GND: now also C1.2, C10.2, C11.2, C13.2, C14.2, C15.2, C16.2, C3.2, C4.2, C5.2, C6.2, C7.2, C8.1, C9.2, D3.1 (K), H1.1, H2.1, H3.1, H4.1, J1.6, J1.8, J2.6, J2.8, J4.4, J5.A1 (GND), J5.A12 (GND), J5.B1 (GND), J5.B12 (GND), R5.2, SW1.2, SW2.1, U1.2 (GND), U1.8 (S), U2.1 (GND), U2.40 (GND), U2.41 (GND), U4.2 (GND), U5.5, U5.6, U5.7, U5.8, U6.7 (GND), U6.9 (PAD)
- net GNSS_EN: now also J4.6, U2.17 (IO9)
- net GNSS_PPS: now also J4.2, U2.25 (IO48)
- net GNSS_RX: now also J4.5, U2.21 (IO13)
- net GNSS_TX: now also J4.3, U2.24 (IO47)
- net GPIO_0: now also SW2.2, U2.27 (IO0-BOOT)
- net LED_BUILDIN: now also R4.1, U2.38 (IO2)
- net RXC: now also U1.1 (TXD), U2.5 (IO5)
- net TXC: now also U1.4 (RXD), U2.4 (IO4)
- net USB_N: now also J5.A7 (D-), J5.B7 (D-), U2.13 (IO19-USB_N), U5.2
- net USB_P: now also J5.A6 (D+), J5.B6 (D+), U2.14 (IO20-USB-P), U5.3
- new net: C11.1, U6.4 (SS)
- new net: C12.2, L1.1, U6.8 (SW)
- new net: R2.1, U6.6 (COMB)
- new net: C13.1, R2.2
- new net: C12.1, U6.1 (BST)
- new net: R3.2, R5.1, U6.5 (FB)
- new net: D3.2 (A), R4.2
Other:
- note added: "GNSS BUCK"
- note removed: "BUCK SI LDO PAS ASSEZ PUISSANT"
- note removed: "Power"
- company: ${GROUP_NAME} -> (none)
- title: ${PROJECTNAME} -> (none)
