File: exo/ACE 2026/Motherboard/MOBO_V2/_autosave-CAN.kicad_sch (KiCad schematic)
At the start: 7 parts, among them U501 MAX3221

Commit message: Clean up MoBo V2 et V2-1
Connections:
- net GPIO17_U1_TXD: no longer U203.32 (UART_RX)
- net GPIO18_U1_RXD: no longer U203.22 (UART_TX)
Other:
- moved on the sheet: U203E
Changed lines of the file:
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@@
+				)
+			)
+			(project "CAN"
+				(path "/b7f192b8-9b04-4f2f-9876-47892cc3e9de"
+					(reference "#PWR?")
+					(unit 1)
 				)
 			)
@@
 				)
 			)
+			(project "CAN"
+				(path "/b7f192b8-9b04-4f2f-9876-47892cc3e9de"
+					(reference "C?")
+					(unit 1)
+				)
+			)
 		)
 	)
@@
 				)
 			)
+			(project "CAN"
+				(path "/b7f192b8-9b04-4f2f-9876-47892cc3e9de"
+					(reference "C?")
+					(unit 1)
+				)
+			)
 		)
 	)
@@
 				)
 			)
+			(project "CAN"
+				(path "/b7f192b8-9b04-4f2f-9876-47892cc3e9de"
+					(reference "U?")
+					(unit 1)
+				)
+			)
 		)
 	)
@@
 				)
 			)
+			(project "CAN"
+				(path "/b7f192b8-9b04-4f2f-9876-47892cc3e9de"
+					(reference "#PWR?")
+					(unit 1)
+				)
+			)
 		)
 	)
 	(symbol
 		(lib_id "connecteur_m2_key_E:connecteur_SOM_ESP32_V2")
-		(at 36.83 34.29 0)
+		(at 101.6 20.32 0)
 		(unit 5)
 		(exclude_from_sim no)
@@
 		(dnp no)
 		(property "Reference" "U203"
-			(at 33.528 30.734 0)
+			(at 98.298 16.764 0)
 			(effects
 				(font
@@
 		)
 		(property "Value" "~"
-			(at 33.02 27.94 0)
+			(at 97.79 13.97 0)
 			(effects
 				(font
@@
 		)
 		(property "Footprint" "MDT320E01001:AMPHENOL_MDT320E01001"
-			(at 33.02 29.21 0)
+			(at 97.79 15.24 0)
 			(effects
 				(font
@@
 		)
 		(property "Datasheet" ""
-			(at 36.83 24.638 0)
+			(at 101.6 10.668 0)
 			(effects
 				(font
@@
 		)
 		(property "Description" ""
-			(at 36.83 24.638 0)
+			(at 101.6 10.668 0)
 			(effects
 				(font
@@
 					(reference "U203")
 					(unit 5)
+				)
+			)
+			(project "CAN"
+				(path "/b7f192b8-9b04-4f2f-9876-47892cc3e9de"
+					(reference "U?")
+					(unit 1)
 				)
 			)
@@
 				)
 			)
+			(project "CAN"
+				(path "/b7f192b8-9b04-4f2f-9876-47892cc3e9de"
+					(reference "C?")
+					(unit 1)
+				)
+			)
 		)
 	)
@@
 				)
 			)
+			(project "CAN"
+				(path "/b7f192b8-9b04-4f2f-9876-47892cc3e9de"
+					(reference "U?")
+					(unit 1)
+				)
+			)
 		)
 	)
@@
 				)
 			)
+			(project "CAN"
+				(path "/b7f192b8-9b04-4f2f-9876-47892cc3e9de"
+					(reference "C?")
+					(unit 1)
+				)
+			)
 		)
 	)
@@
 				)
 			)
+			(project "CAN"
+				(path "/b7f192b8-9b04-4f2f-9876-47892cc3e9de"
+					(reference "#PWR?")
+					(unit 1)
+				)
+			)
 		)
 	)
@@
 				)
 			)
+			(project "CAN"
+				(path "/b7f192b8-9b04-4f2f-9876-47892cc3e9de"
+					(reference "#PWR?")
+					(unit 1)
+				)
+			)
 		)
 	)
@@
 				)
 			)
+			(project "CAN"
+				(path "/b7f192b8-9b04-4f2f-9876-47892cc3e9de"
+					(reference "C?")
+					(unit 1)
+				)
+			)
 		)
 	)
@@
 				)
 			)
+			(project "CAN"
+				(path "/b7f192b8-9b04-4f2f-9876-47892cc3e9de"
+					(reference "#PWR?")
+					(unit 1)
+				)
+			)
 		)
 	)
@@
 				)
 			)
-		)
-	)
+			(project "CAN"
+				(path "/b7f192b8-9b04-4f2f-9876-47892cc3e9de"
+					(reference "#PWR?")
+					(unit 1)
+				)
+			)
+		)
+	)
+	(sheet_instances
+		(path "/"
+			(page "1")
+		)
+	)
