File: exo/ACE 2026/BNOV2/BNO_BREAKOUT.kicad_pcb (KiCad board)
At the start: 2 copper layers, 42 x 61.1 mm, 21 parts, among them M3 MountingHole_3.2mm_M3, U2 PCA9615DPZ, U3 AP7361C-33E

Commit message: Pushing changed files
multiple correctiosn done especially a new Mobo
Parts:
- removed C1: 4.7uF, Capacitor_SMD:C_1812_4532Metric_Pad1.57x3.40mm_HandSolder
- removed D4: D_TVS_Filled, Diode_SMD:D_0805_2012Metric
- removed Ethernet: RJ45, Connector_RJ:RJ45_Amphenol_54602-x08_Horizontal
- removed U2: PCA9615DPZ, Package_SO:TSSOP-10_3x3mm_P0.5mm
- added J2: RJ45, Connector_RJ:RJ45_Amphenol_54602-x08_Horizontal, F.Cu at (129.1, 114.0)
- added SCL: SCL, Connector_PinHeader_2.54mm:PinHeader_1x01_P2.54mm_Vertical, F.Cu at (139.4, 103.2)
- added SDA: SDA, Connector_PinHeader_2.54mm:PinHeader_1x01_P2.54mm_Vertical, F.Cu at (143.6, 103.2)
Routing:
- net /3V3: track 64.2 -> 43.6 mm, vias 9 -> 8
- net GND: track 28.6 -> 14.6 mm, vias 253 -> 254
- net /SDA: track 28.2 -> 36.6 mm
- net /5V: track 29.9 -> 22.0 mm
- net /SCL+: track 7.60 -> 0.00 mm
- net /SCL-: track 7.56 -> 0.00 mm
- net /SCL: track 18.5 -> 25.7 mm
- net /SDA+: track 6.96 -> 0.00 mm
- net /SDA-: track 6.85 -> 0.00 mm
Other:
- board text added: "BNO avec Protection anti-static"
- board text added: "PCB créer par: Jacob T."
- board text removed: "BNO avec I2C différentiel Protection anti-static"
- board text removed: "PCB créer par: Filip O. & Jacob T."
