File: exo/ACE 2026/Motherboard/MoBo_V2-1/Connecteurs.kicad_sch (KiCad schematic)
At the start: 40 parts, among them J701 RJ45, J702 RJ45, J703 RJ45

Commit message: Pushing changed files
multiple correctiosn done especially a new Mobo
Parts:
- removed H701, H702, H703, H704: MountingHole, MountingHole:MountingHole_3.2mm_M3, symbol Mechanical:MountingHole
- removed H705: MountingHole SoM, MountingHole:MountingHole_3.2mm_M3, symbol Mechanical:MountingHole
- removed JP1, JP2: SolderJumper_3_Bridged12, symbol Jumper:SolderJumper_3_Bridged12
- removed JP703, JP704, JP705, JP706, JP707, JP708, JP709, JP710, JP711, JP712, JP713, JP714: SolderJumper_2_Bridged, Jumper:SolderJumper-2_P1.3mm_Bridged_RoundedPad1.0x1.5mm, symbol Jumper:SolderJumper_2_Bridged
- removed R1, R10, R12, R13, R15, R16, R18, R3, R4, R6, R7, R9: 600, Resistor_SMD:R_0603_1608Metric_Pad0.98x0.95mm_HandSolder, symbol Device:R_US
- removed R11, R14, R17, R2, R5, R8: 110, Resistor_SMD:R_0603_1608Metric_Pad0.98x0.95mm_HandSolder, symbol Device:R_US
- added H1, H2, H3, H4: MountingHole, MountingHole:MountingHole_3.2mm_M3_ISO14580, symbol Mechanical:MountingHole
- added JP701, JP702: SolderJumper_3_Bridged12, Jumper:SolderJumper-3_P1.3mm_Bridged12_RoundedPad1.0x1.5mm, symbol Jumper:SolderJumper_3_Bridged12
- added R701, R702, R703, R704, R705, R706: 1k, Resistor_SMD:R_0805_2012Metric_Pad1.20x1.40mm_HandSolder, symbol Device:R_US
Connections:
- net CAN+: now also JP701.1 (A), JP701.2 (C)
- net CAN-: now also JP702.1 (A), JP702.2 (C)
- net DOS_SCL+ renamed I2C_SDA_0_TCA
- net I2C_SDA_0_TCA: now also R701.2
- net DOS_SCL- renamed I2C_SCL_0_TCA
- net I2C_SCL_0_TCA: now also R704.2
- net DOS_SDA+ renamed EXTRA_DOS_A0
- net DOS_SDA- renamed EXTRA_DOS_D2
- net D_SCL+ renamed I2C_SDA_1_TCA
- net I2C_SDA_1_TCA: now also R702.2
- net D_SCL- renamed I2C_SCL_1_TCA
- net I2C_SCL_1_TCA: now also R705.2
- net D_SDA+ renamed EXTRA_JAMBE_DR_A1
- net D_SDA- renamed EXTRA_JAMBE_DR_D3
- net G_SCL+ renamed I2C_SDA_2_TCA
- net I2C_SDA_2_TCA: now also R703.2
- net G_SCL- renamed I2C_SCL_2_TCA
- net I2C_SCL_2_TCA: now also R706.2
- net G_SDA+ renamed EXTRA_JAMBE_GA_A2
- net G_SDA- renamed EXTRA_JAMBE_GA_D4
- new net ESP32_RX: JP701.3 (B)
- new net ESP32_TX: JP702.3 (B)
- new net Vcc_3V3: R701.1, R702.1, R703.1, R704.1, R705.1, R706.1
Other:
- note removed: "Z_{eff} = 100 Ohm Voir datasheet PCA9615DP pour plus d'info"
