File: exo/ACE 2026/Moustache/Projet moustache.kicad_pcb (KiCad board)
At the start: 2 copper layers, 113.5 x 52.9 mm, 11 parts

Commit message: Pushing changed files
multiple correctiosn done especially a new Mobo
Parts:
- added C202: 4,7µF, Capacitor_SMD:C_0805_2012Metric_Pad1.18x1.45mm_HandSolder, F.Cu at (167.0, 60.5)
- added C204: 4,7µF, Capacitor_SMD:C_0805_2012Metric_Pad1.18x1.45mm_HandSolder, F.Cu at (171.5, 60.5)
- added D201: Green_power, Diode_SMD:D_0805_2012Metric, F.Cu at (168.0, 49.0)
- added R203: 330, Resistor_SMD:R_0805_2012Metric_Pad1.20x1.40mm_HandSolder, F.Cu at (164.0, 50.0)
- added R701: 1k, Resistor_SMD:R_0805_2012Metric_Pad1.20x1.40mm_HandSolder, F.Cu at (132.0, 61.0)
- added R704: 1k, Resistor_SMD:R_0805_2012Metric_Pad1.20x1.40mm_HandSolder, F.Cu at (127.5, 61.0)
- added TP201: TP_GND_IN, TestPoint:TestPoint_Pad_4.0x4.0mm, F.Cu at (179.5, 62.0)
- added TP203: TP_3v3, TestPoint:TestPoint_Pad_D4.0mm, F.Cu at (175.5, 68.7)
- added TP204: TP_5V, TestPoint:TestPoint_Pad_D4.0mm, F.Cu at (171.0, 73.5)
- added U201: AP7361C-33E, Package_TO_SOT_SMD:SOT-223-3_TabPin2, F.Cu at (169.0, 54.6)
- renumbered EXT2 to J1, MOTG to J2, BNOT to J3, EXT1 to J4, BNOF to J5, INPUT to J6, MOTH to J7
Connections:
- net +5V renamed Vcc_5V
- net /SCL+ renamed /SDA
- net /SCL- renamed /SCL
- net /SDA+ renamed /EXTRA_1
- net /SDA- renamed /EXTRA_2
Routing:
- net Vcc_3V3: track 0.00 -> 83.7 mm, vias 0 -> 3
- net Vcc_5V: track 122.2 -> 158.4 mm, vias 3 -> 5
- net GND: track 0.00 -> 5.58 mm, vias 453 -> 397
- net /SCL: track 130.5 -> 135.3 mm, vias 6 -> 7
- net /SDA: track 119.7 -> 123.8 mm, vias 6 -> 7
- net Net-(D201-A): track 0.00 -> 3.06 mm
Other:
- board text added: "CAN+ CAN- SDA SCL EXTRA EXTRA 5V GND"
- board text removed: "CAN+ CAN- SCL+ SCL- SDA+ SDA- 5V GND"
