File: rover/2026/CanTestModule/LATEST/CanTestModule.kicad_sch (KiCad schematic)
At the start: 8 parts, among them J1 ETH-RJHSE5081, J2 TerminalBlock

Commit message: 5 pos terminal block
Parts:
- removed J2: TerminalBlock, RoverFootprint:TerminalBlock-4_P5.00mm-691137710004, symbol RoverLibrary:TerminalBlock-4-691137710004
- added J2: TerminalBlock-5-691137710005, RoverFootprint:TerminalBlock-5_P5.00mm-691137710005, symbol RoverLibrary:TerminalBlock-5-691137710005
Connections:
- net 24V_in: now also J2.2
- net CANH: now also J2.4
- net CANL: now also J2.5
- net GND: now also J2.1, J2.3
